Commit message: Added mock controllers for both 2f and 3f grippers allowing for full simulation of the cell, joint values need to be changed though.

File: p5_ws/src/lbr_fri/lbr_fri_ros2_stack/lbr_description/urdf/mock_dual_arm/mock_dual_arm.xacro (robot description, xacro)
@@ -2,5 +2,5 @@
 <!-- top level -->
 <robot xmlns:xacro="http://www.ros.org/wiki/xacro" name="mock_dual_arm">
-  <!-- Setup of Hardware & Joints for Rigt_Arm_Mock -->
+  <!-- Setup of Hardware & Joints for Right_Arm_Mock -->
   <ros2_control name="lbr_system_interface_right" type="system">
     <hardware>
@@ -10,70 +10,91 @@
       <param name="max_velocity">1.710422666954443</param>
       <command_interface name="position">
+        <param name="min">-2.9670597283903604</param>
+        <param name="max">2.9670597283903604</param>
+      </command_interface>
+      <state_interface name="position">
         <param name="initial_value">0</param>
-	<param name="min">-2.9670597283903604</param>
-	<param name="max">2.9670597283903604</param>
-      </command_interface>
-      <state_interface name="position"/>
-      <state_interface name="velocity"/>
+      </state_interface>
+      <state_interface name="velocity">
+        <param name="initial_value">0.0</param>
+      </state_interface>
     </joint>
     <joint name="right_A2">
       <param name="max_velocity">1.710422666954443</param>
       <command_interface name="position">
+        <param name="min">-2.0943951023931953</param>
+        <param name="max">2.0943951023931953</param>
+      </command_interface>
+      <state_interface name="position">
         <param name="initial_value">0</param>
-	<param name="min">-2.0943951023931953</param>
-	<param name="max">2.0943951023931953</param>
-      </command_interface>
-      <state_interface name="position"/>
-      <state_interface name="velocity"/>
+      </state_interface>
+      <state_interface name="velocity">
+        <param name="initial_value">0.0</param>
+      </state_interface>
     </joint>
     <joint name="right_A3">
       <param name="max_velocity">1.7453292519943295</param>
       <command_interface name="position">
+        <param name="min">-2.9670597283903604</param>
+        <param name="max">2.9670597283903604</param>
+      </command_interface>
+      <state_interface name="position">
         <param name="initial_value">0</param>
-	<param name="min">-2.9670597283903604</param>
-	<param name="max">2.9670597283903604</param>
-      </command_interface>
-      <state_interface name="position"/>
-      <state_interface name="velocity"/>
+      </state_interface>
+      <state_interface name="velocity">
+        <param name="initial_value">0.0</param>
+      </state_interface>
     </joint>
     <joint name="right_A4">
       <param name="max_velocity">2.2689280275926285</param>
       <command_interface name="position">
+        <param name="min">-2.0943951023931953</param>
+        <param name="max">2.0943951023931953</param>
+      </command_interface>
+      <state_interface name="position">
         <param name="initial_value">0</param>
-	<param name="min">-2.0943951023931953</param>
-	<param name="max">2.0943951023931953</param>
-      </command_interface>
-      <state_interface name="position"/>
-      <state_interface name="velocity"/>
+      </state_interface>
+      <state_interface name="velocity">
+        <param name="initial_value">0.0</param>
+      </state_interface>
     </joint>
     <joint name="right_A5">
       <param name="max_velocity">2.443460952792061</param>
       <command_interface name="position">
+        <param name="min">-2.9670597283903604</param>
+        <param name="max">2.9670597283903604</param>
+      </command_interface>
+      <state_interface name="position">
         <param name="initial_value">0</param>
-	<param name="min">-2.9670597283903604</param>
-	<param name="max">2.9670597283903604</param>
-      </command_interface>
-      <state_interface name="position"/>
-      <state_interface name="velocity"/>
+      </state_interface>
+      <state_interface name="velocity">
+        <param name="initial_value">0.0</param>
+      </state_interface>
     </joint>
     <joint name="right_A6">
       <param name="max_velocity">3.141592653589793</param>
       <command_interface name="position">
+        <param name="min">-2.0943951023931953</param>
+        <param name="max">2.0943951023931953</param>
+      </command_interface>
+      <state_interface name="position">
         <param name="initial_value">0</param>
-	<param name="min">-2.0943951023931953</param>
-	<param name="max">2.0943951023931953</param>
-      </command_interface>
-      <state_interface name="position"/>
-      <state_interface name="velocity"/>
+      </state_interface>
+      <state_interface name="velocity">
+        <param name="initial_value">0.0</param>
+      </state_interface>
     </joint>
     <joint name="right_A7">
       <param name="max_velocity">3.141592653589793</param>
       <command_interface name="position">
+        <param name="min">-3.0543261909900763</param>
+        <param name="max">3.0543261909900763</param>
+      </command_interface>
+      <state_interface name="position">
         <param name="initial_value">0</param>
-	<param name="min">-3.0543261909900763</param>
-	<param name="max">3.0543261909900763</param>
-      </command_interface>
-      <state_interface name="position"/>
-      <state_interface name="velocity"/>
+      </state_interface>
+      <state_interface name="velocity">
+        <param name="initial_value">0.0</param>
+      </state_interface>
     </joint>
   </ros2_control>
@@ -86,70 +107,259 @@
       <param name="max_velocity">1.710422666954443</param>
       <command_interface name="position">
+        <param name="min">-2.9670597283903604</param>
+        <param name="max">2.9670597283903604</param>
+      </command_interface>
+      <state_interface name="position">
         <param name="initial_value">0</param>
-	<param name="min">-2.9670597283903604</param>
-	<param name="max">2.9670597283903604</param>
-      </command_interface>
-      <state_interface name="position"/>
-      <state_interface name="velocity"/>
+      </state_interface>
+      <state_interface name="velocity">
+        <param name="initial_value">0.0</param>
+      </state_interface>
     </joint>
     <joint name="left_A2">
       <param name="max_velocity">1.710422666954443</param>
       <command_interface name="position">
+        <param name="min">-2.0943951023931953</param>
+        <param name="max">2.0943951023931953</param>
+      </command_interface>
+      <state_interface name="position">
         <param name="initial_value">0</param>
-	<param name="min">-2.0943951023931953</param>
-	<param name="max">2.0943951023931953</param>
-      </command_interface>
-      <state_interface name="position"/>
-      <state_interface name="velocity"/>
+      </state_interface>
+      <state_interface name="velocity">
+        <param name="initial_value">0.0</param>
+      </state_interface>
     </joint>
     <joint name="left_A3">
       <param name="max_velocity">1.7453292519943295</param>
       <command_interface name="position">
+        <param name="min">-2.9670597283903604</param>
+        <param name="max">2.9670597283903604</param>
+      </command_interface>
+      <state_interface name="position">
         <param name="initial_value">0</param>
-	<param name="min">-2.9670597283903604</param>
-	<param name="max">2.9670597283903604</param>
-      </command_interface>
-      <state_interface name="position"/>
-      <state_interface name="velocity"/>
+      </state_interface>
+      <state_interface name="velocity">
+        <param name="initial_value">0.0</param>
+      </state_interface>
     </joint>
     <joint name="left_A4">
       <param name="max_velocity">2.2689280275926285</param>
       <command_interface name="position">
+        <param name="min">-2.0943951023931953</param>
+        <param name="max">2.0943951023931953</param>
+      </command_interface>
+      <state_interface name="position">
         <param name="initial_value">0</param>
-	<param name="min">-2.0943951023931953</param>
-	<param name="max">2.0943951023931953</param>
-      </command_interface>
-      <state_interface name="position"/>
-      <state_interface name="velocity"/>
+      </state_interface>
+      <state_interface name="velocity">
+        <param name="initial_value">0.0</param>
+      </state_interface>
     </joint>
     <joint name="left_A5">
       <param name="max_velocity">2.443460952792061</param>
       <command_interface name="position">
+        <param name="min">-2.9670597283903604</param>
+        <param name="max">2.9670597283903604</param>
+      </command_interface>
+      <state_interface name="position">
         <param name="initial_value">0</param>
-	<param name="min">-2.9670597283903604</param>
-	<param name="max">2.9670597283903604</param>
-      </command_interface>
-      <state_interface name="position"/>
-      <state_interface name="velocity"/>
+      </state_interface>
+      <state_interface name="velocity">
+        <param name="initial_value">0.0</param>
+      </state_interface>
     </joint>
     <joint name="left_A6">
       <param name="max_velocity">3.141592653589793</param>
       <command_interface name="position">
+        <param name="min">-2.0943951023931953</param>
+        <param name="max">2.0943951023931953</param>
+      </command_interface>
+      <state_interface name="position">
         <param name="initial_value">0</param>
-	<param name="min">-2.0943951023931953</param>
-	<param name="max">2.0943951023931953</param>
-      </command_interface>
-      <state_interface name="position"/>
-      <state_interface name="velocity"/>
+      </state_interface>
+      <state_interface name="velocity">
+        <param name="initial_value">0.0</param>
+      </state_interface>
     </joint>
     <joint name="left_A7">
       <param name="max_velocity">3.141592653589793</param>
       <command_interface name="position">
+        <param name="min">-3.0543261909900763</param>
+        <param name="max">3.0543261909900763</param>
+      </command_interface>
+      <state_interface name="position">
         <param name="initial_value">0</param>
-	<param name="min">-3.0543261909900763</param>
-	<param name="max">3.0543261909900763</param>
-      </command_interface>
-      <state_interface name="position"/>
-      <state_interface name="velocity"/>
+      </state_interface>
+      <state_interface name="velocity">
+        <param name="initial_value">0.0</param>
+      </state_interface>
+    </joint>
+  </ros2_control>
+  <!-- Setup of Hardware for 3F Gripper -->
+  <ros2_control name="3FGripper" type="system">
+    <hardware>
+      <plugin>mock_components/GenericSystem</plugin>
+    </hardware>
+    <joint name="3f_finger_1_joint_1">
+      <param name="max_velocity">1.23</param>
+      <command_interface name="position">
+        <param name="min">0.0495</param>
+        <param name="max">1.2218</param>
+      </command_interface>
+      <state_interface name="position">
+        <param name="initial_value">0.0495</param>
+      </state_interface>
+      <state_interface name="velocity">
+        <param name="initial_value">0.0</param>
+      </state_interface>
+    </joint>
+    <joint name="3f_finger_1_joint_2">
+      <param name="max_velocity">1.24</param>
+      <command_interface name="position">
+        <param name="min">0.0</param>
+        <param name="max">1.5708</param>
+      </command_interface>
+      <state_interface name="position">
+        <param name="initial_value">0.0</param>
+      </state_interface>
+      <state_interface name="velocity">
+        <param name="initial_value">0.0</param>
+      </state_interface>
+    </joint>
+    <joint name="3f_finger_1_joint_3">
+      <param name="max_velocity">1.25</param>
+      <command_interface name="position">
+        <param name="min">-1.2217</param>
+        <param name="max">-0.0523</param>
+      </command_interface>
+      <state_interface name="position">
+        <param name="initial_value">-1.2217</param>
+      </state_interface>
+      <state_interface name="velocity">
+        <param name="initial_value">0.0</param>
+      </state_interface>
+    </joint>
+    <joint name="3f_finger_2_joint_1">
+      <param name="max_velocity">1.23</param>
+      <command_interface name="position">
+        <param name="min">0.0495</param>
+        <param name="max">1.2218</param>
+      </command_interface>
+      <state_interface name="position">
+        <param name="initial_value">0.0495</param>
+      </state_interface>
+      <state_interface name="velocity">
+        <param name="initial_value">0.0</param>
+      </state_interface>
+    </joint>
+    <joint name="3f_finger_2_joint_2">
+      <param name="max_velocity">1.24</param>
+      <command_interface name="position">
+        <param name="min">0.0</param>
+        <param name="max">1.5708</param>
+      </command_interface>
+      <state_interface name="position">
+        <param name="initial_value">0.0</param>
+      </state_interface>
+      <state_interface name="velocity">
+        <param name="initial_value">0.0</param>
+      </state_interface>
+    </joint>
+    <joint name="3f_finger_2_joint_3">
+      <param name="max_velocity">1.25</param>
+      <command_interface name="position">
+        <param name="min">-1.2217</param>
+        <param name="max">-0.0523</param>
+      </command_interface>
+      <state_interface name="position">
+        <param name="initial_value">-1.2217</param>
+      </state_interface>
+      <state_interface name="velocity">
+        <param name="initial_value">0.0</param>
+      </state_interface>
+    </joint>
+    <joint name="3f_finger_middle_joint_1">
+      <param name="max_velocity">1.23</param>
+      <command_interface name="position">
+        <param name="min">0.0495</param>
+        <param name="max">1.2218</param>
+      </command_interface>
+      <state_interface name="position">
+        <param name="initial_value">0.0495</param>
+      </state_interface>
+      <state_interface name="velocity">
+        <param name="initial_value">0.0</param>
+      </state_interface>
+    </joint>
+    <joint name="3f_finger_middle_joint_2">
+      <param name="max_velocity">1.24</param>
+      <command_interface name="position">
+        <param name="min">0.0</param>
+        <param name="max">1.5708</param>
+      </command_interface>
+      <state_interface name="position">
+        <param name="initial_value">0.0</param>
+      </state_interface>
+      <state_interface name="velocity">
+        <param name="initial_value">0.0</param>
+      </state_interface>
+    </joint>
+    <joint name="3f_finger_middle_joint_3">
+      <param name="max_velocity">1.25</param>
+      <command_interface name="position">
+        <param name="min">-1.2217</param>
+        <param name="max">-0.0523</param>
+      </command_interface>
+      <state_interface name="position">
+        <param name="initial_value">-1.2217</param>
+      </state_interface>
+      <state_interface name="velocity">
+        <param name="initial_value">0.0</param>
+      </state_interface>
+    </joint>
+    <joint name="3f_palm_finger_1_joint">
+      <param name="max_velocity">1.23</param>
+      <command_interface name="position">
+        <param name="min">-0.1784</param>
+        <param name="max">0.192</param>
+      </command_interface>
+      <state_interface name="position">
+        <param name="initial_value">-0.1784</param>
+      </state_interface>
+      <state_interface name="velocity">
+        <param name="initial_value">0.0</param>
+      </state_interface>
+    </joint>
+    <joint name="3f_palm_finger_2_joint">
+      <param name="max_velocity">1.23</param>
+      <command_interface name="position">
+        <param name="min">-0.192</param>
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
Commit message: Fixed joint angles for 3F gripper to emulate real world gripper, 2F gripper still missing

File: p5_ws/src/lbr_fri/lbr_fri_ros2_stack/lbr_description/urdf/mock_dual_arm/mock_dual_arm.xacro (robot description, xacro)
@@ -204,9 +204,9 @@
       <param name="max_velocity">1.23</param>
       <command_interface name="position">
-        <param name="min">0.0495</param>
-        <param name="max">1.2218</param>
-      </command_interface>
-      <state_interface name="position">
-        <param name="initial_value">0.0495</param>
+        <param name="min">0.3758</param>
+        <param name="max">1.1276</param>
+      </command_interface>
+      <state_interface name="position">
+        <param name="initial_value">0.3758</param>
       </state_interface>
       <state_interface name="velocity">
@@ -221,5 +221,5 @@
       </command_interface>
       <state_interface name="position">
-        <param name="initial_value">0.0</param>
+        <param name="initial_value">0</param>
       </state_interface>
       <state_interface name="velocity">
@@ -230,9 +230,9 @@
       <param name="max_velocity">1.25</param>
       <command_interface name="position">
-        <param name="min">-1.2217</param>
-        <param name="max">-0.0523</param>
-      </command_interface>
-      <state_interface name="position">
-        <param name="initial_value">-1.2217</param>
+        <param name="min">-0.9531</param>
+        <param name="max">0.7572</param>
+      </command_interface>
+      <state_interface name="position">
+        <param name="initial_value">0.0</param>
       </state_interface>
       <state_interface name="velocity">
@@ -243,9 +243,9 @@
       <param name="max_velocity">1.23</param>
       <command_interface name="position">
-        <param name="min">0.0495</param>
-        <param name="max">1.2218</param>
-      </command_interface>
-      <state_interface name="position">
-        <param name="initial_value">0.0495</param>
+        <param name="min">0.3758</param>
+        <param name="max">1.1276</param>
+      </command_interface>
+      <state_interface name="position">
+        <param name="initial_value">0.3758</param>
       </state_interface>
       <state_interface name="velocity">
@@ -260,5 +260,5 @@
       </command_interface>
       <state_interface name="position">
-        <param name="initial_value">0.0</param>
+        <param name="initial_value">0</param>
       </state_interface>
       <state_interface name="velocity">
@@ -269,9 +269,9 @@
       <param name="max_velocity">1.25</param>
       <command_interface name="position">
-        <param name="min">-1.2217</param>
-        <param name="max">-0.0523</param>
-      </command_interface>
-      <state_interface name="position">
-        <param name="initial_value">-1.2217</param>
+        <param name="min">-0.9531</param>
+        <param name="max">0.7572</param>
+      </command_interface>
+      <state_interface name="position">
+        <param name="initial_value">0.0</param>
       </state_interface>
       <state_interface name="velocity">
@@ -282,9 +282,9 @@
       <param name="max_velocity">1.23</param>
       <command_interface name="position">
-        <param name="min">0.0495</param>
-        <param name="max">1.2218</param>
-      </command_interface>
-      <state_interface name="position">
-        <param name="initial_value">0.0495</param>
+        <param name="min">0.3758</param>
+        <param name="max">1.1276</param>
+      </command_interface>
+      <state_interface name="position">
+        <param name="initial_value">0.3758</param>
       </state_interface>
       <state_interface name="velocity">
@@ -308,9 +308,9 @@
       <param name="max_velocity">1.25</param>
       <command_interface name="position">
-        <param name="min">-1.2217</param>
-        <param name="max">-0.0523</param>
-      </command_interface>
-      <state_interface name="position">
-        <param name="initial_value">-1.2217</param>
+        <param name="min">-0.9531</param>
+        <param name="max">0.7572</param>
+      </command_interface>
+      <state_interface name="position">
+        <param name="initial_value">0</param>
       </state_interface>
       <state_interface name="velocity">
@@ -892,5 +892,5 @@
     <axis xyz="0 0 1"/>
     <origin rpy="0 0 -0.43" xyz="0.020 0 0"/>
-    <limit effort="100" lower="0.0495" upper="1.2218" velocity="1.23"/>
+    <limit effort="100" lower="0.3758" upper="1.1276" velocity="1.23"/>
     <dynamics damping="1" friction="0.1"/>
   </joint>
@@ -900,5 +900,5 @@
     <axis xyz="0 0 1"/>
     <origin rpy="0 0 -0.52" xyz="0.050 -.028 0"/>
-    <limit effort="100" lower="0.0" upper="1.5708" velocity="1.24"/>
+    <limit effort="100" lower="0.0" upper="1.5707" velocity="1.24"/>
     <dynamics damping="1" friction="0.1"/>
   </joint>
@@ -908,5 +908,5 @@
     <axis xyz="0 0 1"/>
     <origin rpy="0 0 0" xyz="0.039 0 0"/>
-    <limit effort="100" lower="-1.2217" upper="-0.0523" velocity="1.25"/>
+    <limit effort="100" lower="-0.9531" upper="0.7572" velocity="1.25"/>
     <dynamics damping="1" friction="0.1"/>
   </joint>
@@ -1008,5 +1008,5 @@
     <axis xyz="0 0 1"/>
     <origin rpy="0 0 -0.43" xyz="0.020 0 0"/>
-    <limit effort="100" lower="0.0495" upper="1.2218" velocity="1.23"/>
+    <limit effort="100" lower="0.3758" upper="1.1276" velocity="1.23"/>
     <dynamics damping="1" friction="0.1"/>
   </joint>
@@ -1016,5 +1016,5 @@
     <axis xyz="0 0 1"/>
     <origin rpy="0 0 -0.52" xyz="0.050 -.028 0"/>
-    <limit effort="100" lower="0.0" upper="1.5708" velocity="1.24"/>
+    <limit effort="100" lower="0.0" upper="1.5707" velocity="1.24"/>
     <dynamics damping="1" friction="0.1"/>
   </joint>
@@ -1024,5 +1024,5 @@
     <axis xyz="0 0 1"/>
     <origin rpy="0 0 0" xyz="0.039 0 0"/>
-    <limit effort="100" lower="-1.2217" upper="-0.0523" velocity="1.25"/>
+    <limit effort="100" lower="-0.9531" upper="0.7572" velocity="1.25"/>
     <dynamics damping="1" friction="0.1"/>
   </joint>
@@ -1124,5 +1124,5 @@
     <axis xyz="0 0 1"/>
     <origin rpy="0 0 -0.43" xyz="0.020 0 0"/>
-    <limit effort="100" lower="0.0495" upper="1.2218" velocity="1.23"/>
+    <limit effort="100" lower="0.3758" upper="1.1276" velocity="1.23"/>
     <dynamics damping="1" friction="0.1"/>
   </joint>
@@ -1132,5 +1132,5 @@
     <axis xyz="0 0 1"/>
     <origin rpy="0 0 -0.52" xyz="0.050 -.028 0"/>
-    <limit effort="100" lower="0.0" upper="1.5708" velocity="1.24"/>
+    <limit effort="100" lower="0.0" upper="1.5707" velocity="1.24"/>
     <dynamics damping="1" friction="0.1"/>
   </joint>
@@ -1140,5 +1140,5 @@
     <axis xyz="0 0 1"/>
     <origin rpy="0 0 0" xyz="0.039 0 0"/>
-    <limit effort="100" lower="-1.2217" upper="-0.0523" velocity="1.25"/>
+    <limit effort="100" lower="-0.9531" upper="0.7572" velocity="1.25"/>
     <dynamics damping="1" friction="0.1"/>
   </joint>
