Commit message: Fixed mock for 2F gripper, with this, simulation of the entire robot operation should now be possible in Rviz

File: p5_ws/src/lbr_fri/lbr_fri_ros2_stack/lbr_description/urdf/mock_dual_arm/mock_dual_arm.xacro (robot description, xacro)
@@ -1443,5 +1443,5 @@
     <child link="left_left_outer_knuckle"/>
     <axis xyz="1 0 0"/>
-    <limit effort="1000" lower="0" upper="0.8" velocity="2.0"/>
+    <limit effort="1000" lower="0" upper="0.8757" velocity="2.0"/>
   </joint>
   <joint name="left_left_outer_finger_joint" type="fixed"> <!-- Changes type from fixed to revolute-->
@@ -1466,6 +1466,6 @@
     <child link="left_left_inner_finger"/>
     <axis xyz="1 0 0"/>
-    <limit effort="1000" lower="0" upper="0.8757" velocity="2.0"/>
-    <mimic joint="left_finger_joint" multiplier="1" offset="0"/>
+    <limit effort="1000" lower="-0.8757" upper="0" velocity="2.0"/>
+    <mimic joint="left_finger_joint" multiplier="-1" offset="0"/>
   </joint>
   <joint name="left_left_inner_finger_pad_joint" type="fixed">
@@ -1480,5 +1480,5 @@
     <child link="left_right_outer_knuckle"/>
     <axis xyz="1 0 0"/>
-    <limit effort="1000" lower="0" upper="0.81" velocity="2.0"/>
+    <limit effort="1000" lower="0" upper="0.8757" velocity="2.0"/>
     <mimic joint="left_finger_joint" multiplier="1" offset="0"/>
   </joint>
@@ -1504,6 +1504,6 @@
     <child link="left_right_inner_finger"/>
     <axis xyz="1 0 0"/>
-    <limit effort="1000" lower="0" upper="0.8757" velocity="2.0"/>
-    <mimic joint="left_finger_joint" multiplier="1" offset="0"/>
+    <limit effort="1000" lower="-0.8757" upper="0" velocity="2.0"/>
+    <mimic joint="left_finger_joint" multiplier="-1" offset="0"/>
   </joint>
   <joint name="left_right_inner_finger_pad_joint" type="fixed">
