Commit message: Added new moveit_config pack isaac

File: p6_ws/src/lbr_fri/lbr_fri_ros2_stack/lbr_description/urdf/isaac_dual_arm/isaac_dual_arm.xacro (robot description, xacro)
@@ -1,221 +1,372 @@
-<?xml version="1.0" ?>
-<!-- =================================================================================== -->
-<!-- |    This document was autogenerated by xacro from src/lbr_fri/lbr_fri_ros2_stack/lbr_description/urdf/dual_arm/dual_arm.xacro | -->
-<!-- |    EDITING THIS FILE BY HAND IS NOT RECOMMENDED                                 | -->
-<!-- =================================================================================== -->
+<?xml version="1.0"?>
 <!-- top level -->
-<robot name="dual_arm">
-  <!-- include the right iiwa7 macro wit table
-    <xacro:include filename="$(find lbr_description)/urdf/dual_arm/dual_arm_description.xacro" />
-    -->
+<robot xmlns:xacro="http://www.ros.org/wiki/xacro" name="mock_dual_arm">
+  <!-- Setup of Hardware & Joints for Right_Arm_Mock -->
   <ros2_control name="lbr_system_interface_right" type="system">
     <hardware>
-      <plugin>lbr_ros2_control::SystemInterface</plugin>
-      <param name="fri_client_sdk_major_version">1</param>
-      <param name="fri_client_sdk_minor_version">15</param>
-      <param name="client_command_mode">position</param>
-      <param name="port_id">30200</param>
-      <param name="remote_host">INADDR_ANY</param>
-      <param name="rt_prio">80</param>
-      <param name="pid_p">0.1</param>
-      <param name="pid_i">0.0</param>
-      <param name="pid_d">0.0</param>
-      <param name="pid_i_max">0.0</param>
-      <param name="pid_i_min">0.0</param>
-      <param name="pid_antiwindup">False</param>
-      <param name="command_guard_variant">default</param>
-      <param name="external_torque_cutoff_frequency">10</param>
-      <param name="measured_torque_cutoff_frequency">10</param>
-      <param name="open_loop">True</param>
+      <plugin>topic_based_ros2_control/TopicBasedSystem</plugin>
+      <param name="joint_commands_topic">/right_arm/isaac_joint_commands</param>
+      <param name="joint_state_topic">/right_arm/isaac_joint_states</param>
     </hardware>
-    <sensor name="auxiliary_sensor">
-      <!-- see KUKA::FRI::LBRState -->
-      <state_interface name="sample_time"/>
-      <state_interface name="session_state"/>
-      <state_interface name="connection_quality"/>
-      <state_interface name="safety_state"/>
-      <state_interface name="operation_mode"/>
-      <state_interface name="drive_state"/>
-      <state_interface name="client_command_mode"/>
-      <state_interface name="overlay_type"/>
-      <state_interface name="control_mode"/>
-      <state_interface name="time_stamp_sec"/>
-      <state_interface name="time_stamp_nano_sec"/>
-      <state_interface name="tracking_performance"/>
-    </sensor>
-    <sensor name="estimated_ft_sensor">
-      <param name="chain_root">right_link_0</param>
-      <param name="chain_tip">right_link_ee</param>
-      <param name="damping">0.2</param>
-      <param name="force_x_th">2.0</param>
-      <param name="force_y_th">2.0</param>
-      <param name="force_z_th">2.0</param>
-      <param name="torque_x_th">0.5</param>
-      <param name="torque_y_th">0.5</param>
-      <param name="torque_z_th">0.5</param>
-      <state_interface name="force.x"/>
-      <state_interface name="force.y"/>
-      <state_interface name="force.z"/>
-      <state_interface name="torque.x"/>
-      <state_interface name="torque.y"/>
-      <state_interface name="torque.z"/>
-    </sensor>
-    <!-- FRI Cartesian impedance control mode -->
-    <gpio name="wrench">
-      <command_interface name="force.x"/>
-      <command_interface name="force.y"/>
-      <command_interface name="force.z"/>
-      <command_interface name="torque.x"/>
-      <command_interface name="torque.y"/>
-      <command_interface name="torque.z"/>
-    </gpio>
     <joint name="right_A1">
-      <param name="min_position">-2.9670597283903604</param>
-      <param name="max_position">2.9670597283903604</param>
       <param name="max_velocity">1.710422666954443</param>
-      <param name="max_torque">200</param>
       <command_interface name="position">
         <param name="min">-2.9670597283903604</param>
         <param name="max">2.9670597283903604</param>
       </command_interface>
-      <command_interface name="effort">
-        <param name="min">-200</param>
-        <param name="max"> 200</param>
-      </command_interface>
-      <state_interface name="position"/>
-      <state_interface name="velocity"/>
-      <state_interface name="effort"/>
-      <state_interface name="commanded_joint_position"/>
-      <state_interface name="commanded_torque"/>
-      <state_interface name="external_torque"/>
-      <state_interface name="ipo_joint_position"/>
+      <state_interface name="position">
+        <param name="initial_value">0</param>
+      </state_interface>
+      <state_interface name="velocity">
+        <param name="initial_value">0.0</param>
+      </state_interface>
     </joint>
     <joint name="right_A2">
-      <param name="min_position">-2.0943951023931953</param>
-      <param name="max_position">2.0943951023931953</param>
       <param name="max_velocity">1.710422666954443</param>
-      <param name="max_torque">200</param>
       <command_interface name="position">
         <param name="min">-2.0943951023931953</param>
         <param name="max">2.0943951023931953</param>
       </command_interface>
-      <command_interface name="effort">
-        <param name="min">-200</param>
-        <param name="max"> 200</param>
-      </command_interface>
-      <state_interface name="position"/>
-      <state_interface name="velocity"/>
-      <state_interface name="effort"/>
-      <state_interface name="commanded_joint_position"/>
-      <state_interface name="commanded_torque"/>
-      <state_interface name="external_torque"/>
-      <state_interface name="ipo_joint_position"/>
+      <state_interface name="position">
+        <param name="initial_value">0</param>
+      </state_interface>
+      <state_interface name="velocity">
+        <param name="initial_value">0.0</param>
+      </state_interface>
     </joint>
     <joint name="right_A3">
-      <param name="min_position">-2.9670597283903604</param>
-      <param name="max_position">2.9670597283903604</param>
       <param name="max_velocity">1.7453292519943295</param>
-      <param name="max_torque">200</param>
       <command_interface name="position">
         <param name="min">-2.9670597283903604</param>
         <param name="max">2.9670597283903604</param>
       </command_interface>
-      <command_interface name="effort">
-        <param name="min">-200</param>
-        <param name="max"> 200</param>
-      </command_interface>
-      <state_interface name="position"/>
-      <state_interface name="velocity"/>
-      <state_interface name="effort"/>
-      <state_interface name="commanded_joint_position"/>
-      <state_interface name="commanded_torque"/>
-      <state_interface name="external_torque"/>
-      <state_interface name="ipo_joint_position"/>
+      <state_interface name="position">
+        <param name="initial_value">0</param>
+      </state_interface>
+      <state_interface name="velocity">
+        <param name="initial_value">0.0</param>
+      </state_interface>
     </joint>
     <joint name="right_A4">
-      <param name="min_position">-2.0943951023931953</param>
-      <param name="max_position">2.0943951023931953</param>
       <param name="max_velocity">2.2689280275926285</param>
-      <param name="max_torque">200</param>
       <command_interface name="position">
         <param name="min">-2.0943951023931953</param>
         <param name="max">2.0943951023931953</param>
       </command_interface>
-      <command_interface name="effort">
-        <param name="min">-200</param>
-        <param name="max"> 200</param>
-      </command_interface>
-      <state_interface name="position"/>
-      <state_interface name="velocity"/>
-      <state_interface name="effort"/>
-      <state_interface name="commanded_joint_position"/>
-      <state_interface name="commanded_torque"/>
-      <state_interface name="external_torque"/>
-      <state_interface name="ipo_joint_position"/>
+      <state_interface name="position">
+        <param name="initial_value">0</param>
+      </state_interface>
+      <state_interface name="velocity">
+        <param name="initial_value">0.0</param>
+      </state_interface>
     </joint>
     <joint name="right_A5">
-      <param name="min_position">-2.9670597283903604</param>
-      <param name="max_position">2.9670597283903604</param>
       <param name="max_velocity">2.443460952792061</param>
-      <param name="max_torque">200</param>
       <command_interface name="position">
         <param name="min">-2.9670597283903604</param>
         <param name="max">2.9670597283903604</param>
       </command_interface>
-      <command_interface name="effort">
-        <param name="min">-200</param>
-        <param name="max"> 200</param>
-      </command_interface>
-      <state_interface name="position"/>
-      <state_interface name="velocity"/>
-      <state_interface name="effort"/>
-      <state_interface name="commanded_joint_position"/>
-      <state_interface name="commanded_torque"/>
-      <state_interface name="external_torque"/>
-      <state_interface name="ipo_joint_position"/>
+      <state_interface name="position">
+        <param name="initial_value">0</param>
+      </state_interface>
+      <state_interface name="velocity">
+        <param name="initial_value">0.0</param>
+      </state_interface>
     </joint>
     <joint name="right_A6">
-      <param name="min_position">-2.0943951023931953</param>
-      <param name="max_position">2.0943951023931953</param>
       <param name="max_velocity">3.141592653589793</param>
-      <param name="max_torque">200</param>
       <command_interface name="position">
         <param name="min">-2.0943951023931953</param>
         <param name="max">2.0943951023931953</param>
       </command_interface>
-      <command_interface name="effort">
-        <param name="min">-200</param>
-        <param name="max"> 200</param>
-      </command_interface>
-      <state_interface name="position"/>
-      <state_interface name="velocity"/>
-      <state_interface name="effort"/>
-      <state_interface name="commanded_joint_position"/>
-      <state_interface name="commanded_torque"/>
-      <state_interface name="external_torque"/>
-      <state_interface name="ipo_joint_position"/>
+      <state_interface name="position">
+        <param name="initial_value">0</param>
+      </state_interface>
+      <state_interface name="velocity">
+        <param name="initial_value">0.0</param>
+      </state_interface>
     </joint>
     <joint name="right_A7">
-      <param name="min_position">-3.0543261909900763</param>
-      <param name="max_position">3.0543261909900763</param>
       <param name="max_velocity">3.141592653589793</param>
-      <param name="max_torque">200</param>
       <command_interface name="position">
         <param name="min">-3.0543261909900763</param>
         <param name="max">3.0543261909900763</param>
       </command_interface>
-      <command_interface name="effort">
-        <param name="min">-200</param>
-        <param name="max"> 200</param>
-      </command_interface>
-      <state_interface name="position"/>
-      <state_interface name="velocity"/>
-      <state_interface name="effort"/>
-      <state_interface name="commanded_joint_position"/>
-      <state_interface name="commanded_torque"/>
-      <state_interface name="external_torque"/>
-      <state_interface name="ipo_joint_position"/>
+      <state_interface name="position">
+        <param name="initial_value">0</param>
+      </state_interface>
+      <state_interface name="velocity">
+        <param name="initial_value">0.0</param>
+      </state_interface>
     </joint>
   </ros2_control>
+  <!-- Setup of Hardware & Joints for Left_Arm_Mock -->
+  <ros2_control name="lbr_system_interface_left" type="system">
+    <hardware>
+      <plugin>topic_based_ros2_control/TopicBasedSystem</plugin>
+      <param name="joint_commands_topic">/left_arm/isaac_joint_commands</param>
+      <param name="joint_state_topic">/left_arm/isaac_joint_states</param>
+    </hardware>
+    <joint name="left_A1">
+      <param name="max_velocity">1.710422666954443</param>
+      <command_interface name="position">
+        <param name="min">-2.9670597283903604</param>
+        <param name="max">2.9670597283903604</param>
+      </command_interface>
+      <state_interface name="position">
+        <param name="initial_value">0</param>
+      </state_interface>
+      <state_interface name="velocity">
+        <param name="initial_value">0.0</param>
+      </state_interface>
+    </joint>
+    <joint name="left_A2">
+      <param name="max_velocity">1.710422666954443</param>
+      <command_interface name="position">
+        <param name="min">-2.0943951023931953</param>
+        <param name="max">2.0943951023931953</param>
+      </command_interface>
+      <state_interface name="position">
+        <param name="initial_value">0</param>
+      </state_interface>
+      <state_interface name="velocity">
+        <param name="initial_value">0.0</param>
+      </state_interface>
+    </joint>
+    <joint name="left_A3">
+      <param name="max_velocity">1.7453292519943295</param>
+      <command_interface name="position">
+        <param name="min">-2.9670597283903604</param>
+        <param name="max">2.9670597283903604</param>
+      </command_interface>
+      <state_interface name="position">
+        <param name="initial_value">0</param>
+      </state_interface>
+      <state_interface name="velocity">
+        <param name="initial_value">0.0</param>
+      </state_interface>
+    </joint>
+    <joint name="left_A4">
+      <param name="max_velocity">2.2689280275926285</param>
+      <command_interface name="position">
+        <param name="min">-2.0943951023931953</param>
+        <param name="max">2.0943951023931953</param>
+      </command_interface>
+      <state_interface name="position">
+        <param name="initial_value">0</param>
+      </state_interface>
+      <state_interface name="velocity">
+        <param name="initial_value">0.0</param>
+      </state_interface>
+    </joint>
+    <joint name="left_A5">
+      <param name="max_velocity">2.443460952792061</param>
+      <command_interface name="position">
+        <param name="min">-2.9670597283903604</param>
+        <param name="max">2.9670597283903604</param>
+      </command_interface>
+      <state_interface name="position">
+        <param name="initial_value">0</param>
+      </state_interface>
+      <state_interface name="velocity">
+        <param name="initial_value">0.0</param>
+      </state_interface>
+    </joint>
+    <joint name="left_A6">
+      <param name="max_velocity">3.141592653589793</param>
+      <command_interface name="position">
+        <param name="min">-2.0943951023931953</param>
+        <param name="max">2.0943951023931953</param>
+      </command_interface>
+      <state_interface name="position">
+        <param name="initial_value">0</param>
+      </state_interface>
+      <state_interface name="velocity">
+        <param name="initial_value">0.0</param>
+      </state_interface>
+    </joint>
+    <joint name="left_A7">
+      <param name="max_velocity">3.141592653589793</param>
+      <command_interface name="position">
+        <param name="min">-3.0543261909900763</param>
+        <param name="max">3.0543261909900763</param>
+      </command_interface>
+      <state_interface name="position">
+        <param name="initial_value">0</param>
+      </state_interface>
+      <state_interface name="velocity">
+        <param name="initial_value">0.0</param>
+      </state_interface>
+    </joint>
+  </ros2_control>
+  <!-- Setup of Hardware for 3F Gripper -->
+  <ros2_control name="3FGripper" type="system">
+    <hardware>
+      <plugin>mock_components/GenericSystem</plugin>
+    </hardware>
+    <joint name="3f_finger_1_joint_1">
+      <param name="max_velocity">1.23</param>
+      <command_interface name="position">
+        <param name="min">0.3758</param>
+        <param name="max">1.1276</param>
+      </command_interface>
+      <state_interface name="position">
+        <param name="initial_value">0.3758</param>
+      </state_interface>
+      <state_interface name="velocity">
+        <param name="initial_value">0.0</param>
+      </state_interface>
+    </joint>
+    <joint name="3f_finger_1_joint_2">
+      <param name="max_velocity">1.24</param>
+      <command_interface name="position">
+        <param name="min">0.0</param>
+        <param name="max">1.5708</param>
+      </command_interface>
+      <state_interface name="position">
+        <param name="initial_value">0</param>
+      </state_interface>
+      <state_interface name="velocity">
+        <param name="initial_value">0.0</param>
+      </state_interface>
+    </joint>
+    <joint name="3f_finger_1_joint_3">
+      <param name="max_velocity">1.25</param>
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
Commit message: Made isaac urdf

File: p6_ws/src/lbr_fri/lbr_fri_ros2_stack/lbr_description/urdf/isaac_dual_arm/isaac_dual_arm.xacro (robot description, xacro)
@@ -2,10 +2,10 @@
 <!-- top level -->
 <robot xmlns:xacro="http://www.ros.org/wiki/xacro" name="isaac_dual_arm">
-  <!-- Setup of Hardware & Joints for Right_Arm_Mock -->
+  <!-- Setup of Hardware & Joints for Right_Arm_Isaac -->
   <ros2_control name="lbr_system_interface_right" type="system">
     <hardware>
       <plugin>topic_based_ros2_control/TopicBasedSystem</plugin>
-      <param name="joint_commands_topic">/right_arm/isaac_joint_commands</param>
-      <param name="joint_state_topic">/right_arm/isaac_joint_states</param>
+      <param name="joint_commands_topic">/isaac_joint_commands</param>
+      <param name="joint_state_topic">/isaac_joint_states</param>
     </hardware>
     <joint name="right_A1">
@@ -101,10 +101,8 @@
     </joint>
   </ros2_control>
-  <!-- Setup of Hardware & Joints for Left_Arm_Mock -->
+  <!-- Setup of Hardware & Joints for Left_Arm_Isaac -->
   <ros2_control name="lbr_system_interface_left" type="system">
     <hardware>
-      <plugin>topic_based_ros2_control/TopicBasedSystem</plugin>
-      <param name="joint_commands_topic">/left_arm/isaac_joint_commands</param>
-      <param name="joint_state_topic">/left_arm/isaac_joint_states</param>
+      <plugin>mock_components/GenericSystem</plugin>
     </hardware>
     <joint name="left_A1">
@@ -159,5 +157,5 @@
         <param name="initial_value">0.0</param>
       </state_interface>
-    </joint>
+    </joint>right_arm
     <joint name="left_A5">
       <param name="max_velocity">2.443460952792061</param>

Commit message: Updated URDF with camera arm mount and new collision box

File: p6_ws/src/lbr_fri/lbr_fri_ros2_stack/lbr_description/urdf/isaac_dual_arm/isaac_dual_arm.xacro (robot description, xacro)
@@ -1599,5 +1599,21 @@
 	    </geometry>
 	</collision>
-    </link>
+  </link>
+  <!-- camera arm mount -->
+  <link name="camera_arm_mount">
+	<visual>
+	    <origin xyz="0 0 0" rpy="0 0 0"/>
+	    <geometry>
+	        <mesh filename="package://lbr_description/meshes/camera_arm_mount/Mount_realsense_camera_Default.stl" scale="0.001 0.001 0.001"/>
+	    </geometry>
+	    <material name="steel_satin"/>
+	</visual>
+	<collision>
+	    <origin xyz="0 0 0" rpy="0 0 0"/>
+	    <geometry>
+	        <mesh ilename="package://lbr_description/meshes/camera_arm_mount/Mount_realsense_camera_Default.stl"  scale="0.001 0.001 0.001"/>
+	    </geometry>
+	</collision>
+  </link>
   <!--joint between world and table-->
   <joint name="world_joint" type="fixed">
@@ -1636,9 +1652,15 @@
     <origin rpy="0 0 -2.35619449 " xyz="0.795181 0.79431 0.815"/>
   </joint>
-  <!-- joint between left iiwa7 and 2f gripper-->
+  <!-- joint between left iiwa7 and camera arm mount-->
+  <joint name="left_ee_cam" type="fixed">
+    <parent link="left_link_ee"/>
+    <child link="camera_arm_mount"/>
+    <origin rpy="0 0 0" xyz="0 0 0"/>
+  </joint>
+  <!-- joint between camera arm mount and 2f gripper-->
   <joint name="left_ee_mount" type="fixed">
-    <parent link="left_link_ee"/>
+    <parent link="camera_arm_mount"/>
     <child link="left_robotiq_arg2f_base_link"/>
-    <origin rpy="0 0 0" xyz="0 0 0"/>
+    <origin rpy="0 0 0" xyz="0 0 0.012"/>
   </joint>
   <!-- joint between left arm ee and 2f gripper-->

Commit message: Fixed xacro with proper camera mount collision and new srdf

File: p6_ws/src/lbr_fri/lbr_fri_ros2_stack/lbr_description/urdf/isaac_dual_arm/isaac_dual_arm.xacro (robot description, xacro)
@@ -2,7 +2,7 @@
 <!-- top level -->
 <robot xmlns:xacro="http://www.ros.org/wiki/xacro" name="isaac_dual_arm">
-<!-- Setup of Hardware & Joints for Right_Arm_Isaac -->
-<xacro:include filename="$(find isaac_dual_arm_moveit_config)/config/isaac_dual_arm.ros2_control.xacro"/>
-<!-- Links & Joints for the Right Arm -->
+  <!-- Setup of Hardware & Joints for Right_Arm_Isaac -->
+  <xacro:include filename="$(find isaac_dual_arm_moveit_config)/config/isaac_dual_arm.ros2_control.xacro"/>
+  <!-- Links & Joints for the Right Arm -->
   <link name="right_link_0">
     <inertial>
@@ -1248,5 +1248,5 @@
 	    <origin xyz="0 0 0" rpy="0 0 0"/>
 	    <geometry>
-	        <mesh ilename="package://lbr_description/meshes/camera_arm_mount/Mount_realsense_camera_Default.stl"  scale="0.001 0.001 0.001"/>
+	        <mesh filename="package://lbr_description/meshes/camera_arm_mount/Mount_realsense_camera_Default.stl" scale="0.001 0.001 0.001"/>
 	    </geometry>
 	</collision>
@@ -1302,5 +1302,5 @@
   <!-- joint between left arm ee and 2f gripper-->
   <joint name="2f_ee_tool0" type="fixed">
-    <parent link="left_link_ee"/>
+    <parent link="camera_arm_mount"/>
     <child link="2f_tool0"/>
     <origin rpy="0 3.14 0" xyz="0 0 0.165"/>
