Commit message: New isaac xacro with separted ros2 control

File: p6_ws/src/lbr_fri/lbr_fri_ros2_stack/lbr_description/urdf/isaac_dual_arm/isaac_dual_arm.urdf (robot description, URDF)
Before this commit: robot isaac_dual_arm, 47 links, 46 joints
Links:
- added link camera_arm_mount; collision mesh ilename=package://lbr_description/meshes/camera_arm_mount/Mount_rea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 scale=0.001 0.001 0.001; visual mesh filename=package://lbr_description/meshes/camera_arm_mount/Mount_rea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 scale=0.001 0.001 0.001
Joints:
- added joint left_ee_cam: type fixed, parent left_link_ee, child camera_arm_mount, origin xyz=0 0 0 rpy=0 0 0
- joint left_ee_mount: origin xyz=0 0 0 rpy=0 0 0 -> xyz=0 0 0.012 rpy=0 0 0; parent left_link_ee -> camera_arm_mount

File: p6_ws/src/lbr_fri/lbr_fri_ros2_stack/lbr_description/urdf/isaac_dual_arm/isaac_dual_arm.xacro (robot description, xacro)
@@ -2,370 +2,6 @@
 <!-- top level -->
 <robot xmlns:xacro="http://www.ros.org/wiki/xacro" name="isaac_dual_arm">
-  <!-- Setup of Hardware & Joints for Right_Arm_Isaac -->
-  <ros2_control name="lbr_system_interface_right" type="system">
-    <hardware>
-      <plugin>topic_based_ros2_control/TopicBasedSystem</plugin>
-      <param name="joint_commands_topic">/right_isaac_joint_commands</param>
-      <param name="joint_states_topic">/right_isaac_joint_states</param>
-    </hardware>
-    <joint name="right_A1">
-      <param name="max_velocity">1.710422666954443</param>
-      <command_interface name="position">
-        <param name="min">-2.9670597283903604</param>
-        <param name="max">2.9670597283903604</param>
-      </command_interface>
-      <state_interface name="position">
-        <param name="initial_value">0</param>
-      </state_interface>
-      <state_interface name="velocity">
-        <param name="initial_value">0.0</param>
-      </state_interface>
-    </joint>
-    <joint name="right_A2">
-      <param name="max_velocity">1.710422666954443</param>
-      <command_interface name="position">
-        <param name="min">-2.0943951023931953</param>
-        <param name="max">2.0943951023931953</param>
-      </command_interface>
-      <state_interface name="position">
-        <param name="initial_value">0</param>
-      </state_interface>
-      <state_interface name="velocity">
-        <param name="initial_value">0.0</param>
-      </state_interface>
-    </joint>
-    <joint name="right_A3">
-      <param name="max_velocity">1.7453292519943295</param>
-      <command_interface name="position">
-        <param name="min">-2.9670597283903604</param>
-        <param name="max">2.9670597283903604</param>
-      </command_interface>
-      <state_interface name="position">
-        <param name="initial_value">0</param>
-      </state_interface>
-      <state_interface name="velocity">
-        <param name="initial_value">0.0</param>
-      </state_interface>
-    </joint>
-    <joint name="right_A4">
-      <param name="max_velocity">2.2689280275926285</param>
-      <command_interface name="position">
-        <param name="min">-2.0943951023931953</param>
-        <param name="max">2.0943951023931953</param>
-      </command_interface>
-      <state_interface name="position">
-        <param name="initial_value">0</param>
-      </state_interface>
-      <state_interface name="velocity">
-        <param name="initial_value">0.0</param>
-      </state_interface>
-    </joint>
-    <joint name="right_A5">
-      <param name="max_velocity">2.443460952792061</param>
-      <command_interface name="position">
-        <param name="min">-2.9670597283903604</param>
-        <param name="max">2.9670597283903604</param>
-      </command_interface>
-      <state_interface name="position">
-        <param name="initial_value">0</param>
-      </state_interface>
-      <state_interface name="velocity">
-        <param name="initial_value">0.0</param>
-      </state_interface>
-    </joint>
-    <joint name="right_A6">
-      <param name="max_velocity">3.141592653589793</param>
-      <command_interface name="position">
-        <param name="min">-2.0943951023931953</param>
-        <param name="max">2.0943951023931953</param>
-      </command_interface>
-      <state_interface name="position">
-        <param name="initial_value">0</param>
-      </state_interface>
-      <state_interface name="velocity">
-        <param name="initial_value">0.0</param>
-      </state_interface>
-    </joint>
-    <joint name="right_A7">
-      <param name="max_velocity">3.141592653589793</param>
-      <command_interface name="position">
-        <param name="min">-3.0543261909900763</param>
-        <param name="max">3.0543261909900763</param>
-      </command_interface>
-      <state_interface name="position">
-        <param name="initial_value">0</param>
-      </state_interface>
-      <state_interface name="velocity">
-        <param name="initial_value">0.0</param>
-      </state_interface>
-    </joint>
-  </ros2_control>
-  <!-- Setup of Hardware & Joints for Left_Arm_Isaac -->
-  <ros2_control name="lbr_system_interface_left" type="system">
-    <hardware>
-      <plugin>topic_based_ros2_control/TopicBasedSystem</plugin>
-      <param name="joint_commands_topic">/left_isaac_joint_commands</param>
-      <param name="joint_states_topic">/left_isaac_joint_states</param>
-    </hardware>
-    <joint name="left_A1">
-      <param name="max_velocity">1.710422666954443</param>
-      <command_interface name="position">
-        <param name="min">-2.9670597283903604</param>
-        <param name="max">2.9670597283903604</param>
-      </command_interface>
-      <state_interface name="position">
-        <param name="initial_value">0</param>
-      </state_interface>
-      <state_interface name="velocity">
-        <param name="initial_value">0.0</param>
-      </state_interface>
-    </joint>
-    <joint name="left_A2">
-      <param name="max_velocity">1.710422666954443</param>
-      <command_interface name="position">
-        <param name="min">-2.0943951023931953</param>
-        <param name="max">2.0943951023931953</param>
-      </command_interface>
-      <state_interface name="position">
-        <param name="initial_value">0</param>
-      </state_interface>
-      <state_interface name="velocity">
-        <param name="initial_value">0.0</param>
-      </state_interface>
-    </joint>
-    <joint name="left_A3">
-      <param name="max_velocity">1.7453292519943295</param>
-      <command_interface name="position">
-        <param name="min">-2.9670597283903604</param>
-        <param name="max">2.9670597283903604</param>
-      </command_interface>
-      <state_interface name="position">
-        <param name="initial_value">0</param>
-      </state_interface>
-      <state_interface name="velocity">
-        <param name="initial_value">0.0</param>
-      </state_interface>
-    </joint>
-    <joint name="left_A4">
-      <param name="max_velocity">2.2689280275926285</param>
-      <command_interface name="position">
-        <param name="min">-2.0943951023931953</param>
-        <param name="max">2.0943951023931953</param>
-      </command_interface>
-      <state_interface name="position">
-        <param name="initial_value">0</param>
-      </state_interface>
-      <state_interface name="velocity">
-        <param name="initial_value">0.0</param>
-      </state_interface>
-    </joint>right_arm
-    <joint name="left_A5">
-      <param name="max_velocity">2.443460952792061</param>
-      <command_interface name="position">
-        <param name="min">-2.9670597283903604</param>
-        <param name="max">2.9670597283903604</param>
-      </command_interface>
-      <state_interface name="position">
-        <param name="initial_value">0</param>
-      </state_interface>
-      <state_interface name="velocity">
-        <param name="initial_value">0.0</param>
-      </state_interface>
-    </joint>
-    <joint name="left_A6">
-      <param name="max_velocity">3.141592653589793</param>
-      <command_interface name="position">
-        <param name="min">-2.0943951023931953</param>
-        <param name="max">2.0943951023931953</param>
-      </command_interface>
-      <state_interface name="position">
-        <param name="initial_value">0</param>
-      </state_interface>
-      <state_interface name="velocity">
-        <param name="initial_value">0.0</param>
-      </state_interface>
-    </joint>
-    <joint name="left_A7">
-      <param name="max_velocity">3.141592653589793</param>
-      <command_interface name="position">
-        <param name="min">-3.0543261909900763</param>
-        <param name="max">3.0543261909900763</param>
-      </command_interface>
-      <state_interface name="position">
-        <param name="initial_value">0</param>
-      </state_interface>
-      <state_interface name="velocity">
-        <param name="initial_value">0.0</param>
-      </state_interface>
-    </joint>
-  </ros2_control>
-  <!-- Setup of Hardware for 3F Gripper -->
-  <ros2_control name="3FGripper" type="system">
-    <hardware>
-      <plugin>mock_components/GenericSystem</plugin>
-    </hardware>
-    <joint name="3f_finger_1_joint_1">
-      <param name="max_velocity">1.23</param>
-      <command_interface name="position">
-        <param name="min">0.3758</param>
-        <param name="max">1.1276</param>
-      </command_interface>
-      <state_interface name="position">
-        <param name="initial_value">0.3758</param>
-      </state_interface>
-      <state_interface name="velocity">
-        <param name="initial_value">0.0</param>
-      </state_interface>
-    </joint>
-    <joint name="3f_finger_1_joint_2">
-      <param name="max_velocity">1.24</param>
-      <command_interface name="position">
-        <param name="min">0.0</param>
-        <param name="max">1.5708</param>
-      </command_interface>
-      <state_interface name="position">
-        <param name="initial_value">0</param>
-      </state_interface>
-      <state_interface name="velocity">
-        <param name="initial_value">0.0</param>
-      </state_interface>
-    </joint>
-    <joint name="3f_finger_1_joint_3">
-      <param name="max_velocity">1.25</param>
-      <command_interface name="position">
-        <param name="min">-0.9531</param>
-        <param name="max">0.7572</param>
-      </command_interface>
-      <state_interface name="position">
-        <param name="initial_value">0.0</param>
-      </state_interface>
-      <state_interface name="velocity">
-        <param name="initial_value">0.0</param>
-      </state_interface>
-    </joint>
-    <joint name="3f_finger_2_joint_1">
-      <param name="max_velocity">1.23</param>
-      <command_interface name="position">
-        <param name="min">0.3758</param>
-        <param name="max">1.1276</param>
-      </command_interface>
-      <state_interface name="position">
-        <param name="initial_value">0.3758</param>
-      </state_interface>
-      <state_interface name="velocity">
-        <param name="initial_value">0.0</param>
-      </state_interface>
-    </joint>
-    <joint name="3f_finger_2_joint_2">
-      <param name="max_velocity">1.24</param>
-      <command_interface name="position">
-        <param name="min">0.0</param>
-        <param name="max">1.5708</param>
-      </command_interface>
-      <state_interface name="position">
-        <param name="initial_value">0</param>
-      </state_interface>
-      <state_interface name="velocity">
-        <param name="initial_value">0.0</param>
-      </state_interface>
-    </joint>
-    <joint name="3f_finger_2_joint_3">
-      <param name="max_velocity">1.25</param>
-      <command_interface name="position">
-        <param name="min">-0.9531</param>
-        <param name="max">0.7572</param>
-      </command_interface>
-      <state_interface name="position">
-        <param name="initial_value">0.0</param>
-      </state_interface>
-      <state_interface name="velocity">
-        <param name="initial_value">0.0</param>
-      </state_interface>
-    </joint>
-    <joint name="3f_finger_middle_joint_1">
-      <param name="max_velocity">1.23</param>
-      <command_interface name="position">
-        <param name="min">0.3758</param>
-        <param name="max">1.1276</param>
-      </command_interface>
-      <state_interface name="position">
-        <param name="initial_value">0.3758</param>
-      </state_interface>
-      <state_interface name="velocity">
-        <param name="initial_value">0.0</param>
-      </state_interface>
-    </joint>
-    <joint name="3f_finger_middle_joint_2">
-      <param name="max_velocity">1.24</param>
-      <command_interface name="position">
-        <param name="min">0.0</param>
-        <param name="max">1.5708</param>
-      </command_interface>
-      <state_interface name="position">
-        <param name="initial_value">0.0</param>
-      </state_interface>
-      <state_interface name="velocity">
-        <param name="initial_value">0.0</param>
-      </state_interface>
-    </joint>
-    <joint name="3f_finger_middle_joint_3">
-      <param name="max_velocity">1.25</param>
-      <command_interface name="position">
-        <param name="min">-0.9531</param>
-        <param name="max">0.7572</param>
-      </command_interface>
-      <state_interface name="position">
-        <param name="initial_value">0</param>
-      </state_interface>
-      <state_interface name="velocity">
-        <param name="initial_value">0.0</param>
-      </state_interface>
-    </joint>
-    <joint name="3f_palm_finger_1_joint">
-      <param name="max_velocity">1.23</param>
-      <command_interface name="position">
-        <param name="min">-0.1784</param>
-        <param name="max">0.192</param>
-      </command_interface>
-      <state_interface name="position">
-        <param name="initial_value">-0.1784</param>
-      </state_interface>
-      <state_interface name="velocity">
-        <param name="initial_value">0.0</param>
-      </state_interface>
-    </joint>
-    <joint name="3f_palm_finger_2_joint">
-      <param name="max_velocity">1.23</param>
-      <command_interface name="position">
-        <param name="min">-0.192</param>
-        <param name="max">0.1784</param>
-      </command_interface>
-      <state_interface name="position">
-        <param name="initial_value">-0.192</param>
-      </state_interface>
-      <state_interface name="velocity">
-        <param name="initial_value">0.0</param>
-      </state_interface>
-    </joint>
-  </ros2_control>
-  <!-- Setup of Hardware for 2F Gripper -->
-  <ros2_control name="2FGripper" type="system">
-    <hardware>
-      <plugin>mock_components/GenericSystem</plugin>
-    </hardware>
-    <joint name="left_finger_joint">
-      <param name="max_velocity">2</param>
-      <command_interface name="position">
-        <param name="min">0.0</param>
-        <param name="max">0.8</param>
-      </command_interface>
-      <state_interface name="position">
-        <param name="initial_value">0.0</param>
-      </state_interface>
-      <state_interface name="velocity">
-        <param name="initial_value">0.0</param>
-      </state_interface>
-    </joint>
-  </ros2_control>
+<!-- Setup of Hardware & Joints for Right_Arm_Isaac -->
+<xacro:include filename="$(find isaac_dual_arm_moveit_config)/config/isaac_dual_arm.ros2_control.xacro"/>
 <!-- Links & Joints for the Right Arm -->
   <link name="right_link_0">
