Commit message: Added new 2f robotiq gripper, and updated srdf

File: p6_ws/src/lbr_fri/lbr_fri_ros2_stack/lbr_description/urdf/robotiq-2f-85-gripper/robotiq_85_gripper.urdf.xacro (robot description, xacro)
@@ -10,10 +10,10 @@
       <visual>
         <geometry>
-          <mesh filename="package://robot_description/meshes/ur5/visual/robotiq_85_base_link.dae"/>
-        </geometry>
-      </visual>
-      <collision>
-        <geometry>
-          <mesh filename="package://robot_description/meshes/ur5/collision/robotiq_85_base_link.stl"/>
+          <mesh filename="package://lbr_description/meshes/robotiq_2f_85_gripper/visual/robotiq_85_base_link.dae"/>
+        </geometry>
+      </visual>
+      <collision>
+        <geometry>
+          <mesh filename="package://lbr_description/meshes/robotiq_2f_85_gripper/collision/robotiq_85_base_link.stl"/>
         </geometry>
       </collision>
@@ -44,10 +44,10 @@
       <visual>
         <geometry>
-          <mesh filename="package://robot_description/meshes/ur5/visual/robotiq_85_knuckle_link.dae"/>
-        </geometry>
-      </visual>
-      <collision>
-        <geometry>
-          <mesh filename="package://robot_description/meshes/ur5/collision/robotiq_85_knuckle_link.stl"/>
+          <mesh filename="package://lbr_description/meshes/robotiq_2f_85_gripper/visual/robotiq_85_knuckle_link.dae"/>
+        </geometry>
+      </visual>
+      <collision>
+        <geometry>
+          <mesh filename="package://lbr_description/meshes/robotiq_2f_85_gripper/collision/robotiq_85_knuckle_link.stl"/>
         </geometry>
       </collision>
@@ -63,10 +63,10 @@
       <visual>
         <geometry>
-          <mesh filename="package://robot_description/meshes/ur5/visual/robotiq_85_knuckle_link.dae"/>
-        </geometry>
-      </visual>
-      <collision>
-        <geometry>
-          <mesh filename="package://robot_description/meshes/ur5/collision/robotiq_85_knuckle_link.stl"/>
+          <mesh filename="package://lbr_description/meshes/robotiq_2f_85_gripper/visual/robotiq_85_knuckle_link.dae"/>
+        </geometry>
+      </visual>
+      <collision>
+        <geometry>
+          <mesh filename="package://lbr_description/meshes/robotiq_2f_85_gripper/collision/robotiq_85_knuckle_link.stl"/>
         </geometry>
       </collision>
@@ -92,10 +92,10 @@
       <visual>
         <geometry>
-          <mesh filename="package://robot_description/meshes/ur5/visual/robotiq_85_finger_link.dae"/>
-        </geometry>
-      </visual>
-      <collision>
-        <geometry>
-          <mesh filename="package://robot_description/meshes/ur5/collision/robotiq_85_finger_link.stl"/>
+          <mesh filename="package://lbr_description/meshes/robotiq_2f_85_gripper/visual/robotiq_85_finger_link.dae"/>
+        </geometry>
+      </visual>
+      <collision>
+        <geometry>
+          <mesh filename="package://lbr_description/meshes/robotiq_2f_85_gripper/collision/robotiq_85_finger_link.stl"/>
         </geometry>
       </collision>
@@ -111,10 +111,10 @@
       <visual>
         <geometry>
-          <mesh filename="package://robot_description/meshes/ur5/visual/robotiq_85_finger_link.dae"/>
-        </geometry>
-      </visual>
-      <collision>
-        <geometry>
-          <mesh filename="package://robot_description/meshes/ur5/collision/robotiq_85_finger_link.stl"/>
+          <mesh filename="package://lbr_description/meshes/robotiq_2f_85_gripper/visual/robotiq_85_finger_link.dae"/>
+        </geometry>
+      </visual>
+      <collision>
+        <geometry>
+          <mesh filename="package://lbr_description/meshes/robotiq_2f_85_gripper/collision/robotiq_85_finger_link.stl"/>
         </geometry>
       </collision>
@@ -146,10 +146,10 @@
       <visual>
         <geometry>
-          <mesh filename="package://robot_description/meshes/ur5/visual/robotiq_85_inner_knuckle_link.dae"/>
-        </geometry>
-      </visual>
-      <collision>
-        <geometry>
-          <mesh filename="package://robot_description/meshes/ur5/collision/robotiq_85_inner_knuckle_link.stl"/>
+          <mesh filename="package://lbr_description/meshes/robotiq_2f_85_gripper/visual/robotiq_85_inner_knuckle_link.dae"/>
+        </geometry>
+      </visual>
+      <collision>
+        <geometry>
+          <mesh filename="package://lbr_description/meshes/robotiq_2f_85_gripper/collision/robotiq_85_inner_knuckle_link.stl"/>
         </geometry>
       </collision>
@@ -165,10 +165,10 @@
       <visual>
         <geometry>
-          <mesh filename="package://robot_description/meshes/ur5/visual/robotiq_85_inner_knuckle_link.dae"/>
-        </geometry>
-      </visual>
-      <collision>
-        <geometry>
-          <mesh filename="package://robot_description/meshes/ur5/collision/robotiq_85_inner_knuckle_link.stl"/>
+          <mesh filename="package://lbr_description/meshes/robotiq_2f_85_gripper/visual/robotiq_85_inner_knuckle_link.dae"/>
+        </geometry>
+      </visual>
+      <collision>
+        <geometry>
+          <mesh filename="package://lbr_description/meshes/robotiq_2f_85_gripper/collision/robotiq_85_inner_knuckle_link.stl"/>
         </geometry>
       </collision>
@@ -200,10 +200,10 @@
       <visual>
         <geometry>
-          <mesh filename="package://robot_description/meshes/ur5/visual/robotiq_85_finger_tip_link.dae"/>
-        </geometry>
-      </visual>
-      <collision>
-        <geometry>
-          <mesh filename="package://robot_description/meshes/ur5/collision/robotiq_85_finger_tip_link.stl"/>
+          <mesh filename="package://lbr_description/meshes/robotiq_2f_85_gripper/visual/robotiq_85_finger_tip_link.dae"/>
+        </geometry>
+      </visual>
+      <collision>
+        <geometry>
+          <mesh filename="package://lbr_description/meshes/robotiq_2f_85_gripper/collision/robotiq_85_finger_tip_link.stl"/>
         </geometry>
       </collision>
@@ -219,10 +219,10 @@
       <visual>
         <geometry>
-          <mesh filename="package://robot_description/meshes/ur5/visual/robotiq_85_finger_tip_link.dae"/>
-        </geometry>
-      </visual>
-      <collision>
-        <geometry>
-          <mesh filename="package://robot_description/meshes/ur5/collision/robotiq_85_finger_tip_link.stl"/>
+          <mesh filename="package://lbr_description/meshes/robotiq_2f_85_gripper/visual/robotiq_85_finger_tip_link.dae"/>
+        </geometry>
+      </visual>
+      <collision>
+        <geometry>
+          <mesh filename="package://lbr_description/meshes/robotiq_2f_85_gripper/collision/robotiq_85_finger_tip_link.stl"/>
         </geometry>
       </collision>
@@ -235,5 +235,5 @@
       </inertial>
     </link>
-    <!-- Improve grasping physics -->
+    <!-- Improve grasping physics
     <gazebo reference="${prefix}robotiq_85_left_finger_tip_link">
       <kp>1000000.0</kp>
@@ -250,4 +250,5 @@
       <minDepth>0.001</minDepth>
     </gazebo>
+    -->
   </xacro:macro>
 </robot>

File: p6_ws/src/lbr_fri/lbr_fri_ros2_stack/lbr_moveit_config/isaac_dual_arm_moveit_config/config/isaac_dual_arm.ros2_control.xacro (robot description, xacro)
@@ -191,5 +191,5 @@
     </joint>
     <!-- Setup of Hardware for 2F Gripper -->
-    <joint name="left_finger_joint">
+    <joint name="2f_robotiq_85_left_knuckle_joint">
       <param name="max_velocity">2</param>
       <command_interface name="position">

Commit message: Name change for 2f gripper in isaac xacro and urdf

File: p6_ws/src/lbr_fri/lbr_fri_ros2_stack/lbr_description/urdf/isaac_dual_arm/isaac_dual_arm.urdf (robot description, URDF)
Before this commit: robot isaac_dual_arm, 52 links, 51 joints
Links:
- removed link 2f_robotiq_85_base_link
- removed link 2f_robotiq_85_left_finger_link
- removed link 2f_robotiq_85_left_finger_tip_link
- removed link 2f_robotiq_85_left_inner_knuckle_link
- removed link 2f_robotiq_85_left_knuckle_link
- removed link 2f_robotiq_85_right_finger_link
- removed link 2f_robotiq_85_right_finger_tip_link
- removed link 2f_robotiq_85_right_inner_knuckle_link
- removed link 2f_robotiq_85_right_knuckle_link
- added link left_2f_robotiq_85_base_link, mass 0.636951; collision mesh filename=package://lbr_description/meshes/robotiq_2f_85_gripper/coll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; visual mesh filename=package://lbr_description/meshes/robotiq_2f_85_gripper/visu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
- added link left_2f_robotiq_85_left_finger_link, mass 0.027309; collision mesh filename=package://lbr_description/meshes/robotiq_2f_85_gripper/coll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; visual mesh filename=package://lbr_description/meshes/robotiq_2f_85_gripper/visu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
- added link left_2f_robotiq_85_left_finger_tip_link, mass 0.019555; collision mesh filename=package://lbr_description/meshes/robotiq_2f_85_gripper/coll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; visual mesh filename=package://lbr_description/meshes/robotiq_2f_85_gripper/visu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
- added link left_2f_robotiq_85_left_inner_knuckle_link, mass 0.029951; collision mesh filename=package://lbr_description/meshes/robotiq_2f_85_gripper/coll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; visual mesh filename=package://lbr_description/meshes/robotiq_2f_85_gripper/visu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
- added link left_2f_robotiq_85_left_knuckle_link, mass 0.018491; collision mesh filename=package://lbr_description/meshes/robotiq_2f_85_gripper/coll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; visual mesh filename=package://lbr_description/meshes/robotiq_2f_85_gripper/visu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
- added link left_2f_robotiq_85_right_finger_link, mass 0.027309; collision mesh filename=package://lbr_description/meshes/robotiq_2f_85_gripper/coll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; visual mesh filename=package://lbr_description/meshes/robotiq_2f_85_gripper/visu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
- added link left_2f_robotiq_85_right_finger_tip_link, mass 0.019555; collision mesh filename=package://lbr_description/meshes/robotiq_2f_85_gripper/coll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; visual mesh filename=package://lbr_description/meshes/robotiq_2f_85_gripper/visu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
- added link left_2f_robotiq_85_right_inner_knuckle_link, mass 0.029951; collision mesh filename=package://lbr_description/meshes/robotiq_2f_85_gripper/coll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; visual mesh filename=package://lbr_description/meshes/robotiq_2f_85_gripper/visu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
- added link left_2f_robotiq_85_right_knuckle_link, mass 0.018491; collision mesh filename=package://lbr_description/meshes/robotiq_2f_85_gripper/coll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; visual mesh filename=package://lbr_description/meshes/robotiq_2f_85_gripper/visu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
Joints:
- removed joint 2f_robotiq_85_base_joint
- removed joint 2f_robotiq_85_left_finger_joint
- removed joint 2f_robotiq_85_left_finger_tip_joint
- removed joint 2f_robotiq_85_left_inner_knuckle_joint
- removed joint 2f_robotiq_85_left_knuckle_joint
- removed joint 2f_robotiq_85_right_finger_joint
- removed joint 2f_robotiq_85_right_finger_tip_joint
- removed joint 2f_robotiq_85_right_inner_knuckle_joint
- removed joint 2f_robotiq_85_right_knuckle_joint
- added joint left_2f_robotiq_85_base_joint: type fixed, parent camera_arm_mount, child left_2f_robotiq_85_base_link, origin xyz=0 0 0.012 rpy=0 -1.5707 0
- added joint left_2f_robotiq_85_left_finger_joint: type fixed, parent left_2f_robotiq_85_left_knuckle_link, child left_2f_robotiq_85_left_finger_link, origin xyz=-0.00408552455 -0.03148604435 0.0 rpy=0 0 0
- added joint left_2f_robotiq_85_left_finger_tip_joint: type continuous, parent left_2f_robotiq_85_left_inner_knuckle_link, child left_2f_robotiq_85_left_finger_tip_link, origin xyz=0.04303959807 -0.03759940821 0.0 rpy=0.0 0.0 0.0, axis 0 0 1, limit lower=-3.14 upper=3.14 effort=0.1 velocity=100.0, mimic joint=left_2f_robotiq_85_left_knuckle_joint multiplier=-1
- added joint left_2f_robotiq_85_left_inner_knuckle_joint: type continuous, parent left_2f_robotiq_85_base_link, child left_2f_robotiq_85_left_inner_knuckle_link, origin xyz=0.06142 0.0127 0 rpy=3.141592653589793 0.0 0.0, axis 0 0 1, limit lower=-3.14 upper=3.14 effort=0.1 velocity=100.0, mimic joint=left_2f_robotiq_85_left_knuckle_joint offset=0
- added joint left_2f_robotiq_85_left_knuckle_joint: type revolute, parent left_2f_robotiq_85_base_link, child left_2f_robotiq_85_left_knuckle_link, origin xyz=0.05490451627 0.03060114443 0.0 rpy=3.141592653589793 0.0 0.0, axis 0 0 1, limit lower=0.0 upper=0.80285 effort=1000 velocity=0.5
- added joint left_2f_robotiq_85_right_finger_joint: type fixed, parent left_2f_robotiq_85_right_knuckle_link, child left_2f_robotiq_85_right_finger_link, origin xyz=-0.00408552455 -0.03148604435 0.0 rpy=0 0 0
- added joint left_2f_robotiq_85_right_finger_tip_joint: type continuous, parent left_2f_robotiq_85_right_inner_knuckle_link, child left_2f_robotiq_85_right_finger_tip_link, origin xyz=0.04303959807 -0.03759940821  0.0 rpy=0.0 0.0 0.0, axis 0 0 1, limit lower=-3.14 upper=3.14 effort=0.1 velocity=100.0, mimic joint=left_2f_robotiq_85_left_knuckle_joint multiplier=-1
- added joint left_2f_robotiq_85_right_inner_knuckle_joint: type continuous, parent left_2f_robotiq_85_base_link, child left_2f_robotiq_85_right_inner_knuckle_link, origin xyz=0.06142 -0.0127 0 rpy=0 0 0, axis 0 0 1, limit lower=-3.14 upper=3.14 effort=0.1 velocity=100.0, mimic joint=left_2f_robotiq_85_left_knuckle_joint offset=0
- added joint left_2f_robotiq_85_right_knuckle_joint: type continuous, parent left_2f_robotiq_85_base_link, child left_2f_robotiq_85_right_knuckle_link, origin xyz=0.05490451627 -0.03060114443 0.0 rpy=0.0 0.0 0.0, axis 0 0 1, limit lower=-3.14 upper=3.14 effort=1000 velocity=100.0, mimic joint=left_2f_robotiq_85_left_knuckle_joint

File: p6_ws/src/lbr_fri/lbr_fri_ros2_stack/lbr_description/urdf/isaac_dual_arm/isaac_dual_arm.xacro (robot description, xacro)
@@ -850,5 +850,5 @@
   </joint>
   <!-- 2F GRIPPER -->
-  <xacro:robotiq_85_gripper prefix="2f_" parent="camera_arm_mount">
+  <xacro:robotiq_85_gripper prefix="left_2f_" parent="camera_arm_mount">
     <origin xyz="0 0 0.012" rpy="0 -1.5707 0"/>
   </xacro:robotiq_85_gripper>
