Commit message: Updated the name of every link in 3f gripper to a_3f. Isaac sim does not like numbers as the first character in names

File: p6_ws/src/lbr_fri/lbr_fri_ros2_stack/lbr_description/urdf/isaac_dual_arm/isaac_dual_arm.urdf (robot description, URDF)
Before this commit: robot isaac_dual_arm, 49 links, 48 joints
Links:
- removed link 3f_finger_1_link_0
- removed link 3f_finger_1_link_1
- removed link 3f_finger_1_link_2
- removed link 3f_finger_1_link_3
- removed link 3f_finger_2_link_0
- removed link 3f_finger_2_link_1
- removed link 3f_finger_2_link_2
- removed link 3f_finger_2_link_3
- removed link 3f_finger_middle_link_0
- removed link 3f_finger_middle_link_1
- removed link 3f_finger_middle_link_2
- removed link 3f_finger_middle_link_3
- removed link 3f_palm
- removed link 3f_tool0
- added link a_3f_finger_1_link_0, mass 0.05; collision mesh filename=package://lbr_description/meshes/robotiq-3f-gripper_articul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; visual mesh filename=package://lbr_description/meshes/robotiq-3f-gripper_articul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
- added link a_3f_finger_1_link_1, mass 0.15; collision mesh filename=package://lbr_description/meshes/robotiq-3f-gripper_articul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; visual mesh filename=package://lbr_description/meshes/robotiq-3f-gripper_articul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
- added link a_3f_finger_1_link_2, mass 0.15; collision mesh filename=package://lbr_description/meshes/robotiq-3f-gripper_articul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; visual mesh filename=package://lbr_description/meshes/robotiq-3f-gripper_articul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
- added link a_3f_finger_1_link_3, mass 0.05; collision mesh filename=package://lbr_description/meshes/robotiq-3f-gripper_articul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; visual mesh filename=package://lbr_description/meshes/robotiq-3f-gripper_articul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
- added link a_3f_finger_2_link_0, mass 0.05; collision mesh filename=package://lbr_description/meshes/robotiq-3f-gripper_articul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; visual mesh filename=package://lbr_description/meshes/robotiq-3f-gripper_articul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
- added link a_3f_finger_2_link_1, mass 0.15; collision mesh filename=package://lbr_description/meshes/robotiq-3f-gripper_articul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; visual mesh filename=package://lbr_description/meshes/robotiq-3f-gripper_articul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
- added link a_3f_finger_2_link_2, mass 0.15; collision mesh filename=package://lbr_description/meshes/robotiq-3f-gripper_articul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; visual mesh filename=package://lbr_description/meshes/robotiq-3f-gripper_articul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
- added link a_3f_finger_2_link_3, mass 0.05; collision mesh filename=package://lbr_description/meshes/robotiq-3f-gripper_articul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; visual mesh filename=package://lbr_description/meshes/robotiq-3f-gripper_articul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
- added link a_3f_finger_middle_link_0, mass 0.05; collision mesh filename=package://lbr_description/meshes/robotiq-3f-gripper_articul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; visual mesh filename=package://lbr_description/meshes/robotiq-3f-gripper_articul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
- added link a_3f_finger_middle_link_1, mass 0.15; collision mesh filename=package://lbr_description/meshes/robotiq-3f-gripper_articul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; visual mesh filename=package://lbr_description/meshes/robotiq-3f-gripper_articul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
- added link a_3f_finger_middle_link_2, mass 0.15; collision mesh filename=package://lbr_description/meshes/robotiq-3f-gripper_articul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; visual mesh filename=package://lbr_description/meshes/robotiq-3f-gripper_articul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
- added link a_3f_finger_middle_link_3, mass 0.05; collision mesh filename=package://lbr_description/meshes/robotiq-3f-gripper_articul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; visual mesh filename=package://lbr_description/meshes/robotiq-3f-gripper_articul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
- added link a_3f_palm; collision mesh filename=package://lbr_description/meshes/robotiq-3f-gripper_articul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; visual mesh filename=package://lbr_description/meshes/robotiq-3f-gripper_articul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
- added link a_3f_tool0
- added link back_wall; collision mesh filename=package://lbr_description/meshes/table/collision/Back_wall.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 scale=0.001 0.001 0.001; visual mesh filename=package://lbr_description/meshes/table/collision/Back_wall.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 scale=0.001 0.001 0.001
- added link left_side_wall; collision mesh filename=package://lbr_description/meshes/table/collision/Side_wall.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 scale=0.001 0.001 0.001
- added link right_side_wall; collision mesh filename=package://lbr_description/meshes/table/collision/Side_wall.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 scale=0.001 0.001 0.001
Joints:
- removed joint 3f_finger_1_joint_1
- removed joint 3f_finger_1_joint_2
- removed joint 3f_finger_1_joint_3
- removed joint 3f_finger_2_joint_1
- removed joint 3f_finger_2_joint_2
- removed joint 3f_finger_2_joint_3
- removed joint 3f_finger_middle_joint_1
- removed joint 3f_finger_middle_joint_2
- removed joint 3f_finger_middle_joint_3
- removed joint 3f_palm_finger_1_joint
- removed joint 3f_palm_finger_2_joint
- removed joint 3f_palm_finger_middle_joint
- removed joint 3f_palm_tool0
- added joint a_3f_finger_1_joint_1: type revolute, parent a_3f_finger_1_link_0, child a_3f_finger_1_link_1, origin xyz=0.020 0 0 rpy=0 0 -0.43, axis 0 0 1, limit lower=0.3758 upper=1.1276 effort=100 velocity=1.23
- added joint a_3f_finger_1_joint_2: type revolute, parent a_3f_finger_1_link_1, child a_3f_finger_1_link_2, origin xyz=0.050 -.028 0 rpy=0 0 -0.52, axis 0 0 1, limit lower=0.0 upper=1.5707 effort=100 velocity=1.24
- added joint a_3f_finger_1_joint_3: type revolute, parent a_3f_finger_1_link_2, child a_3f_finger_1_link_3, origin xyz=0.039 0 0 rpy=0 0 0, axis 0 0 1, limit lower=-0.9531 upper=0.7572 effort=100 velocity=1.25
- added joint a_3f_finger_2_joint_1: type revolute, parent a_3f_finger_2_link_0, child a_3f_finger_2_link_1, origin xyz=0.020 0 0 rpy=0 0 -0.43, axis 0 0 1, limit lower=0.3758 upper=1.1276 effort=100 velocity=1.23
- added joint a_3f_finger_2_joint_2: type revolute, parent a_3f_finger_2_link_1, child a_3f_finger_2_link_2, origin xyz=0.050 -.028 0 rpy=0 0 -0.52, axis 0 0 1, limit lower=0.0 upper=1.5707 effort=100 velocity=1.24
- added joint a_3f_finger_2_joint_3: type revolute, parent a_3f_finger_2_link_2, child a_3f_finger_2_link_3, origin xyz=0.039 0 0 rpy=0 0 0, axis 0 0 1, limit lower=-0.9531 upper=0.7572 effort=100 velocity=1.25
- added joint a_3f_finger_middle_joint_1: type revolute, parent a_3f_finger_middle_link_0, child a_3f_finger_middle_link_1, origin xyz=0.020 0 0 rpy=0 0 -0.43, axis 0 0 1, limit lower=0.3758 upper=1.1276 effort=100 velocity=1.23
- added joint a_3f_finger_middle_joint_2: type revolute, parent a_3f_finger_middle_link_1, child a_3f_finger_middle_link_2, origin xyz=0.050 -.028 0 rpy=0 0 -0.52, axis 0 0 1, limit lower=0.0 upper=1.5707 effort=100 velocity=1.24
- added joint a_3f_finger_middle_joint_3: type revolute, parent a_3f_finger_middle_link_2, child a_3f_finger_middle_link_3, origin xyz=0.039 0 0 rpy=0 0 0, axis 0 0 1, limit lower=-0.9531 upper=0.7572 effort=100 velocity=1.25
- added joint a_3f_palm_finger_1_joint: type revolute, parent a_3f_palm, child a_3f_finger_1_link_0, origin xyz=-0.0455 0.0214 0.036 rpy=0 3.1416 -1.57, axis 0 1 0, limit lower=-0.1784 upper=0.192 effort=100 velocity=1.23
- added joint a_3f_palm_finger_2_joint: type revolute, parent a_3f_palm, child a_3f_finger_2_link_0, origin xyz=-0.0455 0.0214 -0.036 rpy=0 3.1416 -1.57, axis 0 1 0, limit lower=-0.192 upper=0.1784 effort=100 velocity=1.23
- added joint a_3f_palm_finger_middle_joint: type fixed, parent a_3f_palm, child a_3f_finger_middle_link_0, origin xyz=0.0455 0.0214 0 rpy=0 0 1.57, axis 0 0 1
- added joint a_3f_palm_tool0: type fixed, parent a_3f_palm, child a_3f_tool0, origin xyz=0.0 0.15 0 rpy=0 -1.5707 1.5707
- added joint back_wall_joint: type fixed, parent world, child back_wall, origin xyz=0 0 0 rpy=0 0 0
- added joint left_side_wall_joint: type fixed, parent world, child left_side_wall, origin xyz=0 0 0 rpy=0 0 0
- added joint right_side_wall_joint: type fixed, parent world, child right_side_wall, origin xyz=0 0 0 rpy=0 0 0
- joint adapter_mount: child 3f_palm -> a_3f_palm

File: p6_ws/src/lbr_fri/lbr_fri_ros2_stack/lbr_description/urdf/isaac_dual_arm/isaac_dual_arm.xacro (robot description, xacro)
@@ -461,5 +461,5 @@
 	</link>
     <!-- link list -->
-  <link name="3f_finger_1_link_0">
+  <link name="a_3f_finger_1_link_0">
     <visual>
       <origin rpy="0 0 0" xyz="0.020 0 0"/>
@@ -484,5 +484,5 @@
     </inertial>
   </link>
-  <link name="3f_finger_1_link_1">
+  <link name="a_3f_finger_1_link_1">
     <visual>
       <origin rpy="0 0 -0.52" xyz="0.050 -.028 0"/>
@@ -505,5 +505,5 @@
     </inertial>
   </link>
-  <link name="3f_finger_1_link_2">
+  <link name="a_3f_finger_1_link_2">
     <visual>
       <origin rpy="0 0 0" xyz="0.039 0 0.0075"/>
@@ -526,5 +526,5 @@
     </inertial>
   </link>
-  <link name="3f_finger_1_link_3">
+  <link name="a_3f_finger_1_link_3">
     <visual>
       <origin rpy="0 0 0.52" xyz="0 0 0"/>
@@ -549,7 +549,7 @@
   <!-- end of link list -->
   <!-- 3f joint list -->
-  <joint name="3f_finger_1_joint_1" type="revolute">
-    <parent link="3f_finger_1_link_0"/>
-    <child link="3f_finger_1_link_1"/>
+  <joint name="a_3f_finger_1_joint_1" type="revolute">
+    <parent link="a_3f_finger_1_link_0"/>
+    <child link="a_3f_finger_1_link_1"/>
     <axis xyz="0 0 1"/>
     <origin rpy="0 0 -0.43" xyz="0.020 0 0"/>
@@ -557,7 +557,7 @@
     <dynamics damping="1" friction="0.1"/>
   </joint>
-  <joint name="3f_finger_1_joint_2" type="revolute">
-    <parent link="3f_finger_1_link_1"/>
-    <child link="3f_finger_1_link_2"/>
+  <joint name="a_3f_finger_1_joint_2" type="revolute">
+    <parent link="a_3f_finger_1_link_1"/>
+    <child link="a_3f_finger_1_link_2"/>
     <axis xyz="0 0 1"/>
     <origin rpy="0 0 -0.52" xyz="0.050 -.028 0"/>
@@ -565,7 +565,7 @@
     <dynamics damping="1" friction="0.1"/>
   </joint>
-  <joint name="3f_finger_1_joint_3" type="revolute">
-    <parent link="3f_finger_1_link_2"/>
-    <child link="3f_finger_1_link_3"/>
+  <joint name="a_3f_finger_1_joint_3" type="revolute">
+    <parent link="a_3f_finger_1_link_2"/>
+    <child link="a_3f_finger_1_link_3"/>
     <axis xyz="0 0 1"/>
     <origin rpy="0 0 0" xyz="0.039 0 0"/>
@@ -575,5 +575,5 @@
   <!-- end of joint list -->
   <!-- link list -->
-  <link name="3f_finger_2_link_0">
+  <link name="a_3f_finger_2_link_0">
     <visual>
       <origin rpy="0 0 0" xyz="0.020 0 0"/>
@@ -598,5 +598,5 @@
     </inertial>
   </link>
-  <link name="3f_finger_2_link_1">
+  <link name="a_3f_finger_2_link_1">
     <visual>
       <origin rpy="0 0 -0.52" xyz="0.050 -.028 0"/>
@@ -619,5 +619,5 @@
     </inertial>
   </link>
-  <link name="3f_finger_2_link_2">
+  <link name="a_3f_finger_2_link_2">
     <visual>
       <origin rpy="0 0 0" xyz="0.039 0 0.0075"/>
@@ -640,5 +640,5 @@
     </inertial>
   </link>
-  <link name="3f_finger_2_link_3">
+  <link name="a_3f_finger_2_link_3">
     <visual>
       <origin rpy="0 0 0.52" xyz="0 0 0"/>
@@ -663,7 +663,7 @@
   <!-- end of link list -->
   <!-- joint list -->
-  <joint name="3f_finger_2_joint_1" type="revolute">
-    <parent link="3f_finger_2_link_0"/>
-    <child link="3f_finger_2_link_1"/>
+  <joint name="a_3f_finger_2_joint_1" type="revolute">
+    <parent link="a_3f_finger_2_link_0"/>
+    <child link="a_3f_finger_2_link_1"/>
     <axis xyz="0 0 1"/>
     <origin rpy="0 0 -0.43" xyz="0.020 0 0"/>
@@ -671,7 +671,7 @@
     <dynamics damping="1" friction="0.1"/>
   </joint>
-  <joint name="3f_finger_2_joint_2" type="revolute">
-    <parent link="3f_finger_2_link_1"/>
-    <child link="3f_finger_2_link_2"/>
+  <joint name="a_3f_finger_2_joint_2" type="revolute">
+    <parent link="a_3f_finger_2_link_1"/>
+    <child link="a_3f_finger_2_link_2"/>
     <axis xyz="0 0 1"/>
     <origin rpy="0 0 -0.52" xyz="0.050 -.028 0"/>
@@ -679,7 +679,7 @@
     <dynamics damping="1" friction="0.1"/>
   </joint>
-  <joint name="3f_finger_2_joint_3" type="revolute">
-    <parent link="3f_finger_2_link_2"/>
-    <child link="3f_finger_2_link_3"/>
+  <joint name="a_3f_finger_2_joint_3" type="revolute">
+    <parent link="a_3f_finger_2_link_2"/>
+    <child link="a_3f_finger_2_link_3"/>
     <axis xyz="0 0 1"/>
     <origin rpy="0 0 0" xyz="0.039 0 0"/>
@@ -689,5 +689,5 @@
   <!-- end of joint list -->
   <!-- link list -->
-  <link name="3f_finger_middle_link_0">
+  <link name="a_3f_finger_middle_link_0">
     <visual>
       <origin rpy="0 0 0" xyz="0.020 0 0"/>
@@ -712,5 +712,5 @@
     </inertial>
   </link>
-  <link name="3f_finger_middle_link_1">
+  <link name="a_3f_finger_middle_link_1">
     <visual>
       <origin rpy="0 0 -0.52" xyz="0.050 -.028 0"/>
@@ -733,5 +733,5 @@
     </inertial>
   </link>
-  <link name="3f_finger_middle_link_2">
+  <link name="a_3f_finger_middle_link_2">
     <visual>
       <origin rpy="0 0 0" xyz="0.039 0 0.0075"/>
@@ -754,5 +754,5 @@
     </inertial>
   </link>
-  <link name="3f_finger_middle_link_3">
+  <link name="a_3f_finger_middle_link_3">
     <visual>
       <origin rpy="0 0 0.52" xyz="0 0 0"/>
@@ -777,7 +777,7 @@
   <!-- end of link list -->
   <!-- joint list -->
-  <joint name="3f_finger_middle_joint_1" type="revolute">
-    <parent link="3f_finger_middle_link_0"/>
-    <child link="3f_finger_middle_link_1"/>
+  <joint name="a_3f_finger_middle_joint_1" type="revolute">
+    <parent link="a_3f_finger_middle_link_0"/>
+    <child link="a_3f_finger_middle_link_1"/>
     <axis xyz="0 0 1"/>
     <origin rpy="0 0 -0.43" xyz="0.020 0 0"/>
@@ -785,7 +785,7 @@
     <dynamics damping="1" friction="0.1"/>
   </joint>
-  <joint name="3f_finger_middle_joint_2" type="revolute">
-    <parent link="3f_finger_middle_link_1"/>
-    <child link="3f_finger_middle_link_2"/>
+  <joint name="a_3f_finger_middle_joint_2" type="revolute">
+    <parent link="a_3f_finger_middle_link_1"/>
+    <child link="a_3f_finger_middle_link_2"/>
     <axis xyz="0 0 1"/>
     <origin rpy="0 0 -0.52" xyz="0.050 -.028 0"/>
@@ -793,7 +793,7 @@
     <dynamics damping="1" friction="0.1"/>
   </joint>
-  <joint name="3f_finger_middle_joint_3" type="revolute">
-    <parent link="3f_finger_middle_link_2"/>
-    <child link="3f_finger_middle_link_3"/>
+  <joint name="a_3f_finger_middle_joint_3" type="revolute">
+    <parent link="a_3f_finger_middle_link_2"/>
+    <child link="a_3f_finger_middle_link_3"/>
     <axis xyz="0 0 1"/>
     <origin rpy="0 0 0" xyz="0.039 0 0"/>
@@ -803,5 +803,5 @@
   <!-- end of joint list -->
   <!-- link list -->
-  <link name="3f_palm">
+  <link name="a_3f_palm">
     <visual>
       <geometry>
@@ -819,5 +819,5 @@
     </collision>
   </link>
-  <link name="3f_tool0"/>
+  <link name="a_3f_tool0"/>
   <inertial>
     <origin rpy="0 0 0" xyz="0 0 0"/>
@@ -827,7 +827,7 @@
   <!-- end of link list -->
   <!-- joint list -->
-  <joint name="3f_palm_finger_1_joint" type="revolute">
-    <parent link="3f_palm"/>
-    <child link="3f_finger_1_link_0"/>
+  <joint name="a_3f_palm_finger_1_joint" type="revolute">
+    <parent link="a_3f_palm"/>
+    <child link="a_3f_finger_1_link_0"/>
     <axis xyz="0 1 0"/>
     <origin rpy="0 3.1416 -1.57" xyz="-0.0455 0.0214 0.036"/>
@@ -835,7 +835,7 @@
     <dynamics damping="1.0" friction="0.1"/>
   </joint>
-  <joint name="3f_palm_finger_2_joint" type="revolute">
-    <parent link="3f_palm"/>
-    <child link="3f_finger_2_link_0"/>
+  <joint name="a_3f_palm_finger_2_joint" type="revolute">
+    <parent link="a_3f_palm"/>
+    <child link="a_3f_finger_2_link_0"/>
     <axis xyz="0 1 0"/>
     <origin rpy="0 3.1416 -1.57" xyz="-0.0455 0.0214 -0.036"/>
@@ -843,7 +843,7 @@
     <dynamics damping="1.0" friction="0.1"/>
   </joint>
-  <joint name="3f_palm_finger_middle_joint" type="fixed">
-    <parent link="3f_palm"/>
-    <child link="3f_finger_middle_link_0"/>
+  <joint name="a_3f_palm_finger_middle_joint" type="fixed">
+    <parent link="a_3f_palm"/>
+    <child link="a_3f_finger_middle_link_0"/>
     <axis xyz="0 0 1"/>
     <origin rpy="0 0 1.57" xyz="0.0455 0.0214 0"/>
@@ -1016,11 +1016,11 @@
   <joint name="adapter_mount" type="fixed">
 	  <parent link="gripper_mounting_plate" />
-	  <child link="3f_palm" />
+	  <child link="a_3f_palm" />
 	  <origin xyz="0 0 0.0745" rpy="1.57079633 0 -1.57079633"/>
   </joint>
   <!-- joint between 3f gripper and 3f tool0-->
-  <joint name="3f_palm_tool0" type="fixed">
-    <parent link="3f_palm"/>
-    <child link="3f_tool0"/>
+  <joint name="a_3f_palm_tool0" type="fixed">
+    <parent link="a_3f_palm"/>
+    <child link="a_3f_tool0"/>
     <origin rpy="0 -1.5707 1.5707" xyz="0.0 0.15 0"/>
   </joint>

File: p6_ws/src/lbr_fri/lbr_fri_ros2_stack/lbr_moveit_config/isaac_dual_arm_moveit_config/config/isaac_dual_arm.ros2_control.xacro (robot description, xacro)
@@ -191,5 +191,5 @@
     </joint>
     <!-- Setup of Hardware for 2F Gripper -->
-    <joint name="2f_robotiq_85_left_knuckle_joint">
+    <joint name="left_2f_robotiq_85_left_knuckle_joint">
       <param name="max_velocity">2</param>
       <command_interface name="position">
@@ -204,11 +204,6 @@
       </state_interface>
     </joint>
-    </ros2_control>
-   <!--Setup of Hardware for 3F Gripper -->
-  <ros2_control name="3FGripper" type="system">
-    <hardware>
-      <plugin>mock_components/GenericSystem</plugin>
-    </hardware>
-    <joint name="3f_finger_1_joint_1">
+    <!-- Hardware setup fpr 3f gripper -->
+    <joint name="a_3f_finger_1_joint_1">
       <param name="max_velocity">1.23</param>
       <command_interface name="position">
@@ -223,5 +218,5 @@
       </state_interface>
     </joint>
-    <joint name="3f_finger_1_joint_2">
+    <joint name="a_3f_finger_1_joint_2">
       <param name="max_velocity">1.24</param>
       <command_interface name="position">
@@ -236,5 +231,5 @@
       </state_interface>
     </joint>
-    <joint name="3f_finger_1_joint_3">
+    <joint name="a_3f_finger_1_joint_3">
       <param name="max_velocity">1.25</param>
       <command_interface name="position">
@@ -249,5 +244,5 @@
       </state_interface>
     </joint>
-    <joint name="3f_finger_2_joint_1">
+    <joint name="a_3f_finger_2_joint_1">
       <param name="max_velocity">1.23</param>
       <command_interface name="position">
@@ -262,5 +257,5 @@
       </state_interface>
     </joint>
-    <joint name="3f_finger_2_joint_2">
+    <joint name="a_3f_finger_2_joint_2">
       <param name="max_velocity">1.24</param>
       <command_interface name="position">
@@ -275,5 +270,5 @@
       </state_interface>
     </joint>
-    <joint name="3f_finger_2_joint_3">
+    <joint name="a_3f_finger_2_joint_3">
       <param name="max_velocity">1.25</param>
       <command_interface name="position">
@@ -288,5 +283,5 @@
       </state_interface>
     </joint>
-    <joint name="3f_finger_middle_joint_1">
+    <joint name="a_3f_finger_middle_joint_1">
       <param name="max_velocity">1.23</param>
       <command_interface name="position">
@@ -301,5 +296,5 @@
       </state_interface>
     </joint>
-    <joint name="3f_finger_middle_joint_2">
+    <joint name="a_3f_finger_middle_joint_2">
       <param name="max_velocity">1.24</param>
       <command_interface name="position">
@@ -314,5 +309,5 @@
       </state_interface>
     </joint>
-    <joint name="3f_finger_middle_joint_3">
+    <joint name="a_3f_finger_middle_joint_3">
       <param name="max_velocity">1.25</param>
       <command_interface name="position">
@@ -327,5 +322,5 @@
       </state_interface>
     </joint>
-    <joint name="3f_palm_finger_1_joint">
+    <joint name="a_3f_palm_finger_1_joint">
       <param name="max_velocity">1.23</param>
       <command_interface name="position">
@@ -340,5 +335,5 @@
       </state_interface>
     </joint>
-    <joint name="3f_palm_finger_2_joint">
+    <joint name="a_3f_palm_finger_2_joint">
       <param name="max_velocity">1.23</param>
       <command_interface name="position">

Commit message: Both arms and gripeprs are now working in isaacsim!

File: p6_ws/src/lbr_fri/lbr_fri_ros2_stack/lbr_description/urdf/isaac_dual_arm/isaac_dual_arm.urdf (robot description, URDF)
Before this commit: robot isaac_dual_arm, 52 links, 51 joints
Links:
- removed link back_wall
- removed link left_side_wall
- removed link right_side_wall
Joints:
- removed joint back_wall_joint
- removed joint left_side_wall_joint
- removed joint right_side_wall_joint

Commit message: Finished the mock controllers for the grippers in dual_arm_moveit_config

File: p6_ws/src/lbr_fri/lbr_fri_ros2_stack/lbr_description/urdf/isaac_dual_arm/isaac_dual_arm.urdf (robot description, URDF)
Before this commit: robot isaac_dual_arm, 49 links, 48 joints
Links:
- added link back_wall; collision mesh filename=package://lbr_description/meshes/table/collision/Back_wall.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 scale=0.001 0.001 0.001; visual mesh filename=package://lbr_description/meshes/table/collision/Back_wall.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 scale=0.001 0.001 0.001
- added link left_side_wall; collision mesh filename=package://lbr_description/meshes/table/collision/Side_wall.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 scale=0.001 0.001 0.001
- added link right_side_wall; collision mesh filename=package://lbr_description/meshes/table/collision/Side_wall.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 scale=0.001 0.001 0.001
Joints:
- added joint back_wall_joint: type fixed, parent world, child back_wall, origin xyz=0 0 0 rpy=0 0 0
- added joint left_side_wall_joint: type fixed, parent world, child left_side_wall, origin xyz=0 0 0 rpy=0 0 0
- added joint right_side_wall_joint: type fixed, parent world, child right_side_wall, origin xyz=0 0 0 rpy=0 0 0

File: p6_ws/src/lbr_fri/lbr_fri_ros2_stack/lbr_moveit_config/dual_arm_moveit_config/config/dual_arm.ros2_control.xacro (robot description, xacro)
@@ -358,4 +358,10 @@
       </state_interface>
     </joint>
+  </ros2_control>
+  <!-- Setup of Hardware for 2F Gripper -->
+  <ros2_control name="2FGripper" type="system">
+    <hardware>
+      <plugin>mock_components/GenericSystem</plugin>
+    </hardware>
   <!-- Setup of Hardware for 2F Gripper -->
     <joint name="left_2f_robotiq_85_left_knuckle_joint">
