Commit message: Added a simple camera location to RViz alongside a client/service package that can take images of the simulation window and pass them to a client

File: p6_ws/src/lbr_fri/lbr_fri_ros2_stack/lbr_description/urdf/dual_arm/dual_arm.urdf (robot description, URDF)
Before this commit: robot mock_dual_arm, 48 links, 47 joints
Links:
- removed link camera_link_sky
Joints:
- removed joint cam_table
- joint 3f_finger_1_joint_1: limit lower=0.3758 upper=1.1276 effort=100 velocity=1.23 -> lower=0.0495 upper=1.2218 effort=100 velocity=1.23
- joint 3f_finger_1_joint_2: limit lower=0.0 upper=1.5707 effort=100 velocity=1.24 -> lower=0.0 upper=1.5708 effort=100 velocity=1.24
- joint 3f_finger_1_joint_3: limit lower=-0.9531 upper=0.7572 effort=100 velocity=1.25 -> lower=-1.2217 upper=-0.0523 effort=100 velocity=1.25
- joint 3f_finger_2_joint_1: limit lower=0.3758 upper=1.1276 effort=100 velocity=1.23 -> lower=0.0495 upper=1.2218 effort=100 velocity=1.23
- joint 3f_finger_2_joint_2: limit lower=0.0 upper=1.5707 effort=100 velocity=1.24 -> lower=0.0 upper=1.5708 effort=100 velocity=1.24
- joint 3f_finger_2_joint_3: limit lower=-0.9531 upper=0.7572 effort=100 velocity=1.25 -> lower=-1.2217 upper=-0.0523 effort=100 velocity=1.25
- joint 3f_finger_middle_joint_1: limit lower=0.3758 upper=1.1276 effort=100 velocity=1.23 -> lower=0.0495 upper=1.2218 effort=100 velocity=1.23
- joint 3f_finger_middle_joint_2: limit lower=0.0 upper=1.5707 effort=100 velocity=1.24 -> lower=0.0 upper=1.5708 effort=100 velocity=1.24
- joint 3f_finger_middle_joint_3: limit lower=-0.9531 upper=0.7572 effort=100 velocity=1.25 -> lower=-1.2217 upper=-0.0523 effort=100 velocity=1.25
- joint left_finger_joint: limit lower=0 upper=0.8757 effort=1000 velocity=2.0 -> lower=0 upper=0.8 effort=1000 velocity=2.0
- joint left_left_inner_finger_joint: limit lower=-0.8757 upper=0 effort=1000 velocity=2.0 -> lower=0 upper=0.8757 effort=1000 velocity=2.0
- joint left_right_inner_finger_joint: limit lower=-0.8757 upper=0 effort=1000 velocity=2.0 -> lower=0 upper=0.8757 effort=1000 velocity=2.0
- joint left_right_outer_knuckle_joint: limit lower=0 upper=0.8757 effort=1000 velocity=2.0 -> lower=0 upper=0.81 effort=1000 velocity=2.0
- joint mount_left: parent table -> world

File: p6_ws/src/lbr_fri/lbr_fri_ros2_stack/lbr_description/urdf/dual_arm/dual_arm.xacro (robot description, xacro)
@@ -1630,5 +1630,5 @@
     </collision>
   </link>
-  <!-- the wooden laser cut camera mount-->
+  <!-- the wooden laser cut camera mount
   <link name="cam_mount">
     <visual>
@@ -1640,4 +1640,5 @@
     </visual>
   </link>
+  -->
   <!-- 3f gripper adapter / mounting plate -->
   <link name="gripper_mounting_plate">
@@ -1661,5 +1662,5 @@
     <child link="table"/>
   </joint>
-  <!--joint between table and wooden camera mount-->
+  <!--joint between table and wooden camera mount
   <joint name="cam_table_joint" type="fixed">
     <parent link="table"/>
@@ -1667,9 +1668,10 @@
     <origin rpy="1.57079633 0 0" xyz="0.489819 0.84691 1.428"/>
   </joint>
+  -->
   <!--joint between table and right iiwa7 -->
   <joint name="mount_right" type="fixed">
     <parent link="table"/>
     <child link="right_link_0"/>
-    <origin rpy="0.785398163 0 -1.57079633" xyz="0.268524 0.756691 1.037203"/>
+    <origin rpy="0 0 -0.785398163" xyz="0.145181 0.79431 0.815"/>
   </joint>
   <!-- joint between right iiwa7 and 3f gripper-->
@@ -1685,9 +1687,9 @@
         <origin xyz="0 0 0.0745" rpy="1.57079633 0 -1.57079633"/>
     </joint>
-  <!-- joint between left arm and world -->
+  <!-- joint between left arm and table -->
   <joint name="mount_left" type="fixed">
-    <parent link="world"/>
+    <parent link="table"/>
     <child link="left_link_0"/>
-    <origin rpy="-0.785398163 0 -1.57079633" xyz="0.711114 0.756691 1.037203"/>
+    <origin rpy="0 0 -2.35619449 " xyz="0.795181 0.79431 0.815"/>
   </joint>
   <!-- joint between left iiwa7 and 2f gripper-->

File: p6_ws/src/lbr_fri/lbr_fri_ros2_stack/lbr_description/urdf/isaac_dual_arm/isaac_dual_arm.xacro (robot description, xacro)
@@ -5,5 +5,7 @@
   <ros2_control name="lbr_system_interface_right" type="system">
     <hardware>
-      <plugin>mock_components/GenericSystem</plugin>
+      <plugin>topic_based_ros2_control/TopicBasedSystem</plugin>
+      <param name="joint_commands_topic">/right_arm/isaac_joint_commands</param>
+      <param name="joint_state_topic">/right_arm/isaac_joint_states</param>
     </hardware>
     <joint name="right_A1">
@@ -102,5 +104,7 @@
   <ros2_control name="lbr_system_interface_left" type="system">
     <hardware>
-      <plugin>mock_components/GenericSystem</plugin>
+      <plugin>topic_based_ros2_control/TopicBasedSystem</plugin>
+      <param name="joint_commands_topic">/left_arm/isaac_joint_commands</param>
+      <param name="joint_state_topic">/left_arm/isaac_joint_states</param>
     </hardware>
     <joint name="left_A1">
@@ -794,6 +798,6 @@
     <origin rpy="0 0 0" xyz="0 0 0.035"/>
   </joint>
-  <link name="left_link_ee"/>
-  <link name="camera_link_sky"/>
+  <link name="left_link_ee">
+	</link>
     <!-- link list -->
   <link name="3f_finger_1_link_0">
@@ -1644,9 +1648,3 @@
     <origin rpy="0 3.14 0" xyz="0 0 0.165"/>
   </joint>
-  <!-- joint between left arm ee and camera-->
-  <joint name="cam_table" type="fixed">
-    <parent link="table"/>
-    <child link="camera_link_sky"/>
-    <origin rpy="0 0 0" xyz="0.5 0.5 2.2"/>
-  </joint>
 </robot>

Commit message: Updated dual_arm.urdf

File: p6_ws/src/lbr_fri/lbr_fri_ros2_stack/lbr_description/urdf/dual_arm/dual_arm.urdf (robot description, URDF)
Before this commit: robot dual_arm, 47 links, 46 joints
Links:
- removed link 3f_finger_1_link_0
- removed link 3f_finger_1_link_1
- removed link 3f_finger_1_link_2
- removed link 3f_finger_1_link_3
- removed link 3f_finger_2_link_0
- removed link 3f_finger_2_link_1
- removed link 3f_finger_2_link_2
- removed link 3f_finger_2_link_3
- removed link 3f_finger_middle_link_0
- removed link 3f_finger_middle_link_1
- removed link 3f_finger_middle_link_2
- removed link 3f_finger_middle_link_3
- removed link 3f_palm
- removed link 3f_tool0
- removed link left_left_inner_finger
- removed link left_left_inner_finger_pad
- removed link left_left_inner_knuckle
- removed link left_left_outer_finger
- removed link left_left_outer_knuckle
- removed link left_right_inner_finger
- removed link left_right_inner_finger_pad
- removed link left_right_inner_knuckle
- removed link left_right_outer_finger
- removed link left_right_outer_knuckle
- removed link left_robotiq_arg2f_base_link
- removed link table
- added link a_3f_finger_1_link_0, mass 0.05; collision mesh filename=package://lbr_description/meshes/robotiq-3f-gripper_articul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; visual mesh filename=package://lbr_description/meshes/robotiq-3f-gripper_articul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
- added link a_3f_finger_1_link_1, mass 0.15; collision mesh filename=package://lbr_description/meshes/robotiq-3f-gripper_articul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; visual mesh filename=package://lbr_description/meshes/robotiq-3f-gripper_articul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
- added link a_3f_finger_1_link_2, mass 0.15; collision mesh filename=package://lbr_description/meshes/robotiq-3f-gripper_articul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; visual mesh filename=package://lbr_description/meshes/robotiq-3f-gripper_articul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
- added link a_3f_finger_1_link_3, mass 0.05; collision mesh filename=package://lbr_description/meshes/robotiq-3f-gripper_articul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; visual mesh filename=package://lbr_description/meshes/robotiq-3f-gripper_articul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
- added link a_3f_finger_2_link_0, mass 0.05; collision mesh filename=package://lbr_description/meshes/robotiq-3f-gripper_articul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; visual mesh filename=package://lbr_description/meshes/robotiq-3f-gripper_articul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
- added link a_3f_finger_2_link_1, mass 0.15; collision mesh filename=package://lbr_description/meshes/robotiq-3f-gripper_articul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; visual mesh filename=package://lbr_description/meshes/robotiq-3f-gripper_articul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
- added link a_3f_finger_2_link_2, mass 0.15; collision mesh filename=package://lbr_description/meshes/robotiq-3f-gripper_articul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; visual mesh filename=package://lbr_description/meshes/robotiq-3f-gripper_articul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
- added link a_3f_finger_2_link_3, mass 0.05; collision mesh filename=package://lbr_description/meshes/robotiq-3f-gripper_articul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; visual mesh filename=package://lbr_description/meshes/robotiq-3f-gripper_articul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
- added link a_3f_finger_middle_link_0, mass 0.05; collision mesh filename=package://lbr_description/meshes/robotiq-3f-gripper_articul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; visual mesh filename=package://lbr_description/meshes/robotiq-3f-gripper_articul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
- added link a_3f_finger_middle_link_1, mass 0.15; collision mesh filename=package://lbr_description/meshes/robotiq-3f-gripper_articul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; visual mesh filename=package://lbr_description/meshes/robotiq-3f-gripper_articul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
- added link a_3f_finger_middle_link_2, mass 0.15; collision mesh filename=package://lbr_description/meshes/robotiq-3f-gripper_articul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; visual mesh filename=package://lbr_description/meshes/robotiq-3f-gripper_articul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
- added link a_3f_finger_middle_link_3, mass 0.05; collision mesh filename=package://lbr_description/meshes/robotiq-3f-gripper_articul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; visual mesh filename=package://lbr_description/meshes/robotiq-3f-gripper_articul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
- added link a_3f_palm; collision mesh filename=package://lbr_description/meshes/robotiq-3f-gripper_articul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; visual mesh filename=package://lbr_description/meshes/robotiq-3f-gripper_articul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
- added link a_3f_tool0
- added link back_wall; collision mesh filename=package://lbr_description/meshes/table/collision/Back_wall.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 scale=0.001 0.001 0.001; visual mesh filename=package://lbr_description/meshes/table/collision/Back_wall.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 scale=0.001 0.001 0.001
- added link camera_arm_mount; collision mesh filename=package://lbr_description/meshes/camera_arm_mount/Mount_rea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 scale=0.001 0.001 0.001; visual mesh filename=package://lbr_description/meshes/camera_arm_mount/Mount_rea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 scale=0.001 0.001 0.001
- added link left_2f_robotiq_85_base_link, mass 0.636951; collision mesh filename=package://lbr_description/meshes/robotiq_2f_85_gripper/coll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; visual mesh filename=package://lbr_description/meshes/robotiq_2f_85_gripper/visu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
- added link left_2f_robotiq_85_left_finger_link, mass 0.027309; collision mesh filename=package://lbr_description/meshes/robotiq_2f_85_gripper/coll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; visual mesh filename=package://lbr_description/meshes/robotiq_2f_85_gripper/visu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
- added link left_2f_robotiq_85_left_finger_tip_link, mass 0.019555; collision mesh filename=package://lbr_description/meshes/robotiq_2f_85_gripper/coll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; visual mesh filename=package://lbr_description/meshes/robotiq_2f_85_gripper/visu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
- added link left_2f_robotiq_85_left_inner_knuckle_link, mass 0.029951; collision mesh filename=package://lbr_description/meshes/robotiq_2f_85_gripper/coll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; visual mesh filename=package://lbr_description/meshes/robotiq_2f_85_gripper/visu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
- added link left_2f_robotiq_85_left_knuckle_link, mass 0.018491; collision mesh filename=package://lbr_description/meshes/robotiq_2f_85_gripper/coll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; visual mesh filename=package://lbr_description/meshes/robotiq_2f_85_gripper/visu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
- added link left_2f_robotiq_85_right_finger_link, mass 0.027309; collision mesh filename=package://lbr_description/meshes/robotiq_2f_85_gripper/coll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; visual mesh filename=package://lbr_description/meshes/robotiq_2f_85_gripper/visu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
- added link left_2f_robotiq_85_right_finger_tip_link, mass 0.019555; collision mesh filename=package://lbr_description/meshes/robotiq_2f_85_gripper/coll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; visual mesh filename=package://lbr_description/meshes/robotiq_2f_85_gripper/visu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
- added link left_2f_robotiq_85_right_inner_knuckle_link, mass 0.029951; collision mesh filename=package://lbr_description/meshes/robotiq_2f_85_gripper/coll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; visual mesh filename=package://lbr_description/meshes/robotiq_2f_85_gripper/visu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
- added link left_2f_robotiq_85_right_knuckle_link, mass 0.018491; collision mesh filename=package://lbr_description/meshes/robotiq_2f_85_gripper/coll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; visual mesh filename=package://lbr_description/meshes/robotiq_2f_85_gripper/visu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
- added link left_box; collision mesh filename=package://lbr_description/meshes/table/collision/Side_box.s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 scale=0.001 0.001 0.001
- added link left_side_wall; collision mesh filename=package://lbr_description/meshes/table/collision/Side_wall.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 scale=0.001 0.001 0.001
- added link right_box; collision mesh filename=package://lbr_description/meshes/table/collision/Side_box.s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 scale=0.001 0.001 0.001
- added link right_side_wall; collision mesh filename=package://lbr_description/meshes/table/collision/Side_wall.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 scale=0.001 0.001 0.001
- added link table_top, mass 1382.7919279449686; collision mesh filename=package://lbr_description/meshes/table/collision/Table_top.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 scale=0.001 0.001 0.001; visual mesh filename=package://lbr_description/meshes/table/visual/Table_top.stl scale=0.001 0.001 0.001
- added link wooden_top; visual mesh filename=package://lbr_description/meshes/table/visual/Wooden_top.stl scale=0.001 0.001 0.001
Joints:
- removed joint 3f_finger_1_joint_1
- removed joint 3f_finger_1_joint_2
- removed joint 3f_finger_1_joint_3
- removed joint 3f_finger_2_joint_1
- removed joint 3f_finger_2_joint_2
- removed joint 3f_finger_2_joint_3
- removed joint 3f_finger_middle_joint_1
- removed joint 3f_finger_middle_joint_2
- removed joint 3f_finger_middle_joint_3
- removed joint 3f_palm_finger_1_joint
- removed joint 3f_palm_finger_2_joint
- removed joint 3f_palm_finger_middle_joint
- removed joint 3f_palm_tool0
- removed joint left_ee_mount
- removed joint left_finger_joint
- removed joint left_left_inner_finger_joint
- removed joint left_left_inner_finger_pad_joint
- removed joint left_left_inner_knuckle_joint
- removed joint left_left_outer_finger_joint
- removed joint left_right_inner_finger_joint
- removed joint left_right_inner_finger_pad_joint
- removed joint left_right_inner_knuckle_joint
- removed joint left_right_outer_finger_joint
- removed joint left_right_outer_knuckle_joint
- added joint a_3f_finger_1_joint_1: type revolute, parent a_3f_finger_1_link_0, child a_3f_finger_1_link_1, origin xyz=0.020 0 0 rpy=0 0 -0.43, axis 0 0 1, limit lower=0.3758 upper=1.1276 effort=100 velocity=1.23
- added joint a_3f_finger_1_joint_2: type revolute, parent a_3f_finger_1_link_1, child a_3f_finger_1_link_2, origin xyz=0.050 -.028 0 rpy=0 0 -0.52, axis 0 0 1, limit lower=0.0 upper=1.5707 effort=100 velocity=1.24
- added joint a_3f_finger_1_joint_3: type revolute, parent a_3f_finger_1_link_2, child a_3f_finger_1_link_3, origin xyz=0.039 0 0 rpy=0 0 0, axis 0 0 1, limit lower=-0.9531 upper=0.7572 effort=100 velocity=1.25
- added joint a_3f_finger_2_joint_1: type revolute, parent a_3f_finger_2_link_0, child a_3f_finger_2_link_1, origin xyz=0.020 0 0 rpy=0 0 -0.43, axis 0 0 1, limit lower=0.3758 upper=1.1276 effort=100 velocity=1.23
- added joint a_3f_finger_2_joint_2: type revolute, parent a_3f_finger_2_link_1, child a_3f_finger_2_link_2, origin xyz=0.050 -.028 0 rpy=0 0 -0.52, axis 0 0 1, limit lower=0.0 upper=1.5707 effort=100 velocity=1.24
- added joint a_3f_finger_2_joint_3: type revolute, parent a_3f_finger_2_link_2, child a_3f_finger_2_link_3, origin xyz=0.039 0 0 rpy=0 0 0, axis 0 0 1, limit lower=-0.9531 upper=0.7572 effort=100 velocity=1.25
- added joint a_3f_finger_middle_joint_1: type revolute, parent a_3f_finger_middle_link_0, child a_3f_finger_middle_link_1, origin xyz=0.020 0 0 rpy=0 0 -0.43, axis 0 0 1, limit lower=0.3758 upper=1.1276 effort=100 velocity=1.23
- added joint a_3f_finger_middle_joint_2: type revolute, parent a_3f_finger_middle_link_1, child a_3f_finger_middle_link_2, origin xyz=0.050 -.028 0 rpy=0 0 -0.52, axis 0 0 1, limit lower=0.0 upper=1.5707 effort=100 velocity=1.24
- added joint a_3f_finger_middle_joint_3: type revolute, parent a_3f_finger_middle_link_2, child a_3f_finger_middle_link_3, origin xyz=0.039 0 0 rpy=0 0 0, axis 0 0 1, limit lower=-0.9531 upper=0.7572 effort=100 velocity=1.25
- added joint a_3f_palm_finger_1_joint: type revolute, parent a_3f_palm, child a_3f_finger_1_link_0, origin xyz=-0.0455 0.0214 0.036 rpy=0 3.1416 -1.57, axis 0 1 0, limit lower=-0.1784 upper=0.192 effort=100 velocity=1.23
- added joint a_3f_palm_finger_2_joint: type revolute, parent a_3f_palm, child a_3f_finger_2_link_0, origin xyz=-0.0455 0.0214 -0.036 rpy=0 3.1416 -1.57, axis 0 1 0, limit lower=-0.192 upper=0.1784 effort=100 velocity=1.23
- added joint a_3f_palm_finger_middle_joint: type fixed, parent a_3f_palm, child a_3f_finger_middle_link_0, origin xyz=0.0455 0.0214 0 rpy=0 0 1.57, axis 0 0 1
- added joint a_3f_palm_tool0: type fixed, parent a_3f_palm, child a_3f_tool0, origin xyz=0.0 0.15 0 rpy=0 -1.5707 1.5707
- added joint back_wall_joint: type fixed, parent world, child back_wall, origin xyz=0 0 0 rpy=0 0 0
- added joint left_2f_robotiq_85_base_joint: type fixed, parent camera_arm_mount, child left_2f_robotiq_85_base_link, origin xyz=0 0 0.012 rpy=0 -1.5707 0
- added joint left_2f_robotiq_85_left_finger_joint: type fixed, parent left_2f_robotiq_85_left_knuckle_link, child left_2f_robotiq_85_left_finger_link, origin xyz=-0.00408552455 -0.03148604435 0.0 rpy=0 0 0
- added joint left_2f_robotiq_85_left_finger_tip_joint: type continuous, parent left_2f_robotiq_85_left_inner_knuckle_link, child left_2f_robotiq_85_left_finger_tip_link, origin xyz=0.04303959807 -0.03759940821 0.0 rpy=0.0 0.0 0.0, axis 0 0 1, limit lower=-3.14 upper=3.14 effort=0.1 velocity=100.0, mimic joint=left_2f_robotiq_85_left_knuckle_joint multiplier=-1
- added joint left_2f_robotiq_85_left_inner_knuckle_joint: type continuous, parent left_2f_robotiq_85_base_link, child left_2f_robotiq_85_left_inner_knuckle_link, origin xyz=0.06142 0.0127 0 rpy=3.141592653589793 0.0 0.0, axis 0 0 1, limit lower=-3.14 upper=3.14 effort=0.1 velocity=100.0, mimic joint=left_2f_robotiq_85_left_knuckle_joint offset=0
- added joint left_2f_robotiq_85_left_knuckle_joint: type revolute, parent left_2f_robotiq_85_base_link, child left_2f_robotiq_85_left_knuckle_link, origin xyz=0.05490451627 0.03060114443 0.0 rpy=3.141592653589793 0.0 0.0, axis 0 0 1, limit lower=0.0 upper=0.80285 effort=1000 velocity=0.5
- added joint left_2f_robotiq_85_right_finger_joint: type fixed, parent left_2f_robotiq_85_right_knuckle_link, child left_2f_robotiq_85_right_finger_link, origin xyz=-0.00408552455 -0.03148604435 0.0 rpy=0 0 0
- added joint left_2f_robotiq_85_right_finger_tip_joint: type continuous, parent left_2f_robotiq_85_right_inner_knuckle_link, child left_2f_robotiq_85_right_finger_tip_link, origin xyz=0.04303959807 -0.03759940821  0.0 rpy=0.0 0.0 0.0, axis 0 0 1, limit lower=-3.14 upper=3.14 effort=0.1 velocity=100.0, mimic joint=left_2f_robotiq_85_left_knuckle_joint multiplier=-1
- added joint left_2f_robotiq_85_right_inner_knuckle_joint: type continuous, parent left_2f_robotiq_85_base_link, child left_2f_robotiq_85_right_inner_knuckle_link, origin xyz=0.06142 -0.0127 0 rpy=0 0 0, axis 0 0 1, limit lower=-3.14 upper=3.14 effort=0.1 velocity=100.0, mimic joint=left_2f_robotiq_85_left_knuckle_joint offset=0
- added joint left_2f_robotiq_85_right_knuckle_joint: type continuous, parent left_2f_robotiq_85_base_link, child left_2f_robotiq_85_right_knuckle_link, origin xyz=0.05490451627 -0.03060114443 0.0 rpy=0.0 0.0 0.0, axis 0 0 1, limit lower=-3.14 upper=3.14 effort=1000 velocity=100.0, mimic joint=left_2f_robotiq_85_left_knuckle_joint
- added joint left_box_joint: type fixed, parent world, child left_box, origin xyz=0 0 0 rpy=0 0 0
- added joint left_ee_cam: type fixed, parent left_link_ee, child camera_arm_mount, origin xyz=0 0 0 rpy=0 0 3.14
- added joint left_side_wall_joint: type fixed, parent world, child left_side_wall, origin xyz=0 0 0 rpy=0 0 0
- added joint right_box_joint: type fixed, parent world, child right_box, origin xyz=0 0 0 rpy=0 0 0
- added joint right_side_wall_joint: type fixed, parent world, child right_side_wall, origin xyz=0 0 0 rpy=0 0 0
- added joint wooden_top_joint: type fixed, parent table_top, child wooden_top
- joint 2f_ee_tool0: parent left_link_ee -> camera_arm_mount
- joint adapter_mount: child 3f_palm -> a_3f_palm
- joint mount_left: parent world -> table_top
- joint mount_right: parent table -> table_top
- joint world_joint: child table -> table_top

Commit message: Updated the 3f gripper, to include a mounting plate

File: p6_ws/src/lbr_fri/lbr_fri_ros2_stack/lbr_description/urdf/dual_arm/dual_arm.urdf (robot description, URDF)
Before this commit: robot dual_arm, 52 links, 51 joints
Links:
- added link palm_adapter_mounting_plate; collision mesh filename=package://lbr_description/meshes/a_3f_palm_adapter/a_3f_pal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 scale=0.001 0.001 0.001; visual mesh filename=package://lbr_description/meshes/a_3f_palm_adapter/a_3f_pal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 scale=0.001 0.001 0.001
Joints:
- added joint plam_adapter_mount: type fixed, parent palm_adapter_mounting_plate, child a_3f_palm, origin xyz=0 0 0.0745 rpy=1.57079633 0 -1.57079633
- joint 2f_ee_tool0: origin xyz=0 0 0.165 rpy=0 3.14 0 -> xyz=0 0 0.195 rpy=0 3.14 0
- joint a_3f_palm_tool0: origin xyz=0.0 0.15 0 rpy=0 -1.5707 1.5707 -> xyz=0.0 0.173 0 rpy=0 -1.5707 1.5707
- joint adapter_mount: child a_3f_palm -> palm_adapter_mounting_plate; origin xyz=0 0 0.0745 rpy=1.57079633 0 -1.57079633 -> xyz=0 0 0.02 rpy=0 0 0
- joint right_side_wall_joint: origin xyz=0 0 0 rpy=0 0 0 -> xyz=-0.4 0 0 rpy=0 0 0

File: p6_ws/src/lbr_fri/lbr_fri_ros2_stack/lbr_description/urdf/dual_arm/dual_arm.xacro (robot description, xacro)
@@ -960,4 +960,19 @@
 	</collision>
   </link>
+  <link name="palm_adapter_mounting_plate">
+	<visual>
+	    <origin xyz="0 0 0.01" rpy="0 0 0"/>
+	    <geometry>
+	        <mesh filename="package://lbr_description/meshes/a_3f_palm_adapter/a_3f_palm_adapter.stl" scale="0.001 0.001 0.001"/>
+	    </geometry>
+	    <material name="steel_satin"/>
+	</visual>
+	<collision>
+	    <origin xyz="0 0 0" rpy="0 0 0"/>
+	    <geometry>
+	        <mesh filename="package://lbr_description/meshes/a_3f_palm_adapter/a_3f_palm_adapter.stl" scale="0.001 0.001 0.001"/>
+	    </geometry>
+	</collision>
+  </link>
   <!-- Camera arm mount -->
   <link name="camera_arm_mount">
@@ -1027,6 +1042,11 @@
   <joint name="adapter_mount" type="fixed">
 	  <parent link="gripper_mounting_plate" />
+	  <child link="palm_adapter_mounting_plate" />
+	  <origin xyz="0 0 0.02" rpy="0 0 0"/>
+  </joint>
+  <joint name="plam_adapter_mount" type="fixed">
+	  <parent link="palm_adapter_mounting_plate" />
 	  <child link="a_3f_palm" />
-	  <origin xyz="0 0 0.0945" rpy="1.57079633 0 -1.57079633"/>
+	  <origin xyz="0 0 0.0745" rpy="1.57079633 0 -1.57079633"/>
   </joint>
   <!-- joint between 3f gripper and 3f tool0-->
