Commit message: Updated xacro with new cell setup. Both visual and collision

File: p6_ws/src/lbr_fri/lbr_fri_ros2_stack/lbr_description/urdf/dual_arm/dual_arm.xacro (robot description, xacro)
@@ -1630,5 +1630,5 @@
     </collision>
   </link>
-  <!-- the wooden laser cut camera mount-->
+  <!-- the wooden laser cut camera mount
   <link name="cam_mount">
     <visual>
@@ -1640,4 +1640,5 @@
     </visual>
   </link>
+  -->
   <!-- 3f gripper adapter / mounting plate -->
   <link name="gripper_mounting_plate">
@@ -1661,5 +1662,5 @@
     <child link="table"/>
   </joint>
-  <!--joint between table and wooden camera mount-->
+  <!--joint between table and wooden camera mount
   <joint name="cam_table_joint" type="fixed">
     <parent link="table"/>
@@ -1667,9 +1668,10 @@
     <origin rpy="1.57079633 0 0" xyz="0.489819 0.84691 1.428"/>
   </joint>
+  -->
   <!--joint between table and right iiwa7 -->
   <joint name="mount_right" type="fixed">
     <parent link="table"/>
     <child link="right_link_0"/>
-    <origin rpy="0.785398163 0 -1.57079633" xyz="0.268524 0.756691 1.037203"/>
+    <origin rpy="0 0 -0.785398163" xyz="0.145181 0.79431 0.815"/>
   </joint>
   <!-- joint between right iiwa7 and 3f gripper-->
@@ -1689,5 +1691,5 @@
     <parent link="world"/>
     <child link="left_link_0"/>
-    <origin rpy="-0.785398163 0 -1.57079633" xyz="0.711114 0.756691 1.037203"/>
+    <origin rpy="0 0 -2.35619449 " xyz="0.795181 0.79431 0.815"/>
   </joint>
   <!-- joint between left iiwa7 and 2f gripper-->

Commit message: Updated mock xacro too

File: p6_ws/src/lbr_fri/lbr_fri_ros2_stack/lbr_description/urdf/dual_arm/dual_arm.xacro (robot description, xacro)
@@ -1687,7 +1687,7 @@
         <origin xyz="0 0 0.0745" rpy="1.57079633 0 -1.57079633"/>
     </joint>
-  <!-- joint between left arm and world -->
+  <!-- joint between left arm and table -->
   <joint name="mount_left" type="fixed">
-    <parent link="world"/>
+    <parent link="table"/>
     <child link="left_link_0"/>
     <origin rpy="0 0 -2.35619449 " xyz="0.795181 0.79431 0.815"/>

File: p6_ws/src/lbr_fri/lbr_fri_ros2_stack/lbr_description/urdf/isaac_dual_arm/dual_arm.xacro (robot description, xacro)
@@ -1,368 +1,221 @@
-<?xml version="1.0"?>
+<?xml version="1.0" ?>
+<!-- =================================================================================== -->
+<!-- |    This document was autogenerated by xacro from src/lbr_fri/lbr_fri_ros2_stack/lbr_description/urdf/dual_arm/dual_arm.xacro | -->
+<!-- |    EDITING THIS FILE BY HAND IS NOT RECOMMENDED                                 | -->
+<!-- =================================================================================== -->
 <!-- top level -->
-<robot xmlns:xacro="http://www.ros.org/wiki/xacro" name="mock_dual_arm">
-  <!-- Setup of Hardware & Joints for Right_Arm_Mock -->
+<robot name="dual_arm">
+  <!-- include the right iiwa7 macro wit table
+    <xacro:include filename="$(find lbr_description)/urdf/dual_arm/dual_arm_description.xacro" />
+    -->
   <ros2_control name="lbr_system_interface_right" type="system">
     <hardware>
-      <plugin>mock_components/GenericSystem</plugin>
+      <plugin>lbr_ros2_control::SystemInterface</plugin>
+      <param name="fri_client_sdk_major_version">1</param>
+      <param name="fri_client_sdk_minor_version">15</param>
+      <param name="client_command_mode">position</param>
+      <param name="port_id">30200</param>
+      <param name="remote_host">INADDR_ANY</param>
+      <param name="rt_prio">80</param>
+      <param name="pid_p">0.1</param>
+      <param name="pid_i">0.0</param>
+      <param name="pid_d">0.0</param>
+      <param name="pid_i_max">0.0</param>
+      <param name="pid_i_min">0.0</param>
+      <param name="pid_antiwindup">False</param>
+      <param name="command_guard_variant">default</param>
+      <param name="external_torque_cutoff_frequency">10</param>
+      <param name="measured_torque_cutoff_frequency">10</param>
+      <param name="open_loop">True</param>
     </hardware>
+    <sensor name="auxiliary_sensor">
+      <!-- see KUKA::FRI::LBRState -->
+      <state_interface name="sample_time"/>
+      <state_interface name="session_state"/>
+      <state_interface name="connection_quality"/>
+      <state_interface name="safety_state"/>
+      <state_interface name="operation_mode"/>
+      <state_interface name="drive_state"/>
+      <state_interface name="client_command_mode"/>
+      <state_interface name="overlay_type"/>
+      <state_interface name="control_mode"/>
+      <state_interface name="time_stamp_sec"/>
+      <state_interface name="time_stamp_nano_sec"/>
+      <state_interface name="tracking_performance"/>
+    </sensor>
+    <sensor name="estimated_ft_sensor">
+      <param name="chain_root">right_link_0</param>
+      <param name="chain_tip">right_link_ee</param>
+      <param name="damping">0.2</param>
+      <param name="force_x_th">2.0</param>
+      <param name="force_y_th">2.0</param>
+      <param name="force_z_th">2.0</param>
+      <param name="torque_x_th">0.5</param>
+      <param name="torque_y_th">0.5</param>
+      <param name="torque_z_th">0.5</param>
+      <state_interface name="force.x"/>
+      <state_interface name="force.y"/>
+      <state_interface name="force.z"/>
+      <state_interface name="torque.x"/>
+      <state_interface name="torque.y"/>
+      <state_interface name="torque.z"/>
+    </sensor>
+    <!-- FRI Cartesian impedance control mode -->
+    <gpio name="wrench">
+      <command_interface name="force.x"/>
+      <command_interface name="force.y"/>
+      <command_interface name="force.z"/>
+      <command_interface name="torque.x"/>
+      <command_interface name="torque.y"/>
+      <command_interface name="torque.z"/>
+    </gpio>
     <joint name="right_A1">
+      <param name="min_position">-2.9670597283903604</param>
+      <param name="max_position">2.9670597283903604</param>
       <param name="max_velocity">1.710422666954443</param>
+      <param name="max_torque">200</param>
       <command_interface name="position">
         <param name="min">-2.9670597283903604</param>
         <param name="max">2.9670597283903604</param>
       </command_interface>
-      <state_interface name="position">
-        <param name="initial_value">0</param>
-      </state_interface>
-      <state_interface name="velocity">
-        <param name="initial_value">0.0</param>
-      </state_interface>
+      <command_interface name="effort">
+        <param name="min">-200</param>
+        <param name="max"> 200</param>
+      </command_interface>
+      <state_interface name="position"/>
+      <state_interface name="velocity"/>
+      <state_interface name="effort"/>
+      <state_interface name="commanded_joint_position"/>
+      <state_interface name="commanded_torque"/>
+      <state_interface name="external_torque"/>
+      <state_interface name="ipo_joint_position"/>
     </joint>
     <joint name="right_A2">
+      <param name="min_position">-2.0943951023931953</param>
+      <param name="max_position">2.0943951023931953</param>
       <param name="max_velocity">1.710422666954443</param>
+      <param name="max_torque">200</param>
       <command_interface name="position">
         <param name="min">-2.0943951023931953</param>
         <param name="max">2.0943951023931953</param>
       </command_interface>
-      <state_interface name="position">
-        <param name="initial_value">0</param>
-      </state_interface>
-      <state_interface name="velocity">
-        <param name="initial_value">0.0</param>
-      </state_interface>
+      <command_interface name="effort">
+        <param name="min">-200</param>
+        <param name="max"> 200</param>
+      </command_interface>
+      <state_interface name="position"/>
+      <state_interface name="velocity"/>
+      <state_interface name="effort"/>
+      <state_interface name="commanded_joint_position"/>
+      <state_interface name="commanded_torque"/>
+      <state_interface name="external_torque"/>
+      <state_interface name="ipo_joint_position"/>
     </joint>
     <joint name="right_A3">
+      <param name="min_position">-2.9670597283903604</param>
+      <param name="max_position">2.9670597283903604</param>
       <param name="max_velocity">1.7453292519943295</param>
+      <param name="max_torque">200</param>
       <command_interface name="position">
         <param name="min">-2.9670597283903604</param>
         <param name="max">2.9670597283903604</param>
       </command_interface>
-      <state_interface name="position">
-        <param name="initial_value">0</param>
-      </state_interface>
-      <state_interface name="velocity">
-        <param name="initial_value">0.0</param>
-      </state_interface>
+      <command_interface name="effort">
+        <param name="min">-200</param>
+        <param name="max"> 200</param>
+      </command_interface>
+      <state_interface name="position"/>
+      <state_interface name="velocity"/>
+      <state_interface name="effort"/>
+      <state_interface name="commanded_joint_position"/>
+      <state_interface name="commanded_torque"/>
+      <state_interface name="external_torque"/>
+      <state_interface name="ipo_joint_position"/>
     </joint>
     <joint name="right_A4">
+      <param name="min_position">-2.0943951023931953</param>
+      <param name="max_position">2.0943951023931953</param>
       <param name="max_velocity">2.2689280275926285</param>
+      <param name="max_torque">200</param>
       <command_interface name="position">
         <param name="min">-2.0943951023931953</param>
         <param name="max">2.0943951023931953</param>
       </command_interface>
-      <state_interface name="position">
-        <param name="initial_value">0</param>
-      </state_interface>
-      <state_interface name="velocity">
-        <param name="initial_value">0.0</param>
-      </state_interface>
+      <command_interface name="effort">
+        <param name="min">-200</param>
+        <param name="max"> 200</param>
+      </command_interface>
+      <state_interface name="position"/>
+      <state_interface name="velocity"/>
+      <state_interface name="effort"/>
+      <state_interface name="commanded_joint_position"/>
+      <state_interface name="commanded_torque"/>
+      <state_interface name="external_torque"/>
+      <state_interface name="ipo_joint_position"/>
     </joint>
     <joint name="right_A5">
+      <param name="min_position">-2.9670597283903604</param>
+      <param name="max_position">2.9670597283903604</param>
       <param name="max_velocity">2.443460952792061</param>
+      <param name="max_torque">200</param>
       <command_interface name="position">
         <param name="min">-2.9670597283903604</param>
         <param name="max">2.9670597283903604</param>
       </command_interface>
-      <state_interface name="position">
-        <param name="initial_value">0</param>
-      </state_interface>
-      <state_interface name="velocity">
-        <param name="initial_value">0.0</param>
-      </state_interface>
+      <command_interface name="effort">
+        <param name="min">-200</param>
+        <param name="max"> 200</param>
+      </command_interface>
+      <state_interface name="position"/>
+      <state_interface name="velocity"/>
+      <state_interface name="effort"/>
+      <state_interface name="commanded_joint_position"/>
+      <state_interface name="commanded_torque"/>
+      <state_interface name="external_torque"/>
+      <state_interface name="ipo_joint_position"/>
     </joint>
     <joint name="right_A6">
+      <param name="min_position">-2.0943951023931953</param>
+      <param name="max_position">2.0943951023931953</param>
       <param name="max_velocity">3.141592653589793</param>
+      <param name="max_torque">200</param>
       <command_interface name="position">
         <param name="min">-2.0943951023931953</param>
         <param name="max">2.0943951023931953</param>
       </command_interface>
-      <state_interface name="position">
-        <param name="initial_value">0</param>
-      </state_interface>
-      <state_interface name="velocity">
-        <param name="initial_value">0.0</param>
-      </state_interface>
+      <command_interface name="effort">
+        <param name="min">-200</param>
+        <param name="max"> 200</param>
+      </command_interface>
+      <state_interface name="position"/>
+      <state_interface name="velocity"/>
+      <state_interface name="effort"/>
+      <state_interface name="commanded_joint_position"/>
+      <state_interface name="commanded_torque"/>
+      <state_interface name="external_torque"/>
+      <state_interface name="ipo_joint_position"/>
     </joint>
     <joint name="right_A7">
+      <param name="min_position">-3.0543261909900763</param>
+      <param name="max_position">3.0543261909900763</param>
       <param name="max_velocity">3.141592653589793</param>
+      <param name="max_torque">200</param>
       <command_interface name="position">
         <param name="min">-3.0543261909900763</param>
         <param name="max">3.0543261909900763</param>
       </command_interface>
-      <state_interface name="position">
-        <param name="initial_value">0</param>
-      </state_interface>
-      <state_interface name="velocity">
-        <param name="initial_value">0.0</param>
-      </state_interface>
+      <command_interface name="effort">
+        <param name="min">-200</param>
+        <param name="max"> 200</param>
+      </command_interface>
+      <state_interface name="position"/>
+      <state_interface name="velocity"/>
+      <state_interface name="effort"/>
+      <state_interface name="commanded_joint_position"/>
+      <state_interface name="commanded_torque"/>
+      <state_interface name="external_torque"/>
+      <state_interface name="ipo_joint_position"/>
     </joint>
   </ros2_control>
-  <!-- Setup of Hardware & Joints for Left_Arm_Mock -->
-  <ros2_control name="lbr_system_interface_left" type="system">
-    <hardware>
-      <plugin>mock_components/GenericSystem</plugin>
-    </hardware>
-    <joint name="left_A1">
-      <param name="max_velocity">1.710422666954443</param>
-      <command_interface name="position">
-        <param name="min">-2.9670597283903604</param>
-        <param name="max">2.9670597283903604</param>
-      </command_interface>
-      <state_interface name="position">
-        <param name="initial_value">0</param>
-      </state_interface>
-      <state_interface name="velocity">
-        <param name="initial_value">0.0</param>
-      </state_interface>
-    </joint>
-    <joint name="left_A2">
-      <param name="max_velocity">1.710422666954443</param>
-      <command_interface name="position">
-        <param name="min">-2.0943951023931953</param>
-        <param name="max">2.0943951023931953</param>
-      </command_interface>
-      <state_interface name="position">
-        <param name="initial_value">0</param>
-      </state_interface>
-      <state_interface name="velocity">
-        <param name="initial_value">0.0</param>
-      </state_interface>
-    </joint>
-    <joint name="left_A3">
-      <param name="max_velocity">1.7453292519943295</param>
-      <command_interface name="position">
-        <param name="min">-2.9670597283903604</param>
-        <param name="max">2.9670597283903604</param>
-      </command_interface>
-      <state_interface name="position">
-        <param name="initial_value">0</param>
-      </state_interface>
-      <state_interface name="velocity">
-        <param name="initial_value">0.0</param>
-      </state_interface>
-    </joint>
-    <joint name="left_A4">
-      <param name="max_velocity">2.2689280275926285</param>
-      <command_interface name="position">
-        <param name="min">-2.0943951023931953</param>
-        <param name="max">2.0943951023931953</param>
-      </command_interface>
-      <state_interface name="position">
-        <param name="initial_value">0</param>
-      </state_interface>
-      <state_interface name="velocity">
-        <param name="initial_value">0.0</param>
-      </state_interface>
-    </joint>
-    <joint name="left_A5">
-      <param name="max_velocity">2.443460952792061</param>
-      <command_interface name="position">
-        <param name="min">-2.9670597283903604</param>
-        <param name="max">2.9670597283903604</param>
-      </command_interface>
-      <state_interface name="position">
-        <param name="initial_value">0</param>
-      </state_interface>
-      <state_interface name="velocity">
-        <param name="initial_value">0.0</param>
-      </state_interface>
-    </joint>
-    <joint name="left_A6">
-      <param name="max_velocity">3.141592653589793</param>
-      <command_interface name="position">
-        <param name="min">-2.0943951023931953</param>
-        <param name="max">2.0943951023931953</param>
-      </command_interface>
-      <state_interface name="position">
-        <param name="initial_value">0</param>
-      </state_interface>
-      <state_interface name="velocity">
-        <param name="initial_value">0.0</param>
-      </state_interface>
-    </joint>
-    <joint name="left_A7">
-      <param name="max_velocity">3.141592653589793</param>
-      <command_interface name="position">
-        <param name="min">-3.0543261909900763</param>
-        <param name="max">3.0543261909900763</param>
-      </command_interface>
-      <state_interface name="position">
-        <param name="initial_value">0</param>
-      </state_interface>
-      <state_interface name="velocity">
-        <param name="initial_value">0.0</param>
-      </state_interface>
-    </joint>
-  </ros2_control>
-  <!-- Setup of Hardware for 3F Gripper -->
-  <ros2_control name="3FGripper" type="system">
-    <hardware>
-      <plugin>mock_components/GenericSystem</plugin>
-    </hardware>
-    <joint name="3f_finger_1_joint_1">
-      <param name="max_velocity">1.23</param>
-      <command_interface name="position">
-        <param name="min">0.3758</param>
-        <param name="max">1.1276</param>
-      </command_interface>
-      <state_interface name="position">
-        <param name="initial_value">0.3758</param>
-      </state_interface>
-      <state_interface name="velocity">
-        <param name="initial_value">0.0</param>
-      </state_interface>
-    </joint>
-    <joint name="3f_finger_1_joint_2">
-      <param name="max_velocity">1.24</param>
-      <command_interface name="position">
-        <param name="min">0.0</param>
-        <param name="max">1.5708</param>
-      </command_interface>
-      <state_interface name="position">
-        <param name="initial_value">0</param>
-      </state_interface>
-      <state_interface name="velocity">
-        <param name="initial_value">0.0</param>
-      </state_interface>
-    </joint>
-    <joint name="3f_finger_1_joint_3">
-      <param name="max_velocity">1.25</param>
-      <command_interface name="position">
-        <param name="min">-0.9531</param>
-        <param name="max">0.7572</param>
-      </command_interface>
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
File: p6_ws/src/lbr_fri/lbr_fri_ros2_stack/lbr_description/urdf/mock_dual_arm/old_mock_dual_arm.xacro (robot description, xacro)
@@ -1569,5 +1569,5 @@
     </collision>
   </link>
-  <!-- the wooden laser cut camera mount
+  <!-- the wooden laser cut camera mount-->
   <link name="cam_mount">
     <visual>
@@ -1579,5 +1579,4 @@
     </visual>
   </link>
-  -->
   <!-- 3f gripper adapter / mounting plate -->
   <link name="gripper_mounting_plate">
@@ -1601,5 +1600,5 @@
     <child link="table"/>
   </joint>
-  <!--joint between table and wooden camera mount
+  <!--joint between table and wooden camera mount-->
   <joint name="cam_table_joint" type="fixed">
     <parent link="table"/>
@@ -1607,10 +1606,9 @@
     <origin rpy="1.57079633 0 0" xyz="0.489819 0.84691 1.428"/>
   </joint>
-  -->
   <!--joint between table and right iiwa7 -->
   <joint name="mount_right" type="fixed">
     <parent link="table"/>
     <child link="right_link_0"/>
-    <origin rpy="0 0 -0.785398163" xyz="0.145181 0.79431 0.815"/>
+    <origin rpy="0.785398163 0 -1.57079633" xyz="0.268524 0.756691 1.037203"/>
   </joint>
   <!-- joint between right iiwa7 and 3f gripper-->
@@ -1626,9 +1624,9 @@
 	<origin xyz="0 0 0.0745" rpy="1.57079633 0 -1.57079633"/>
     </joint>
-  <!-- joint between left arm and table -->
+  <!-- joint between left arm and world -->
   <joint name="mount_left" type="fixed">
-    <parent link="table"/>
+    <parent link="world"/>
     <child link="left_link_0"/>
-    <origin rpy="0 0 -2.35619449 " xyz="0.795181 0.79431 0.815"/>
+    <origin rpy="-0.785398163 0 -1.57079633" xyz="0.711114 0.756691 1.037203"/>
   </joint>
   <!-- joint between left iiwa7 and 2f gripper-->
