Commit message: Made changes to the xacro yet again. Changed color and collision walls

File: p6_ws/src/lbr_fri/lbr_fri_ros2_stack/lbr_description/urdf/dual_arm/dual_arm.xacro (robot description, xacro)
@@ -2,5 +2,5 @@
 <!-- top level -->
 <robot xmlns:xacro="http://www.ros.org/wiki/xacro" name="isaac_dual_arm">
-  <!-- Setup of Hardware & Joints for kuka interface -->
+  <!-- Setup of Hardware & Joints for Right_Arm_Isaac -->
   <xacro:include filename="$(find dual_arm_moveit_config)/config/dual_arm.ros2_control.xacro"/>
   <!-- MATERIAL LIST -->
@@ -11,6 +11,9 @@
     <color rgba="0.1 0.1 0.1 1"/>
   </material>
+  <material name="steel_satin_old">
+    <color rgba="0.6274509803921569 0.6274509803921569 0.6274509803921569 1"/>
+  </material>
   <material name="steel_satin">
-    <color rgba="0.6274509803921569 0.6274509803921569 0.6274509803921569 1"/>
+    <color rgba="0.3 0.3 0.3 1"/>
   </material>
   <material name="wood">
@@ -18,8 +21,8 @@
   </material>
   <material name="white">
-    <color rgba="0.8 0.8 0.8 1"/>
+    <color rgba="0.9 0.9 0.9 1"/>
   </material>
   <material name="gray">
-	<color rgba="1 0 0 1"/>
+	<color rgba="0.6 0.6 0.6 1"/>
   </material>
   <!-- Links & Joints for the Right Arm -->
@@ -455,4 +458,708 @@
   <link name="left_link_ee">
 	</link>
+    <!-- link list -->
+  <link name="3f_finger_1_link_0">
+    <visual>
+      <origin rpy="0 0 0" xyz="0.020 0 0"/>
+      <geometry>
+	<mesh filename="package://lbr_description/meshes/robotiq-3f-gripper_articulated/visual/link_0.dae"/>
+      </geometry>
+      <material name="steel_satin"/>
+    </visual>
+    <collision>
+      <origin rpy="0 0 0" xyz="0.020 0 0"/>
+      <geometry>
+	<mesh filename="package://lbr_description/meshes/robotiq-3f-gripper_articulated/collision/link_0.STL"/>
+      </geometry>
+      <material name="yellow">
+	<color rgba="0 1 1 1"/>
+      </material>
+    </collision>
+    <inertial>
+      <origin rpy="0 0 0" xyz="0 0 0"/>
+      <mass value="0.05"/>
+      <inertia ixx="0.01" ixy="-0.00002" ixz="0.00001" iyy="0.0008" iyz="0" izz="0.001"/>
+    </inertial>
+  </link>
+  <link name="3f_finger_1_link_1">
+    <visual>
+      <origin rpy="0 0 -0.52" xyz="0.050 -.028 0"/>
+      <geometry>
+	<mesh filename="package://lbr_description/meshes/robotiq-3f-gripper_articulated/visual/link_1.dae"/>
+      </geometry>
+      <material name="steel_satin"/>
+    </visual>
+    <collision>
+      <origin rpy="0 0 -0.52" xyz="0.050 -.028 0"/>
+      <geometry>
+	<mesh filename="package://lbr_description/meshes/robotiq-3f-gripper_articulated/collision/link_1.STL"/>
+      </geometry>
+      <material name="yellow"/>
+    </collision>
+    <inertial>
+      <origin rpy="0 0 0" xyz="0 0 0"/>
+      <mass value="0.15"/>
+      <inertia ixx="0.001859" ixy="-0.000376" ixz="0.000028" iyy="0.012756" iyz="0" izz="0.0024"/>
+    </inertial>
+  </link>
+  <link name="3f_finger_1_link_2">
+    <visual>
+      <origin rpy="0 0 0" xyz="0.039 0 0.0075"/>
+      <geometry>
+	<mesh filename="package://lbr_description/meshes/robotiq-3f-gripper_articulated/visual/link_2.dae"/>
+      </geometry>
+      <material name="steel_satin"/>
+    </visual>
+    <collision>
+      <origin rpy="0 0 0" xyz="0.039 0 0.0075"/>
+      <geometry>
+	<mesh filename="package://lbr_description/meshes/robotiq-3f-gripper_articulated/collision/link_2.STL"/>
+      </geometry>
+      <material name="yellow"/>
+    </collision>
+    <inertial>
+      <origin rpy="0 0 0" xyz="0 0 0"/>
+      <mass value="0.15"/>
+      <inertia ixx="0.001859" ixy="-0.000376" ixz="0.000028" iyy="0.012756" iyz="0" izz="0.0024"/>
+    </inertial>
+  </link>
+  <link name="3f_finger_1_link_3">
+    <visual>
+      <origin rpy="0 0 0.52" xyz="0 0 0"/>
+      <geometry>
+	<mesh filename="package://lbr_description/meshes/robotiq-3f-gripper_articulated/visual/link_3.dae"/>
+      </geometry>
+      <material name="steel_satin"/>
+    </visual>
+    <collision>
+      <origin rpy="0 0 0.52" xyz="0 0 0"/>
+      <geometry>
+	<mesh filename="package://lbr_description/meshes/robotiq-3f-gripper_articulated/collision/link_3.STL"/>
+      </geometry>
+      <material name="yellow"/>
+    </collision>
+    <inertial>
+      <origin rpy="0 0 0" xyz="0 0 0"/>
+      <mass value="0.05"/>
+      <inertia ixx="0.001239" ixy="-0.000251" ixz="0.000019" iyy="0.00085" iyz="0" izz="0.001632"/>
+    </inertial>
+  </link>
+  <!-- end of link list -->
+  <!-- joint list -->
+  <joint name="3f_finger_1_joint_1" type="revolute">
+    <parent link="3f_finger_1_link_0"/>
+    <child link="3f_finger_1_link_1"/>
+    <axis xyz="0 0 1"/>
+    <origin rpy="0 0 -0.43" xyz="0.020 0 0"/>
+    <limit effort="100" lower="0.3758" upper="1.1276" velocity="1.23"/>
+    <dynamics damping="1" friction="0.1"/>
+  </joint>
+  <joint name="3f_finger_1_joint_2" type="revolute">
+    <parent link="3f_finger_1_link_1"/>
+    <child link="3f_finger_1_link_2"/>
+    <axis xyz="0 0 1"/>
+    <origin rpy="0 0 -0.52" xyz="0.050 -.028 0"/>
+    <limit effort="100" lower="0.0" upper="1.5707" velocity="1.24"/>
+    <dynamics damping="1" friction="0.1"/>
+  </joint>
+  <joint name="3f_finger_1_joint_3" type="revolute">
+    <parent link="3f_finger_1_link_2"/>
+    <child link="3f_finger_1_link_3"/>
+    <axis xyz="0 0 1"/>
+    <origin rpy="0 0 0" xyz="0.039 0 0"/>
+    <limit effort="100" lower="-0.9531" upper="0.7572" velocity="1.25"/>
+    <dynamics damping="1" friction="0.1"/>
+  </joint>
+  <!-- end of joint list -->
+  <!-- link list -->
+  <link name="3f_finger_2_link_0">
+    <visual>
+      <origin rpy="0 0 0" xyz="0.020 0 0"/>
+      <geometry>
+	<mesh filename="package://lbr_description/meshes/robotiq-3f-gripper_articulated/visual/link_0.dae"/>
+      </geometry>
+      <material name="steel_satin"/>
+    </visual>
+    <collision>
+      <origin rpy="0 0 0" xyz="0.020 0 0"/>
+      <geometry>
+	<mesh filename="package://lbr_description/meshes/robotiq-3f-gripper_articulated/collision/link_0.STL"/>
+      </geometry>
+      <material name="yellow">
+	<color rgba="0 1 1 1"/>
+      </material>
+    </collision>
+    <inertial>
+      <origin rpy="0 0 0" xyz="0 0 0"/>
+      <mass value="0.05"/>
+      <inertia ixx="0.01" ixy="-0.00002" ixz="0.00001" iyy="0.0008" iyz="0" izz="0.001"/>
+    </inertial>
+  </link>
+  <link name="3f_finger_2_link_1">
+    <visual>
+      <origin rpy="0 0 -0.52" xyz="0.050 -.028 0"/>
+      <geometry>
+	<mesh filename="package://lbr_description/meshes/robotiq-3f-gripper_articulated/visual/link_1.dae"/>
+      </geometry>
+      <material name="steel_satin"/>
+    </visual>
+    <collision>
+      <origin rpy="0 0 -0.52" xyz="0.050 -.028 0"/>
+      <geometry>
+	<mesh filename="package://lbr_description/meshes/robotiq-3f-gripper_articulated/collision/link_1.STL"/>
+      </geometry>
+      <material name="yellow"/>
+    </collision>
+    <inertial>
+      <origin rpy="0 0 0" xyz="0 0 0"/>
+      <mass value="0.15"/>
+      <inertia ixx="0.001859" ixy="-0.000376" ixz="0.000028" iyy="0.012756" iyz="0" izz="0.0024"/>
+    </inertial>
+  </link>
+  <link name="3f_finger_2_link_2">
+    <visual>
+      <origin rpy="0 0 0" xyz="0.039 0 0.0075"/>
+      <geometry>
+	<mesh filename="package://lbr_description/meshes/robotiq-3f-gripper_articulated/visual/link_2.dae"/>
+      </geometry>
+      <material name="steel_satin"/>
+    </visual>
+    <collision>
+      <origin rpy="0 0 0" xyz="0.039 0 0.0075"/>
+      <geometry>
+	<mesh filename="package://lbr_description/meshes/robotiq-3f-gripper_articulated/collision/link_2.STL"/>
+      </geometry>
+      <material name="yellow"/>
+    </collision>
+    <inertial>
+      <origin rpy="0 0 0" xyz="0 0 0"/>
+      <mass value="0.15"/>
+      <inertia ixx="0.001859" ixy="-0.000376" ixz="0.000028" iyy="0.012756" iyz="0" izz="0.0024"/>
+    </inertial>
+  </link>
+  <link name="3f_finger_2_link_3">
+    <visual>
+      <origin rpy="0 0 0.52" xyz="0 0 0"/>
+      <geometry>
+	<mesh filename="package://lbr_description/meshes/robotiq-3f-gripper_articulated/visual/link_3.dae"/>
+      </geometry>
+      <material name="steel_satin"/>
+    </visual>
+    <collision>
+      <origin rpy="0 0 0.52" xyz="0 0 0"/>
+      <geometry>
+	<mesh filename="package://lbr_description/meshes/robotiq-3f-gripper_articulated/collision/link_3.STL"/>
+      </geometry>
+      <material name="yellow"/>
+    </collision>
+    <inertial>
+      <origin rpy="0 0 0" xyz="0 0 0"/>
+      <mass value="0.05"/>
+      <inertia ixx="0.001239" ixy="-0.000251" ixz="0.000019" iyy="0.00085" iyz="0" izz="0.001632"/>
+    </inertial>
+  </link>
+  <!-- end of link list -->
+  <!-- joint list -->
+  <joint name="3f_finger_2_joint_1" type="revolute">
+    <parent link="3f_finger_2_link_0"/>
+    <child link="3f_finger_2_link_1"/>
+    <axis xyz="0 0 1"/>
+    <origin rpy="0 0 -0.43" xyz="0.020 0 0"/>
+    <limit effort="100" lower="0.3758" upper="1.1276" velocity="1.23"/>
+    <dynamics damping="1" friction="0.1"/>
+  </joint>
+  <joint name="3f_finger_2_joint_2" type="revolute">
+    <parent link="3f_finger_2_link_1"/>
+    <child link="3f_finger_2_link_2"/>
+    <axis xyz="0 0 1"/>
+    <origin rpy="0 0 -0.52" xyz="0.050 -.028 0"/>
+    <limit effort="100" lower="0.0" upper="1.5707" velocity="1.24"/>
+    <dynamics damping="1" friction="0.1"/>
+  </joint>
+  <joint name="3f_finger_2_joint_3" type="revolute">
+    <parent link="3f_finger_2_link_2"/>
+    <child link="3f_finger_2_link_3"/>
+    <axis xyz="0 0 1"/>
+    <origin rpy="0 0 0" xyz="0.039 0 0"/>
+    <limit effort="100" lower="-0.9531" upper="0.7572" velocity="1.25"/>
+    <dynamics damping="1" friction="0.1"/>
+  </joint>
+  <!-- end of joint list -->
+  <!-- link list -->
+  <link name="3f_finger_middle_link_0">
+    <visual>
+      <origin rpy="0 0 0" xyz="0.020 0 0"/>
+      <geometry>
+	<mesh filename="package://lbr_description/meshes/robotiq-3f-gripper_articulated/visual/link_0.dae"/>
+      </geometry>
+      <material name="steel_satin"/>
+    </visual>
+    <collision>
+      <origin rpy="0 0 0" xyz="0.020 0 0"/>
+      <geometry>
+	<mesh filename="package://lbr_description/meshes/robotiq-3f-gripper_articulated/collision/link_0.STL"/>
+      </geometry>
+      <material name="yellow">
+	<color rgba="0 1 1 1"/>
+      </material>
+    </collision>
+    <inertial>
+      <origin rpy="0 0 0" xyz="0 0 0"/>
+      <mass value="0.05"/>
+      <inertia ixx="0.01" ixy="-0.00002" ixz="0.00001" iyy="0.0008" iyz="0" izz="0.001"/>
+    </inertial>
+  </link>
+  <link name="3f_finger_middle_link_1">
+    <visual>
+      <origin rpy="0 0 -0.52" xyz="0.050 -.028 0"/>
+      <geometry>
+	<mesh filename="package://lbr_description/meshes/robotiq-3f-gripper_articulated/visual/link_1.dae"/>
+      </geometry>
+      <material name="steel_satin"/>
+    </visual>
+    <collision>
+      <origin rpy="0 0 -0.52" xyz="0.050 -.028 0"/>
+      <geometry>
+	<mesh filename="package://lbr_description/meshes/robotiq-3f-gripper_articulated/collision/link_1.STL"/>
+      </geometry>
+      <material name="yellow"/>
+    </collision>
+    <inertial>
+      <origin rpy="0 0 0" xyz="0 0 0"/>
+      <mass value="0.15"/>
+      <inertia ixx="0.001859" ixy="-0.000376" ixz="0.000028" iyy="0.012756" iyz="0" izz="0.0024"/>
+    </inertial>
+  </link>
+  <link name="3f_finger_middle_link_2">
+    <visual>
+      <origin rpy="0 0 0" xyz="0.039 0 0.0075"/>
+      <geometry>
+	<mesh filename="package://lbr_description/meshes/robotiq-3f-gripper_articulated/visual/link_2.dae"/>
+      </geometry>
+      <material name="steel_satin"/>
+    </visual>
+    <collision>
+      <origin rpy="0 0 0" xyz="0.039 0 0.0075"/>
+      <geometry>
+	<mesh filename="package://lbr_description/meshes/robotiq-3f-gripper_articulated/collision/link_2.STL"/>
+      </geometry>
+      <material name="yellow"/>
+    </collision>
+    <inertial>
+      <origin rpy="0 0 0" xyz="0 0 0"/>
+      <mass value="0.15"/>
+      <inertia ixx="0.001859" ixy="-0.000376" ixz="0.000028" iyy="0.012756" iyz="0" izz="0.0024"/>
+    </inertial>
+  </link>
+  <link name="3f_finger_middle_link_3">
+    <visual>
+      <origin rpy="0 0 0.52" xyz="0 0 0"/>
+      <geometry>
+	<mesh filename="package://lbr_description/meshes/robotiq-3f-gripper_articulated/visual/link_3.dae"/>
+      </geometry>
+      <material name="steel_satin"/>
+    </visual>
+    <collision>
+      <origin rpy="0 0 0.52" xyz="0 0 0"/>
+      <geometry>
+	<mesh filename="package://lbr_description/meshes/robotiq-3f-gripper_articulated/collision/link_3.STL"/>
+      </geometry>
+      <material name="yellow"/>
+    </collision>
+    <inertial>
+      <origin rpy="0 0 0" xyz="0 0 0"/>
+      <mass value="0.05"/>
+      <inertia ixx="0.001239" ixy="-0.000251" ixz="0.000019" iyy="0.00085" iyz="0" izz="0.001632"/>
+    </inertial>
+  </link>
+  <!-- end of link list -->
+  <!-- joint list -->
+  <joint name="3f_finger_middle_joint_1" type="revolute">
+    <parent link="3f_finger_middle_link_0"/>
+    <child link="3f_finger_middle_link_1"/>
+    <axis xyz="0 0 1"/>
+    <origin rpy="0 0 -0.43" xyz="0.020 0 0"/>
+    <limit effort="100" lower="0.3758" upper="1.1276" velocity="1.23"/>
+    <dynamics damping="1" friction="0.1"/>
+  </joint>
+  <joint name="3f_finger_middle_joint_2" type="revolute">
+    <parent link="3f_finger_middle_link_1"/>
+    <child link="3f_finger_middle_link_2"/>
+    <axis xyz="0 0 1"/>
+    <origin rpy="0 0 -0.52" xyz="0.050 -.028 0"/>
+    <limit effort="100" lower="0.0" upper="1.5707" velocity="1.24"/>
+    <dynamics damping="1" friction="0.1"/>
+  </joint>
+  <joint name="3f_finger_middle_joint_3" type="revolute">
+    <parent link="3f_finger_middle_link_2"/>
+    <child link="3f_finger_middle_link_3"/>
+    <axis xyz="0 0 1"/>
+    <origin rpy="0 0 0" xyz="0.039 0 0"/>
+    <limit effort="100" lower="-0.9531" upper="0.7572" velocity="1.25"/>
+    <dynamics damping="1" friction="0.1"/>
+  </joint>
+  <!-- end of joint list -->
+  <!-- link list -->
+  <link name="3f_palm">
+    <visual>
+      <geometry>
+	<mesh filename="package://lbr_description/meshes/robotiq-3f-gripper_articulated/visual/palm.dae"/>
+      </geometry>
+      <material name="steel_satin"/>
+    </visual>
+    <collision>
+      <geometry>
+	<mesh filename="package://lbr_description/meshes/robotiq-3f-gripper_articulated/collision/palm_with_finger_cutouts.stl"/>
+      </geometry>
+      <material name="yellow">
+	<color rgba="0 1 1 1"/>
+      </material>
+    </collision>
+  </link>
+  <link name="3f_tool0"/>
+  <inertial>
+    <origin rpy="0 0 0" xyz="0 0 0"/>
+    <mass value="1.3"/>
+    <inertia ixx="0.006012" ixy="0.000079" ixz="-0.00024" iyy="0.012892" iyz="0" izz="0.002435"/>
+  </inertial>
+  <!-- end of link list -->
+  <!-- joint list -->
+  <joint name="3f_palm_finger_1_joint" type="revolute">
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
File: p6_ws/src/lbr_fri/lbr_fri_ros2_stack/lbr_description/urdf/isaac_dual_arm/isaac_dual_arm.urdf (robot description, URDF)
Before this commit: robot isaac_dual_arm, 53 links, 52 joints
Links:
- removed link back_wall
- removed link left_side_wall
- removed link right_side_wall
- added link wooden_top; visual mesh filename=package://lbr_description/meshes/table/visual/Wooden_top.stl scale=0.001 0.001 0.001
- link table_top: geometry collision mesh filename=package://lbr_description/meshes/table/collision/Table_top.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 scale=0.001 0.001 0.001; visual mesh filename=package://lbr_description/meshes/table/visual/Table_top.stl scale=0.001 0.001 0.001
Joints:
- removed joint back_wall_joint
- removed joint left_side_wall_joint
- removed joint right_side_wall_joint
- added joint wooden_top_joint: type fixed, parent table_top, child wooden_top

File: p6_ws/src/lbr_fri/lbr_fri_ros2_stack/lbr_description/urdf/isaac_dual_arm/isaac_dual_arm.xacro (robot description, xacro)
@@ -11,6 +11,9 @@
     <color rgba="0.1 0.1 0.1 1"/>
   </material>
+  <material name="steel_satin_old">
+    <color rgba="0.6274509803921569 0.6274509803921569 0.6274509803921569 1"/>
+  </material>
   <material name="steel_satin">
-    <color rgba="0.6274509803921569 0.6274509803921569 0.6274509803921569 1"/>
+    <color rgba="0.3 0.3 0.3 1"/>
   </material>
   <material name="wood">
@@ -18,8 +21,8 @@
   </material>
   <material name="white">
-    <color rgba="0.8 0.8 0.8 1"/>
+    <color rgba="0.9 0.9 0.9 1"/>
   </material>
   <material name="gray">
-	<color rgba="1 0 0 1"/>
+	<color rgba="0.6 0.6 0.6 1"/>
   </material>
   <!-- Links & Joints for the Right Arm -->
@@ -462,5 +465,5 @@
 	<mesh filename="package://lbr_description/meshes/robotiq-3f-gripper_articulated/visual/link_0.dae"/>
       </geometry>
-      <material name="gray"/>
+      <material name="steel_satin"/>
     </visual>
     <collision>
@@ -485,5 +488,5 @@
 	<mesh filename="package://lbr_description/meshes/robotiq-3f-gripper_articulated/visual/link_1.dae"/>
       </geometry>
-      <material name="gray"/>
+      <material name="steel_satin"/>
     </visual>
     <collision>
@@ -506,5 +509,5 @@
 	<mesh filename="package://lbr_description/meshes/robotiq-3f-gripper_articulated/visual/link_2.dae"/>
       </geometry>
-      <material name="gray"/>
+      <material name="steel_satin"/>
     </visual>
     <collision>
@@ -527,5 +530,5 @@
 	<mesh filename="package://lbr_description/meshes/robotiq-3f-gripper_articulated/visual/link_3.dae"/>
       </geometry>
-      <material name="gray"/>
+      <material name="steel_satin"/>
     </visual>
     <collision>
@@ -576,5 +579,5 @@
 	<mesh filename="package://lbr_description/meshes/robotiq-3f-gripper_articulated/visual/link_0.dae"/>
       </geometry>
-      <material name="gray"/>
+      <material name="steel_satin"/>
     </visual>
     <collision>
@@ -599,5 +602,5 @@
 	<mesh filename="package://lbr_description/meshes/robotiq-3f-gripper_articulated/visual/link_1.dae"/>
       </geometry>
-      <material name="gray"/>
+      <material name="steel_satin"/>
     </visual>
     <collision>
@@ -620,5 +623,5 @@
 	<mesh filename="package://lbr_description/meshes/robotiq-3f-gripper_articulated/visual/link_2.dae"/>
       </geometry>
-      <material name="gray"/>
+      <material name="steel_satin"/>
     </visual>
     <collision>
@@ -641,5 +644,5 @@
 	<mesh filename="package://lbr_description/meshes/robotiq-3f-gripper_articulated/visual/link_3.dae"/>
       </geometry>
-      <material name="gray"/>
+      <material name="steel_satin"/>
     </visual>
     <collision>
@@ -690,5 +693,5 @@
 	<mesh filename="package://lbr_description/meshes/robotiq-3f-gripper_articulated/visual/link_0.dae"/>
       </geometry>
-      <material name="gray"/>
+      <material name="steel_satin"/>
     </visual>
     <collision>
@@ -713,5 +716,5 @@
 	<mesh filename="package://lbr_description/meshes/robotiq-3f-gripper_articulated/visual/link_1.dae"/>
       </geometry>
-      <material name="gray"/>
+      <material name="steel_satin"/>
     </visual>
     <collision>
@@ -734,5 +737,5 @@
 	<mesh filename="package://lbr_description/meshes/robotiq-3f-gripper_articulated/visual/link_2.dae"/>
       </geometry>
-      <material name="gray"/>
+      <material name="steel_satin"/>
     </visual>
     <collision>
@@ -755,5 +758,5 @@
 	<mesh filename="package://lbr_description/meshes/robotiq-3f-gripper_articulated/visual/link_3.dae"/>
       </geometry>
-      <material name="gray"/>
+      <material name="steel_satin"/>
     </visual>
     <collision>
@@ -803,5 +806,5 @@
 	<mesh filename="package://lbr_description/meshes/robotiq-3f-gripper_articulated/visual/palm.dae"/>
       </geometry>
-      <material name="gray"/>
+      <material name="steel_satin"/>
     </visual>
     <collision>
@@ -1171,5 +1174,5 @@
       <origin rpy="0 0 0" xyz="0 0 0"/>
       <geometry>
-	<mesh filename="package://lbr_description/meshes/table/visual/base_link_low_polly.stl" scale="0.001 0.001 0.001"/>
+	<mesh filename="package://lbr_description/meshes/table/visual/Table_top.stl" scale="0.001 0.001 0.001"/>
       </geometry>
       <material name="steel_satin"/>
@@ -1182,4 +1185,13 @@
     </collision>
   </link>
+  <link name="wooden_top">
+    <visual>
+      <origin rpy="0 0 0" xyz="0 0 0"/>
+      <geometry>
+	<mesh filename="package://lbr_description/meshes/table/visual/Wooden_top.stl" scale="0.001 0.001 0.001"/>
+      </geometry>
+      <material name="white"/>
+    </visual>
+  </link>
   <link name="left_side_wall">
     <collision>
@@ -1199,8 +1211,15 @@
   </link>
   <link name="back_wall">
-    <collision>
-      <origin rpy="0 0 0" xyz="0 0 0"/>
-      <geometry>
-	<mesh filename="package://lbr_description/meshes/table/collision/Back_wall.stl" scale="0.001 0.001 0.001"/>
+    <visual>
+	    <origin xyz="0 0.1 0" rpy="0 0 0"/>
+	    <geometry>
+	        <mesh filename="package://lbr_description/meshes/table/collision/Back_wall.stl" scale="0.001 0.001 0.001"/>
+	    </geometry>
+	    <material name="white"/>
+	  </visual>
+    <collision>
+      <origin rpy="0 0 0" xyz="0 0 0"/>
+      <geometry>
+	        <mesh filename="package://lbr_description/meshes/table/collision/Back_wall.stl" scale="0.001 0.001 0.001"/>
       </geometry>
     </collision>
@@ -1229,5 +1248,5 @@
 	        <mesh filename="package://lbr_description/meshes/gripper_mounting_plate/gripper_mounting_plate.stl" scale="0.001 0.001 0.001"/>
 	    </geometry>
-	    <material name="steel_satin"/>
+	    <material name="gray"/>
 	</visual>
 	<collision>
@@ -1260,4 +1279,8 @@
     <child link="table_top"/>
   </joint>
+  <joint name="wooden_top_joint" type="fixed">
+    <parent link="table_top"/>
+    <child link="wooden_top"/>
+  </joint>
   <joint name="left_side_wall_joint" type="fixed">
     <parent link="world"/>
