Commit message: Working on getting grippers to close in rviz when the real once do

File: p6_ws/src/lbr_fri/lbr_fri_ros2_stack/lbr_description/urdf/dual_arm/dual_arm.xacro (robot description, xacro)
@@ -4,4 +4,6 @@
   <!-- Setup of Hardware & Joints for Right_Arm_Isaac -->
   <xacro:include filename="$(find dual_arm_moveit_config)/config/dual_arm.ros2_control.xacro"/>
+  <!-- Gripper -->
+  <xacro:include filename="$(find lbr_description)/urdf/robotiq-2f-85-gripper/robotiq_85_gripper.urdf.xacro"/>
   <!-- MATERIAL LIST -->
   <material name="aluminum">
@@ -15,5 +17,5 @@
   </material>
   <material name="steel_satin">
-    <color rgba="0.3 0.3 0.3 1"/>
+    <color rgba="0.15 0.15 0.15 1"/>
   </material>
   <material name="wood">
@@ -459,5 +461,5 @@
 	</link>
     <!-- link list -->
-  <link name="3f_finger_1_link_0">
+  <link name="a_3f_finger_1_link_0">
     <visual>
       <origin rpy="0 0 0" xyz="0.020 0 0"/>
@@ -482,5 +484,5 @@
     </inertial>
   </link>
-  <link name="3f_finger_1_link_1">
+  <link name="a_3f_finger_1_link_1">
     <visual>
       <origin rpy="0 0 -0.52" xyz="0.050 -.028 0"/>
@@ -503,5 +505,5 @@
     </inertial>
   </link>
-  <link name="3f_finger_1_link_2">
+  <link name="a_3f_finger_1_link_2">
     <visual>
       <origin rpy="0 0 0" xyz="0.039 0 0.0075"/>
@@ -524,5 +526,5 @@
     </inertial>
   </link>
-  <link name="3f_finger_1_link_3">
+  <link name="a_3f_finger_1_link_3">
     <visual>
       <origin rpy="0 0 0.52" xyz="0 0 0"/>
@@ -546,8 +548,8 @@
   </link>
   <!-- end of link list -->
-  <!-- joint list -->
-  <joint name="3f_finger_1_joint_1" type="revolute">
-    <parent link="3f_finger_1_link_0"/>
-    <child link="3f_finger_1_link_1"/>
+  <!-- 3f joint list -->
+  <joint name="a_3f_finger_1_joint_1" type="revolute">
+    <parent link="a_3f_finger_1_link_0"/>
+    <child link="a_3f_finger_1_link_1"/>
     <axis xyz="0 0 1"/>
     <origin rpy="0 0 -0.43" xyz="0.020 0 0"/>
@@ -555,7 +557,7 @@
     <dynamics damping="1" friction="0.1"/>
   </joint>
-  <joint name="3f_finger_1_joint_2" type="revolute">
-    <parent link="3f_finger_1_link_1"/>
-    <child link="3f_finger_1_link_2"/>
+  <joint name="a_3f_finger_1_joint_2" type="revolute">
+    <parent link="a_3f_finger_1_link_1"/>
+    <child link="a_3f_finger_1_link_2"/>
     <axis xyz="0 0 1"/>
     <origin rpy="0 0 -0.52" xyz="0.050 -.028 0"/>
@@ -563,7 +565,7 @@
     <dynamics damping="1" friction="0.1"/>
   </joint>
-  <joint name="3f_finger_1_joint_3" type="revolute">
-    <parent link="3f_finger_1_link_2"/>
-    <child link="3f_finger_1_link_3"/>
+  <joint name="a_3f_finger_1_joint_3" type="revolute">
+    <parent link="a_3f_finger_1_link_2"/>
+    <child link="a_3f_finger_1_link_3"/>
     <axis xyz="0 0 1"/>
     <origin rpy="0 0 0" xyz="0.039 0 0"/>
@@ -573,5 +575,5 @@
   <!-- end of joint list -->
   <!-- link list -->
-  <link name="3f_finger_2_link_0">
+  <link name="a_3f_finger_2_link_0">
     <visual>
       <origin rpy="0 0 0" xyz="0.020 0 0"/>
@@ -596,5 +598,5 @@
     </inertial>
   </link>
-  <link name="3f_finger_2_link_1">
+  <link name="a_3f_finger_2_link_1">
     <visual>
       <origin rpy="0 0 -0.52" xyz="0.050 -.028 0"/>
@@ -617,5 +619,5 @@
     </inertial>
   </link>
-  <link name="3f_finger_2_link_2">
+  <link name="a_3f_finger_2_link_2">
     <visual>
       <origin rpy="0 0 0" xyz="0.039 0 0.0075"/>
@@ -638,5 +640,5 @@
     </inertial>
   </link>
-  <link name="3f_finger_2_link_3">
+  <link name="a_3f_finger_2_link_3">
     <visual>
       <origin rpy="0 0 0.52" xyz="0 0 0"/>
@@ -661,7 +663,7 @@
   <!-- end of link list -->
   <!-- joint list -->
-  <joint name="3f_finger_2_joint_1" type="revolute">
-    <parent link="3f_finger_2_link_0"/>
-    <child link="3f_finger_2_link_1"/>
+  <joint name="a_3f_finger_2_joint_1" type="revolute">
+    <parent link="a_3f_finger_2_link_0"/>
+    <child link="a_3f_finger_2_link_1"/>
     <axis xyz="0 0 1"/>
     <origin rpy="0 0 -0.43" xyz="0.020 0 0"/>
@@ -669,7 +671,7 @@
     <dynamics damping="1" friction="0.1"/>
   </joint>
-  <joint name="3f_finger_2_joint_2" type="revolute">
-    <parent link="3f_finger_2_link_1"/>
-    <child link="3f_finger_2_link_2"/>
+  <joint name="a_3f_finger_2_joint_2" type="revolute">
+    <parent link="a_3f_finger_2_link_1"/>
+    <child link="a_3f_finger_2_link_2"/>
     <axis xyz="0 0 1"/>
     <origin rpy="0 0 -0.52" xyz="0.050 -.028 0"/>
@@ -677,7 +679,7 @@
     <dynamics damping="1" friction="0.1"/>
   </joint>
-  <joint name="3f_finger_2_joint_3" type="revolute">
-    <parent link="3f_finger_2_link_2"/>
-    <child link="3f_finger_2_link_3"/>
+  <joint name="a_3f_finger_2_joint_3" type="revolute">
+    <parent link="a_3f_finger_2_link_2"/>
+    <child link="a_3f_finger_2_link_3"/>
     <axis xyz="0 0 1"/>
     <origin rpy="0 0 0" xyz="0.039 0 0"/>
@@ -687,5 +689,5 @@
   <!-- end of joint list -->
   <!-- link list -->
-  <link name="3f_finger_middle_link_0">
+  <link name="a_3f_finger_middle_link_0">
     <visual>
       <origin rpy="0 0 0" xyz="0.020 0 0"/>
@@ -710,5 +712,5 @@
     </inertial>
   </link>
-  <link name="3f_finger_middle_link_1">
+  <link name="a_3f_finger_middle_link_1">
     <visual>
       <origin rpy="0 0 -0.52" xyz="0.050 -.028 0"/>
@@ -731,5 +733,5 @@
     </inertial>
   </link>
-  <link name="3f_finger_middle_link_2">
+  <link name="a_3f_finger_middle_link_2">
     <visual>
       <origin rpy="0 0 0" xyz="0.039 0 0.0075"/>
@@ -752,5 +754,5 @@
     </inertial>
   </link>
-  <link name="3f_finger_middle_link_3">
+  <link name="a_3f_finger_middle_link_3">
     <visual>
       <origin rpy="0 0 0.52" xyz="0 0 0"/>
@@ -775,7 +777,7 @@
   <!-- end of link list -->
   <!-- joint list -->
-  <joint name="3f_finger_middle_joint_1" type="revolute">
-    <parent link="3f_finger_middle_link_0"/>
-    <child link="3f_finger_middle_link_1"/>
+  <joint name="a_3f_finger_middle_joint_1" type="revolute">
+    <parent link="a_3f_finger_middle_link_0"/>
+    <child link="a_3f_finger_middle_link_1"/>
     <axis xyz="0 0 1"/>
     <origin rpy="0 0 -0.43" xyz="0.020 0 0"/>
@@ -783,7 +785,7 @@
     <dynamics damping="1" friction="0.1"/>
   </joint>
-  <joint name="3f_finger_middle_joint_2" type="revolute">
-    <parent link="3f_finger_middle_link_1"/>
-    <child link="3f_finger_middle_link_2"/>
+  <joint name="a_3f_finger_middle_joint_2" type="revolute">
+    <parent link="a_3f_finger_middle_link_1"/>
+    <child link="a_3f_finger_middle_link_2"/>
     <axis xyz="0 0 1"/>
     <origin rpy="0 0 -0.52" xyz="0.050 -.028 0"/>
@@ -791,7 +793,7 @@
     <dynamics damping="1" friction="0.1"/>
   </joint>
-  <joint name="3f_finger_middle_joint_3" type="revolute">
-    <parent link="3f_finger_middle_link_2"/>
-    <child link="3f_finger_middle_link_3"/>
+  <joint name="a_3f_finger_middle_joint_3" type="revolute">
+    <parent link="a_3f_finger_middle_link_2"/>
+    <child link="a_3f_finger_middle_link_3"/>
     <axis xyz="0 0 1"/>
     <origin rpy="0 0 0" xyz="0.039 0 0"/>
@@ -801,5 +803,5 @@
   <!-- end of joint list -->
   <!-- link list -->
-  <link name="3f_palm">
+  <link name="a_3f_palm">
     <visual>
       <geometry>
@@ -817,5 +819,5 @@
     </collision>
   </link>
-  <link name="3f_tool0"/>
+  <link name="a_3f_tool0"/>
   <inertial>
     <origin rpy="0 0 0" xyz="0 0 0"/>
@@ -825,7 +827,7 @@
   <!-- end of link list -->
   <!-- joint list -->
-  <joint name="3f_palm_finger_1_joint" type="revolute">
-    <parent link="3f_palm"/>
-    <child link="3f_finger_1_link_0"/>
+  <joint name="a_3f_palm_finger_1_joint" type="revolute">
+    <parent link="a_3f_palm"/>
+    <child link="a_3f_finger_1_link_0"/>
     <axis xyz="0 1 0"/>
     <origin rpy="0 3.1416 -1.57" xyz="-0.0455 0.0214 0.036"/>
@@ -833,7 +835,7 @@
     <dynamics damping="1.0" friction="0.1"/>
   </joint>
-  <joint name="3f_palm_finger_2_joint" type="revolute">
-    <parent link="3f_palm"/>
-    <child link="3f_finger_2_link_0"/>
+  <joint name="a_3f_palm_finger_2_joint" type="revolute">
+    <parent link="a_3f_palm"/>
+    <child link="a_3f_finger_2_link_0"/>
     <axis xyz="0 1 0"/>
     <origin rpy="0 3.1416 -1.57" xyz="-0.0455 0.0214 -0.036"/>
@@ -841,326 +843,16 @@
     <dynamics damping="1.0" friction="0.1"/>
   </joint>
-  <joint name="3f_palm_finger_middle_joint" type="fixed">
-    <parent link="3f_palm"/>
-    <child link="3f_finger_middle_link_0"/>
+  <joint name="a_3f_palm_finger_middle_joint" type="fixed">
+    <parent link="a_3f_palm"/>
+    <child link="a_3f_finger_middle_link_0"/>
     <axis xyz="0 0 1"/>
     <origin rpy="0 0 1.57" xyz="0.0455 0.0214 0"/>
   </joint>
-  <!-- end of joint list -->
-  <link name="left_robotiq_arg2f_base_link">
-    <inertial>
-      <origin rpy="0 0 0" xyz="8.625E-08 -4.6583E-06 0.03145"/>
-      <mass value="0.22652"/>
-      <inertia ixx="0.00020005" ixy="-4.2442E-10" ixz="-2.9069E-10" iyy="0.00017832" iyz="-3.4402E-08" izz="0.00013478"/>
-    </inertial>
-    <visual>
-      <origin rpy="0 0 0" xyz="0 0 0"/>
-      <geometry>
-	<mesh filename="package://lbr_description/meshes/robotiq_2f_85_gripper/visual/robotiq_arg2f_85_base_link.dae" scale="0.001 0.001 0.001"/>
-      </geometry>
-      <material name="">
-	<color rgba="0.1 0.1 0.1 1"/>
-      </material>
-    </visual>
-    <collision>
-      <origin rpy="0 0 0" xyz="0 0 0"/>
-      <geometry>
-	<mesh filename="package://lbr_description/meshes/robotiq_2f_85_gripper/collision/robotiq_arg2f_base_link.stl"/>
-      </geometry>
-    </collision>
-  </link>
-  <link name="left_left_outer_knuckle">
-    <!--<inertial>
-	<origin xyz="-0.000200000000003065 0.0199435877845359 0.0292245259211331" rpy="0 0 0" />
-	<mass value="0.00853198276973456" />
-	<inertia ixx="2.89328108496468E-06" ixy="-1.57935047237397E-19" ixz="-1.93980378593255E-19" iyy="1.86719750325683E-06" iyz="-1.21858577871576E-06" izz="1.21905238907251E-06" />
-	</inertial> -->
-    <visual>
-      <origin rpy="0 0 0" xyz="0 0 0"/>
-      <geometry>
-	<mesh filename="package://lbr_description/meshes/robotiq_2f_85_gripper/visual/robotiq_arg2f_85_outer_knuckle.dae" scale="0.001 0.001 0.001"/>
-      </geometry>
-      <material name="">
-	<color rgba="0.792156862745098 0.819607843137255 0.933333333333333 1"/>
-      </material>
-    </visual>
-    <collision>
-      <origin rpy="0 0 0" xyz="0 0 0"/>
-      <geometry>
-	<mesh filename="package://lbr_description/meshes/robotiq_2f_85_gripper/collision/robotiq_arg2f_85_outer_knuckle.dae" scale="0.001 0.001 0.001"/>
-      </geometry>
-    </collision>
-  </link>
-  <link name="left_left_outer_finger">
-    <!--<inertial>
-	<origin xyz="0.00030115855001899 0.0373907951953854 -0.0208027427000385" rpy="0 0 0" />
-	<mass value="0.022614240507152" />
-	<inertia ixx="1.52518312458174E-05" ixy="9.76583423954399E-10" ixz="-5.43838577022588E-10" iyy="6.17694243867776E-06" iyz="6.78636130740228E-06" izz="1.16494917907219E-05" />
-	</inertial> -->
-    <visual>
-      <origin rpy="0 0 0" xyz="0 0 0"/>
-      <geometry>
-	<mesh filename="package://lbr_description/meshes/robotiq_2f_85_gripper/visual/robotiq_arg2f_85_outer_finger.dae" scale="0.001 0.001 0.001"/>
-      </geometry>
-      <material name="">
-	<color rgba="0.1 0.1 0.1 1"/>
-      </material>
-    </visual>
-    <collision>
-      <origin rpy="0 0 0" xyz="0 0 0"/>
-      <geometry>
-	<mesh filename="package://lbr_description/meshes/robotiq_2f_85_gripper/collision/robotiq_arg2f_85_outer_finger.dae" scale="0.001 0.001 0.001"/>
-      </geometry>
-    </collision>
-  </link>
-  <link name="left_left_inner_finger">
-    <!--<inertial>
-	<origin xyz="0.000299999999999317 0.0160078233491243 -0.0136945669206257" rpy="0 0 0" />
-	<mass value="0.0104003125914103" />
-	<inertia ixx="2.71909453810972E-06" ixy="1.35402465472579E-21" ixz="-7.1817349065269E-22" iyy="7.69100314106116E-07" iyz="6.74715432769696E-07" izz="2.30315190420171E-06" />
-	</inertial> -->
-    <visual>
-      <origin rpy="0 0 0" xyz="0 0 0"/>
-      <geometry>
-	<mesh filename="package://lbr_description/meshes/robotiq_2f_85_gripper/visual/robotiq_arg2f_85_inner_finger.dae" scale="0.001 0.001 0.001"/>
-      </geometry>
-      <material name="">
-	<color rgba="0.1 0.1 0.1 1"/>
-      </material>
-    </visual>
-    <collision>
-      <origin rpy="0 0 0" xyz="0 0 0"/>
-      <geometry>
-	<mesh filename="package://lbr_description/meshes/robotiq_2f_85_gripper/collision/robotiq_arg2f_85_inner_finger.dae" scale="0.001 0.001 0.001"/>
-      </geometry>
-    </collision>
-  </link>
-  <link name="left_left_inner_finger_pad">
-    <visual>
-      <origin rpy="0 0 0" xyz="0 0 0"/>
-      <geometry>
-	<box size="0.022 0.00635 0.0375"/>
-      </geometry>
-      <material name="">
-	<color rgba="0.9 0.9 0.9 1"/>
-      </material>
-    </visual>
-    <collision>
-      <origin rpy="0 0 0" xyz="0 0 0"/>
-      <geometry>
-	<box size="0.022 0.00635 0.0375"/>
-      </geometry>
-      <material name="">
-	<color rgba="0.9 0.0 0.0 1"/>
-      </material>
-    </collision>
-  </link>
-  <link name="left_left_inner_knuckle">
-    <!--<inertial>
-	<origin xyz="0.000123011831763771 0.0507850843201817 0.00103968640075166" rpy="0 0 0" />
-       <mass value="0.0271177346495152" />
-	<inertia ixx="2.61910379223783E-05" ixy="-2.43616858946494E-07" ixz="-6.37789906117123E-09" iyy="2.8270243746167E-06" iyz="-5.37200748039765E-07" izz="2.83695868220296E-05" />
-	</inertial> -->
-    <visual>
-      <origin rpy="0 0 0" xyz="0 0 0"/>
-      <geometry>
-	<mesh filename="package://lbr_description/meshes/robotiq_2f_85_gripper/visual/robotiq_arg2f_85_inner_knuckle.dae" scale="0.001 0.001 0.001"/>
-      </geometry>
-      <material name="">
-	<color rgba="0.1 0.1 0.1 1"/>
-      </material>
-    </visual>
-    <collision>
-      <origin rpy="0 0 0" xyz="0 0 0"/>
-      <geometry>
-	<mesh filename="package://lbr_description/meshes/robotiq_2f_85_gripper/collision/robotiq_arg2f_85_inner_knuckle.dae" scale="0.001 0.001 0.001"/>
-      </geometry>
-    </collision>
-  </link>
-  <link name="left_right_outer_knuckle">
-    <!--<inertial>
-	<origin xyz="-0.000200000000003065 0.0199435877845359 0.0292245259211331" rpy="0 0 0" />
-	<mass value="0.00853198276973456" />
-	<inertia ixx="2.89328108496468E-06" ixy="-1.57935047237397E-19" ixz="-1.93980378593255E-19" iyy="1.86719750325683E-06" iyz="-1.21858577871576E-06" izz="1.21905238907251E-06" />
-	</inertial> -->
-    <visual>
-      <origin rpy="0 0 0" xyz="0 0 0"/>
-      <geometry>
-	<mesh filename="package://lbr_description/meshes/robotiq_2f_85_gripper/visual/robotiq_arg2f_85_outer_knuckle.dae" scale="0.001 0.001 0.001"/>
-      </geometry>
-      <material name="">
-	<color rgba="0.792156862745098 0.819607843137255 0.933333333333333 1"/>
-      </material>
-    </visual>
-    <collision>
-      <origin rpy="0 0 0" xyz="0 0 0"/>
-      <geometry>
-	<mesh filename="package://lbr_description/meshes/robotiq_2f_85_gripper/collision/robotiq_arg2f_85_outer_knuckle.dae" scale="0.001 0.001 0.001"/>
-      </geometry>
-    </collision>
-  </link>
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
File: p6_ws/src/lbr_fri/lbr_fri_ros2_stack/lbr_description/urdf/isaac_dual_arm/isaac_dual_arm.xacro (robot description, xacro)
@@ -911,5 +911,5 @@
 	  </visual>
     <collision>
-      <origin rpy="0 0 0" xyz="0 0 0"/>
+      <origin rpy="0 0.1 0" xyz="0 0 0"/>
       <geometry>
 	        <mesh filename="package://lbr_description/meshes/table/collision/Back_wall.stl" scale="0.001 0.001 0.001"/>

Commit message: trasitional grasping algorithm works now. it plots the grasps and is correctly rotated. The angles are minimised,  a -90 rotation is added to the grasp, and center points are tranfslated to world frame.

File: p6_ws/src/lbr_fri/lbr_fri_ros2_stack/lbr_description/urdf/dual_arm/dual_arm.xacro (robot description, xacro)
@@ -1212,5 +1212,5 @@
   <link name="back_wall">
     <visual>
-	    <origin xyz="0 0.1 0" rpy="0 0 0"/>
+	    <origin xyz="0 0.2 0" rpy="0 0 0"/>
 	    <geometry>
 	        <mesh filename="package://lbr_description/meshes/table/collision/Back_wall.stl" scale="0.001 0.001 0.001"/>

Commit message: Fully functional implementation of GraspNet-Baseline, performance seems low, but it's capable of grasping

File: p6_ws/src/lbr_fri/lbr_fri_ros2_stack/lbr_description/urdf/dual_arm/dual_arm.xacro (robot description, xacro)
@@ -1219,5 +1219,5 @@
 	  </visual>
     <collision>
-      <origin rpy="0 0 0" xyz="0 0 0"/>
+      <origin rpy="0 0 0" xyz="0 0.1 0"/>
       <geometry>
 	        <mesh filename="package://lbr_description/meshes/table/collision/Back_wall.stl" scale="0.001 0.001 0.001"/>

Commit message: Changed dummy function list

File: p6_ws/src/lbr_fri/lbr_fri_ros2_stack/lbr_description/urdf/dual_arm/dual_arm.xacro (robot description, xacro)
@@ -994,5 +994,5 @@
     <parent link="world"/>
     <child link="right_side_wall"/>
-    <origin xyz="0 0 0" rpy="0 0 0"/>
+    <origin xyz="-0.2 0 0" rpy="0 0 0"/>
   </joint>
   <joint name="back_wall_joint" type="fixed">

Commit message: changed 3f grippes frame placement so its at the tip. and added translations to match it for grasps

File: p6_ws/src/lbr_fri/lbr_fri_ros2_stack/lbr_description/urdf/dual_arm/dual_arm.xacro (robot description, xacro)
@@ -832,5 +832,5 @@
   <link name="a_3f_tool0"/>
   <inertial>
-    <origin rpy="0 0 0" xyz="0 0 0"/>
+    <origin rpy="0 0 0" xyz="0 0 -0.01"/>
     <mass value="1.3"/>
     <inertia ixx="0.006012" ixy="0.000079" ixz="-0.00024" iyy="0.012892" iyz="0" izz="0.002435"/>

Commit message: Added no general grasp when z_max less than 7 cm. chanced frames in dual_arms so grasps of small items are possible. made translation so objects gets grasped even though gripper only moves its tip to pose.

File: p6_ws/src/lbr_fri/lbr_fri_ros2_stack/lbr_description/urdf/dual_arm/dual_arm.xacro (robot description, xacro)
@@ -832,5 +832,5 @@
   <link name="a_3f_tool0"/>
   <inertial>
-    <origin rpy="0 0 0" xyz="0 0 -0.01"/>
+    <origin rpy="0 0 0" xyz="0 0 0"/>
     <mass value="1.3"/>
     <inertia ixx="0.006012" ixy="0.000079" ixz="-0.00024" iyy="0.012892" iyz="0" izz="0.002435"/>
@@ -1028,5 +1028,5 @@
 	  <parent link="gripper_mounting_plate" />
 	  <child link="a_3f_palm" />
-	  <origin xyz="0 0 0.0745" rpy="1.57079633 0 -1.57079633"/>
+	  <origin xyz="0 0 0.0945" rpy="1.57079633 0 -1.57079633"/>
   </joint>
   <!-- joint between 3f gripper and 3f tool0-->
@@ -1034,5 +1034,5 @@
     <parent link="a_3f_palm"/>
     <child link="a_3f_tool0"/>
-    <origin rpy="0 -1.5707 1.5707" xyz="0.0 0.15 0"/>
+    <origin rpy="0 -1.5707 1.5707" xyz="0.0 0.18 0"/>
   </joint>
   <!-- JOINTS FOR LEFT ARM AND 2F GRIPPER -->

Commit message: callibrated the left arm. added new image pose. made sure no negetaive grasp is returned.

File: p6_ws/src/lbr_fri/lbr_fri_ros2_stack/lbr_description/urdf/dual_arm/dual_arm.xacro (robot description, xacro)
@@ -1034,5 +1034,5 @@
     <parent link="a_3f_palm"/>
     <child link="a_3f_tool0"/>
-    <origin rpy="0 -1.5707 1.5707" xyz="0.0 0.18 0"/>
+    <origin rpy="0 -1.5707 1.5707" xyz="0.0 0.173 0"/>
   </joint>
   <!-- JOINTS FOR LEFT ARM AND 2F GRIPPER -->
@@ -1060,5 +1060,5 @@
     <parent link="camera_arm_mount"/>
     <child link="2f_tool0"/>
-    <origin rpy="0 3.14 0" xyz="0 0 0.165"/>
+    <origin rpy="0 3.14 0" xyz="0 0 0.195"/>
   </joint>
 </robot>

Commit message: LangraphManager file created.

File: p6_ws/src/lbr_fri/lbr_fri_ros2_stack/lbr_description/urdf/dual_arm/dual_arm.xacro (robot description, xacro)
@@ -922,5 +922,5 @@
 	  </visual>
     <collision>
-      <origin xyz="0 0.1 0" rpy="0 0 0"/>
+      <origin xyz="0 0.2 0" rpy="0 0 0"/>
       <geometry>
 	        <mesh filename="package://lbr_description/meshes/table/collision/Back_wall.stl" scale="0.001 0.001 0.001"/>
@@ -994,5 +994,5 @@
     <parent link="world"/>
     <child link="right_side_wall"/>
-    <origin xyz="-0.2 0 0" rpy="0 0 0"/>
+    <origin xyz="-0.4 0 0" rpy="0 0 0"/>
   </joint>
   <joint name="back_wall_joint" type="fixed">

Commit message: Still trying to fix left-hand rule in system, commit to swap branches

File: p6_ws/src/lbr_fri/lbr_fri_ros2_stack/lbr_description/urdf/dual_arm/dual_arm.xacro (robot description, xacro)
@@ -1331,5 +1331,5 @@
     <parent link="3f_palm"/>
     <child link="3f_tool0"/>
-    <origin rpy="0 -1.5707 1.5707" xyz="0.0 0.15 0"/>
+    <origin rpy="0 -1.5707 1.5707" xyz="0.0 0.173 0"/>
   </joint>
   <!-- JOINTS FOR LEFT ARM AND 2F GRIPPER -->
@@ -1356,5 +1356,5 @@
     <parent link="camera_arm_mount"/>
     <child link="2f_tool0"/>
-    <origin rpy="0 3.14 0" xyz="0 0 0.165"/>
+    <origin rpy="0 3.14 0" xyz="0 0 0.195"/>
   </joint>
 </robot>

Commit message: Changed planner

File: p6_ws/src/lbr_fri/lbr_fri_ros2_stack/lbr_description/urdf/dual_arm/dual_arm.xacro (robot description, xacro)
@@ -932,5 +932,5 @@
       <origin rpy="0 0 0" xyz="0 0 0"/>
       <geometry>
-	<mesh filename="package://lbr_description/meshes/table/collision/Side_box.stl" scale="0.001 0.001 0.001"/>
+	<mesh filename="package://lbr_description/meshes/table/collision/Left_side_box.stl" scale="0.001 0.001 0.001"/>
       </geometry>
     </collision>
@@ -938,7 +938,7 @@
   <link name="right_box">
     <collision>
-      <origin rpy="0 0 0" xyz="-1.181 0 0"/>
-      <geometry>
-	<mesh filename="package://lbr_description/meshes/table/collision/Side_box.stl" scale="0.001 0.001 0.001"/>
+      <origin rpy="0 0 0" xyz="0 0 0"/>
+      <geometry>
+	<mesh filename="package://lbr_description/meshes/table/collision/Right_side_box.stl" scale="0.001 0.001 0.001"/>
       </geometry>
     </collision>

File: p6_ws/src/lbr_fri/lbr_fri_ros2_stack/lbr_moveit_config/dual_arm_moveit_config/config/dual_arm.ros2_control.xacro (robot description, xacro)
@@ -548,5 +548,5 @@
       </command_interface>
       <state_interface name="position">
-        <param name="initial_value">-0.1784</param>
+        <param name="initial_value">0.0</param>
       </state_interface>
       <state_interface name="velocity">
@@ -561,5 +561,5 @@
       </command_interface>
       <state_interface name="position">
-        <param name="initial_value">-0.192</param>
+        <param name="initial_value">0.0</param>
       </state_interface>
       <state_interface name="velocity">
