Commit message: Added the new camera tower to the xacro

File: p6_ws/src/lbr_fri/lbr_fri_ros2_stack/lbr_description/urdf/dual_arm/dual_arm.xacro (robot description, xacro)
@@ -869,9 +869,4 @@
   <!-- Table and wall links -->
   <link name="table_top">
-    <inertial>
-      <origin rpy="0 0 0" xyz="0.47511520643410643 0.9340356249199337 1.753635248949686"/>
-      <mass value="1382.7919279449686"/>
-      <inertia ixx="1994.27355" ixy="-0.365832" ixz="-0.552572" iyy="2787.103818" iyz="-145.275916" izz="966.579181"/>
-    </inertial>
     <visual>
       <origin rpy="0 0 0" xyz="0 0 0"/>
@@ -941,4 +936,19 @@
       <geometry>
 	<mesh filename="package://lbr_description/meshes/table/collision/Right_side_box.stl" scale="0.001 0.001 0.001"/>
+      </geometry>
+    </collision>
+  </link>
+  <link name="table_tower">
+    <visual>
+      <origin rpy="0 0 0" xyz="0 0 1.65"/>
+      <geometry>
+	<mesh filename="package://lbr_description/meshes/table/visual/Table_tower.stl" scale="0.001 0.001 0.001"/>
+      </geometry>
+      <material name="gray"/>
+    </visual>
+    <collision>
+      <origin rpy="0 0 0" xyz="0 0 0"/>
+      <geometry>
+	<mesh filename="package://lbr_description/meshes/table/collision/Table_tower.stl" scale="0.001 0.001 0.001"/>
       </geometry>
     </collision>
@@ -1026,4 +1036,9 @@
     <origin xyz="0 0 0" rpy="0 0 0"/>
   </joint>
+  <joint name="tower_joint" type="fixed">
+    <parent link="world"/>
+    <child link="table_tower"/>
+    <origin xyz="0 0 0" rpy="0 0 0"/>
+  </joint>
   <!-- JOINTS FOR RIGHT ARM AND 3F GRIPPER -->
   <!--Joint between table and right iiwa7 -->
